File: plat_power.kicad_pcb (KiCad board)
At the start: 2 copper layers, 100 x 100 mm, 120 parts, among them Con2 DG125-5.0-02P-14-00A(H), U1 LD39050PU33R, U2 TPS5450, U3 KF33BD-TR, U4 TPS5450, U5 TPS5450

Commit message: Add files via upload
Parts:
- removed C3_TANTAL1, C4_TANTAL1, C5_TANTAL1, C6_TANTAL1, C8_TANTAL1, C9_TANTAL1: 10uF, Capacitor_SMD:C_0603_1608Metric
- removed Con2: DG125-5.0-02P-14-00A(H), TerminalBlock_Phoenix:TerminalBlock_Phoenix_MKDS-1,5-2_1x02_P5.00mm_Horizontal
- removed LED1: Green, LED_SMD:LED_0603_1608Metric
- removed con1: ~, Connector_PinHeader_1.00mm:PinHeader_1x04_P1.00mm_Horizontal
- added C27: 100nF, Capacitor_SMD:C_0603_1608Metric, F.Cu at (196.5, 132.0)
- added C42: 100nF, Capacitor_SMD:C_0603_1608Metric, F.Cu at (117.8, 91.0)
- added C43: 10uF, Capacitor_SMD:C_0603_1608Metric, F.Cu at (117.8, 93.5)
- added C44: 100nF, Capacitor_SMD:C_0603_1608Metric, F.Cu at (117.8, 96.0)
- added C45: 10uF, Capacitor_SMD:C_0603_1608Metric, F.Cu at (117.8, 98.5)
- added C46: 100nF, Capacitor_SMD:C_0603_1608Metric, F.Cu at (117.8, 101.0)
- added C47: 10uF, Capacitor_SMD:C_0603_1608Metric, F.Cu at (117.8, 103.5)
- added C48: 100nF, Capacitor_SMD:C_0603_1608Metric, F.Cu at (117.8, 106.0)
- added C49: 100nF, Capacitor_SMD:C_0603_1608Metric, F.Cu at (117.8, 108.6)
- added C50: 100nF, Capacitor_SMD:C_0603_1608Metric, F.Cu at (117.8, 111.1)
- added C51: 100nF, Capacitor_SMD:C_0603_1608Metric, F.Cu at (117.8, 113.6)
- added C52: 100nF, Capacitor_SMD:C_0603_1608Metric, F.Cu at (31.5, 22.0)
- added C53: 100nF, Capacitor_SMD:C_0603_1608Metric, F.Cu at (121.8, 88.5)
- added C54: 100nF, Capacitor_SMD:C_0603_1608Metric, F.Cu at (121.8, 91.0)
- added Con1: ~, Connector_PinHeader_1.00mm:PinHeader_1x02_P1.00mm_Vertical, F.Cu at (222.0, 85.0)
- added Con3: DG125-5.0-02P-14-00A(H), TerminalBlock_Phoenix:TerminalBlock_Phoenix_MKDS-1,5-2_1x02_P5.00mm_Horizontal, F.Cu at (244.5, 91.5)
- added Con4: ~, Connector_PinHeader_1.00mm:PinHeader_1x02_P1.00mm_Vertical, F.Cu at (139.9, 180.8)
- added D30: SS54L, Diode_SMD:D_0603_1608Metric, F.Cu at (159.2, 132.6)
- added J1: Conn_01x05_Pin, Connector_PinHeader_1.00mm:PinHeader_1x05_P1.00mm_Vertical, F.Cu at (149.3, 165.0)
- added J2: Conn_01x05_Pin, Connector_PinHeader_1.00mm:PinHeader_1x05_P1.00mm_Vertical, F.Cu at (152.7, 165.0)
- added J3: Conn_01x05_Pin, Connector_PinHeader_1.00mm:PinHeader_1x05_P1.00mm_Vertical, F.Cu at (156.0, 165.0)
- added J4: Conn_01x05_Pin, Connector_PinHeader_1.00mm:PinHeader_1x05_P1.00mm_Vertical, F.Cu at (159.3, 165.0)
- added J5: Conn_01x05_Pin, Connector_PinHeader_1.00mm:PinHeader_1x05_P1.00mm_Vertical, F.Cu at (162.7, 165.0)
- added J6: Conn_01x05_Pin, Connector_PinHeader_1.00mm:PinHeader_1x05_P1.00mm_Vertical, F.Cu at (166.0, 165.0)
- added JP1: Jumper_3_Open, Jumper:SolderJumper-3_P1.3mm_Bridged123_Pad1.0x1.5mm, F.Cu at (193.0, 56.3)
- added JP2: Jumper_3_Open, Jumper:SolderJumper-3_P1.3mm_Bridged123_Pad1.0x1.5mm, F.Cu at (182.7, 94.5)
- added JP3: Jumper_3_Open, Jumper:SolderJumper-3_P1.3mm_Bridged123_Pad1.0x1.5mm, F.Cu at (186.5, 133.0)
- added JP4: Jumper_3_Open, Jumper:SolderJumper-3_P1.3mm_Bridged123_Pad1.0x1.5mm, F.Cu at (161.7, 181.7)
- added JP5: Jumper_3_Open, Jumper:SolderJumper-3_P1.3mm_Bridged123_Pad1.0x1.5mm, F.Cu at (161.7, 185.5)
- added JP6: Jumper_3_Open, Jumper:SolderJumper-3_P1.3mm_Bridged123_Pad1.0x1.5mm, F.Cu at (161.7, 189.3)
- added JP7: Jumper_3_Open, Jumper:SolderJumper-3_P1.3mm_Bridged123_Pad1.0x1.5mm, F.Cu at (167.3, 181.7)
- added JP8: Jumper_3_Open, Jumper:SolderJumper-3_P1.3mm_Bridged123_Pad1.0x1.5mm, F.Cu at (167.3, 185.5)
- added JP9: Jumper_3_Open, Jumper:SolderJumper-3_P1.3mm_Bridged123_Pad1.0x1.5mm, F.Cu at (167.3, 189.3)
- added R10: 10k, Resistor_SMD:R_0805_2012Metric, F.Cu at (202.0, 114.5)
- added R11: 6.8K, Resistor_SMD:R_0805_2012Metric, F.Cu at (195.5, 116.0)
- added R12: 1, Resistor_SMD:R_0603_1608Metric, F.Cu at (200.0, 131.0)
- added R13: 10m, Resistor_SMD:R_0805_2012Metric, F.Cu at (203.0, 132.0)
- added R14: 1, Resistor_SMD:R_0603_1608Metric, F.Cu at (199.5, 133.5)
- added R18: 1k, Resistor_SMD:R_0805_2012Metric, F.Cu at (140.7, 90.6)
- added R19: 1k, Resistor_SMD:R_0805_2012Metric, F.Cu at (20.0, 33.5)
- added R20: 1k, Resistor_SMD:R_0805_2012Metric, F.Cu at (140.7, 96.5)
- added R24: 1, Resistor_SMD:R_0603_1608Metric, F.Cu at (121.8, 111.1)
- added R25: 1, Resistor_SMD:R_0603_1608Metric, F.Cu at (121.8, 113.6)
- added R26: 10k, Resistor_SMD:R_0805_2012Metric, F.Cu at (140.7, 105.3)
- added R27: 10k, Resistor_SMD:R_0805_2012Metric, F.Cu at (140.7, 108.3)
- added R28: 10m, Resistor_SMD:R_0805_2012Metric, F.Cu at (145.1, 84.7)
- added R29: 10k, Resistor_SMD:R_0805_2012Metric, F.Cu at (145.1, 87.7)
- added R30: 10m, Resistor_SMD:R_0805_2012Metric, F.Cu at (145.1, 90.6)
- added R31: 10m, Resistor_SMD:R_0805_2012Metric, F.Cu at (145.1, 93.5)
- added R32: 1, Resistor_SMD:R_0603_1608Metric, F.Cu at (125.8, 86.0)
- added R33: 1, Resistor_SMD:R_0603_1608Metric, F.Cu at (125.8, 88.5)
- added R34: 1, Resistor_SMD:R_0603_1608Metric, F.Cu at (125.8, 91.0)
- added R35: 1, Resistor_SMD:R_0603_1608Metric, F.Cu at (35.8, 21.0)
- added R36: 1, Resistor_SMD:R_0603_1608Metric, F.Cu at (125.8, 96.0)
- added R37: 1, Resistor_SMD:R_0603_1608Metric, F.Cu at (125.8, 98.5)
- added R38: 10k, Resistor_SMD:R_0805_2012Metric, F.Cu at (20.5, 21.0)
- added R39: 10k, Resistor_SMD:R_0805_2012Metric, F.Cu at (145.1, 99.5)
- added R40: 10m, Resistor_SMD:R_0805_2012Metric, F.Cu at (39.5, 22.5)
- added R41: 10k, Resistor_SMD:R_0805_2012Metric, F.Cu at (145.1, 105.3)
- added R42: 10m, Resistor_SMD:R_0805_2012Metric, F.Cu at (145.1, 108.3)
- added R43: 10m, Resistor_SMD:R_0805_2012Metric, F.Cu at (149.5, 84.7)
- added R44: 1, Resistor_SMD:R_0603_1608Metric, F.Cu at (35.3, 24.5)
- added R45: 1, Resistor_SMD:R_0603_1608Metric, F.Cu at (125.8, 103.5)
- added R46: 1, Resistor_SMD:R_0603_1608Metric, F.Cu at (125.8, 106.0)
- added R47: 1k, Resistor_SMD:R_0805_2012Metric, F.Cu at (149.5, 87.7)
- added R48: 1k, Resistor_SMD:R_0805_2012Metric, F.Cu at (149.5, 90.6)
- added R49: 1k, Resistor_SMD:R_0805_2012Metric, F.Cu at (149.5, 93.5)
- added R5: 10k, Resistor_SMD:R_0805_2012Metric, F.Cu at (210.0, 80.9)
- added R50: 10k, Resistor_SMD:R_0805_2012Metric, F.Cu at (149.5, 96.5)
- added R51: 10k, Resistor_SMD:R_0805_2012Metric, F.Cu at (149.5, 99.5)
- added R52: 10k, Resistor_SMD:R_0805_2012Metric, F.Cu at (149.5, 102.4)
- added R53: 1k, Resistor_SMD:R_0805_2012Metric, F.Cu at (149.5, 105.3)
- added R54: 1k, Resistor_SMD:R_0805_2012Metric, F.Cu at (149.5, 108.3)
- added R55: 1k, Resistor_SMD:R_0805_2012Metric, F.Cu at (153.9, 84.7)
- added R56: 10k, Resistor_SMD:R_0805_2012Metric, F.Cu at (153.9, 87.7)
- added R57: 10k, Resistor_SMD:R_0805_2012Metric, F.Cu at (153.9, 90.6)
- added R58: 10k, Resistor_SMD:R_0805_2012Metric, F.Cu at (153.9, 93.5)
- added R59: 1k, Resistor_SMD:R_0805_2012Metric, F.Cu at (153.9, 96.5)
- added R6: 3.3k, Resistor_SMD:R_0805_2012Metric, F.Cu at (213.0, 80.0)
- added R60: 1k, Resistor_SMD:R_0805_2012Metric, F.Cu at (153.9, 99.5)
- added R61: 1k, Resistor_SMD:R_0805_2012Metric, F.Cu at (153.9, 102.4)
- added R62: 10k, Resistor_SMD:R_0805_2012Metric, F.Cu at (153.9, 105.3)
- added R63: 10k, Resistor_SMD:R_0805_2012Metric, F.Cu at (153.9, 108.3)
- added R64: 10k, Resistor_SMD:R_0805_2012Metric, F.Cu at (158.3, 84.7)
- added R65: 1k, Resistor_SMD:R_0805_2012Metric, F.Cu at (158.3, 87.7)
- added R66: 1k, Resistor_SMD:R_0805_2012Metric, F.Cu at (158.3, 90.6)
- added R67: 1k, Resistor_SMD:R_0805_2012Metric, F.Cu at (158.3, 93.5)
- added R68: 10k, Resistor_SMD:R_0805_2012Metric, F.Cu at (158.3, 96.5)
- added R69: 10k, Resistor_SMD:R_0805_2012Metric, F.Cu at (158.3, 99.5)
- added R70: 10k, Resistor_SMD:R_0805_2012Metric, F.Cu at (158.3, 102.4)
- added U10: PC817, Package_DIP:DIP-4_W7.62mm_SMDSocket_SmallPads, F.Cu at (42.5, 164.9)
- added U11: PC817, Package_DIP:DIP-4_W7.62mm_SMDSocket_SmallPads, F.Cu at (42.5, 171.6)
- added U12: PC817, Package_DIP:DIP-4_W7.62mm_SMDSocket_SmallPads, F.Cu at (42.5, 178.4)
- added U13: PC817, Package_DIP:DIP-4_W7.62mm_SMDSocket_SmallPads, F.Cu at (44.1, 187.3)
- added U14: PC817, Package_DIP:DIP-4_W7.62mm_SMDSocket_SmallPads, F.Cu at (54.2, 164.9)
- added U15: PC817, Package_DIP:DIP-4_W7.62mm_SMDSocket_SmallPads, F.Cu at (54.2, 171.6)
- added U16: PC817, Package_DIP:DIP-4_W7.62mm_SMDSocket_SmallPads, F.Cu at (54.2, 178.4)
- added U17: PC817, Package_DIP:DIP-4_W7.62mm_SMDSocket_SmallPads, F.Cu at (55.8, 187.3)
- added U6: PC817, Package_DIP:DIP-4_W7.62mm_SMDSocket_SmallPads, F.Cu at (30.7, 164.9)
- added U7: PC817, Package_DIP:DIP-4_W7.62mm_SMDSocket_SmallPads, F.Cu at (30.7, 171.6)
- added U8: PC817, Package_DIP:DIP-4_W7.62mm_SMDSocket_SmallPads, F.Cu at (30.7, 178.4)
- added U9: PC817, Package_DIP:DIP-4_W7.62mm_SMDSocket_SmallPads, F.Cu at (32.4, 187.3)
- added con2: KF202, Library_footprints:con_klemnic, F.Cu at (248.7, 83.2)
- C13, C8: footprint Capacitor_SMD:C_1206_3216Metric -> Capacitor_SMD:C_0603_1608Metric
- C26: footprint Capacitor_SMD:C_1206_3216Metric -> Capacitor_Tantalum_SMD:CP_EIA-7343-31_Kemet-D_HandSolder
- C28: value 330uF -> 10nF; footprint Capacitor_Tantalum_SMD:CP_EIA-7343-31_Kemet-D_HandSolder -> Capacitor_SMD:C_0603_1608Metric
- C29: value 4.7uF -> 330uF; footprint Capacitor_SMD:C_1206_3216Metric -> Capacitor_SMD:C_0603_1608Metric
- C30: value 100nF -> 4.7uF
- C34, C36, C38: value 100nF -> 10uF
- D1: value BAS70 -> Green; footprint Diode_SMD:D_0603_1608Metric -> LED_SMD:LED_0603_1608Metric
- D3, D6: value SS54L -> BAS70
- D5: value BAS70 -> SS54L
- M_Con1, M_Con2, M_Con3, M_Con4, M_Con5, M_Con6: footprint Connector_PinHeader_2.00mm:PinHeader_1x06_P2.00mm_Vertical -> Library_footprints:KF202-7.5-6P
- R1, R3, R7, R9: footprint Resistor_SMD:R_0805_2012Metric -> Resistor_SMD:R_0603_1608Metric
- R15: value 1k -> 10k
- R16: value 1k -> 3.3k
- R2, R8: footprint Resistor_SMD:R_2512_6332Metric -> Resistor_SMD:R_0805_2012Metric
- R23: value 1k -> 1; footprint Resistor_SMD:R_0805_2012Metric -> Resistor_SMD:R_0603_1608Metric
- R4: value 1K -> 1k
- moved M_Con6 211.5 mm to (-41.8, 161.4)
- moved M_Con5 202.7 mm to (-41.8, 146.6)
- moved M_Con4 194.6 mm to (-41.8, 131.8)
- moved M_Con3 187.5 mm to (-41.8, 117.0)
- moved M_Con2 176.8 mm to (-41.8, 102.2)
- moved M_Con1 172.1 mm to (-42.0, 88.8)
- moved C38 163.9 mm to (16.5, 40.0), turned to -90 degrees
- moved C39 163.1 mm to (17.0, 43.5)
- moved C33 138.6 mm to (40.0, 37.0)
- moved I7 128.7 mm to (27.0, 22.5)
- moved DRV3 119.4 mm to (29.5, 39.0)
- moved L3 106.6 mm to (210.0, 152.0)
- moved C9 102.3 mm to (260.5, 109.0), turned to -90 degrees
- moved L2 100.6 mm to (210.0, 105.0)
- moved C21 100.4 mm to (260.5, 121.2), turned to -90 degrees
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Connections:
- C13 pad 1: VBUS(PA9) -> +3v3
- C2 pad 2: Net-(D1-K) -> Net-(D2-K)
- C20 pad 2: Net-(D2-K) -> Net-(D3-K)
- C25 pad 1: VBUS(PA9) -> +3v3
- C28 pad 1: +5v -> Net-(U5-BOOT)
- C28 pad 2: GND -> Net-(D6-K)
- C29 pad 1: GND -> +5v
- C29 pad 2: Net-(I3-IN-) -> GND
- C30 pad 2: Net-(DRV1-CCP) -> Net-(JP3-A)
- C31 pad 1: GND -> Net-(DRV1-CCP)
- C31 pad 2: Net-(DRV2-CCP) -> GND
- C32 pad 1: GND -> Net-(DRV2-CCP)
- C32 pad 2: Net-(DRV3-CCP) -> GND
- C33 pad 1: GND -> Net-(DRV3-CCP)
- C33 pad 2: INA1 -> GND
- C34 pad 1: GND -> INA2
- C34 pad 2: INA1 -> GND
- C35 pad 1: GND -> INA2
- C35 pad 2: INA1 -> GND
- C36 pad 1: GND -> INA3
- C36 pad 2: Net-(DRV4-CCP) -> GND
- C37 pad 1: GND -> INA3
- C37 pad 2: Net-(DRV5-CCP) -> GND
- C38 pad 1: GND -> INA1
- C38 pad 2: Net-(DRV6-CCP) -> GND
- C39 pad 1: GND -> INA1
- C39 pad 2: INA1 -> GND
- C40 pad 1: GND -> Net-(DRV4-CCP)
- C40 pad 2: INA1 -> GND
- C41 pad 1: GND -> Net-(DRV5-CCP)
- C41 pad 2: INA1 -> GND
- C5 pad 1: VBUS(PA9) -> Net-(U1-VOUT)
- C6 pad 1: VBUS(PA9) -> Net-(U1-VOUT)
- D1 pad 1: Net-(D1-K) -> GND
- D1 pad 2: GND -> Net-(D1-A)
- D10 pad 1: INA1 -> +14.4v
- D10 pad 2: CONN_M5_2 -> CONN_M2_1
- D11 pad 1: INA1 -> +14.4v
- D11 pad 2: CONN_M5_1 -> CONN_M3_2
- D12 pad 1: INA1 -> +14.4v
- D12 pad 2: CONN_M6_2 -> CONN_M3_1
- D13 pad 1: INA1 -> +14.4v
- D13 pad 2: CONN_M6_1 -> CONN_M4_2
- D14 pad 1: INA1 -> +14.4v
- D14 pad 2: CONN_M1_2 -> CONN_M4_1
- D15 pad 1: INA1 -> +14.4v
- D15 pad 2: CONN_M1_1 -> CONN_M5_2
- D16 pad 1: INA1 -> +14.4v
- D16 pad 2: CONN_M2_2 -> CONN_M5_1
- D17 pad 1: INA1 -> +14.4v
- D17 pad 2: CONN_M2_1 -> CONN_M6_2
- D18 pad 1: CONN_M3_2 -> +14.4v
- D18 pad 2: GND -> CONN_M6_1
- D19 pad 1: CONN_M3_1 -> CONN_M1_2
- D20 pad 1: CONN_M4_2 -> CONN_M1_1
- D21 pad 1: CONN_M4_1 -> CONN_M2_2
- D22 pad 1: CONN_M5_2 -> CONN_M2_1
- D23 pad 1: CONN_M5_1 -> CONN_M3_2
- D24 pad 1: CONN_M6_2 -> CONN_M3_1
- D25 pad 1: CONN_M6_1 -> CONN_M4_2
- D26 pad 1: CONN_M1_2 -> CONN_M4_1
- D27 pad 1: CONN_M1_1 -> CONN_M5_2
- D28 pad 1: CONN_M2_2 -> CONN_M5_1
- D29 pad 1: CONN_M2_1 -> CONN_M6_2
- D3 pad 1: INA1 -> Net-(D3-K)
- D3 pad 2: Net-(D3-A) -> GND
- D4 pad 1: INA1 -> +14.4v
- D5 pad 1: Net-(D5-K) -> +14.4v
- D5 pad 2: GND -> Net-(D5-A)
- D6 pad 1: INA1 -> Net-(D6-K)
- D6 pad 2: CONN_M3_2 -> GND
- D7 pad 1: INA1 -> +14.4v
- D7 pad 2: CONN_M3_1 -> CONN_M1_2
- D8 pad 1: INA1 -> +14.4v
- D8 pad 2: CONN_M4_2 -> CONN_M1_1
- D9 pad 1: INA1 -> +14.4v
- D9 pad 2: CONN_M4_1 -> CONN_M2_2
- DRV1 pad 13: +5v -> D2_2
- DRV1 pad 16: INA1 -> INA2
- DRV1 pad 2: Net-(DRV1-FS#) -> FS2
- DRV1 pad 4: INA1 -> INA2
- DRV1 pad 5: INA1 -> INA2
- DRV2 pad 13: +5v -> D2_3
- DRV2 pad 16: INA1 -> INA3
- DRV2 pad 2: Net-(DRV2-FS#) -> FS3
- DRV2 pad 4: INA1 -> INA3
- DRV2 pad 5: INA1 -> INA3
- DRV3 pad 13: +5v -> D2_1
- DRV3 pad 2: Net-(DRV3-FS#) -> FS1
- DRV4 pad 13: +5v -> D2_5
- DRV4 pad 16: INA1 -> INA5
- DRV4 pad 2: Net-(DRV4-FS#) -> FS5
- DRV4 pad 4: INA1 -> INA5
- DRV4 pad 5: INA1 -> INA5
- DRV5 pad 13: +5v -> D2_6
- DRV5 pad 16: INA1 -> INA6
- DRV5 pad 2: Net-(DRV5-FS#) -> FS6
- DRV5 pad 4: INA1 -> INA6
- DRV5 pad 5: INA1 -> INA6
- DRV6 pad 13: +5v -> D2_4
- DRV6 pad 16: INA1 -> INA4
- DRV6 pad 2: Net-(DRV6-FS#) -> FS4
- DRV6 pad 4: INA1 -> INA4
- DRV6 pad 5: INA1 -> INA4
- I2 pad 1: unconnected-(I2-A1-Pad1) -> GND
- I2 pad 2: unconnected-(I2-A0-Pad2) -> +5v
- I2 pad 3: unconnected-(I2-Alert-Pad3) -> Net-(I2-Alert)
- I2 pad 4: unconnected-(I2-SDA-Pad4) -> SDA_INA
- I2 pad 5: unconnected-(I2-SCL-Pad5) -> SCL_INA
- I3 pad 1: unconnected-(I3-A1-Pad1) -> +5v
- I3 pad 10: INA1 -> Net-(I3-IN+)
- I3 pad 2: unconnected-(I3-A0-Pad2) -> GND
- I3 pad 3: unconnected-(I3-Alert-Pad3) -> Net-(I3-Alert)
- I3 pad 4: unconnected-(I3-SDA-Pad4) -> SDA_INA
- I3 pad 5: unconnected-(I3-SCL-Pad5) -> SCL_INA
- I4 pad 1: unconnected-(I4-A1-Pad1) -> +5v
- I4 pad 10: INA1 -> Net-(I4-IN+)
- I4 pad 2: unconnected-(I4-A0-Pad2) -> SCL_INA
- I4 pad 3: unconnected-(I4-Alert-Pad3) -> D2_5
- I4 pad 4: unconnected-(I4-SDA-Pad4) -> SDA_INA
- I4 pad 5: unconnected-(I4-SCL-Pad5) -> SCL_INA
- I4 pad 8: INA1 -> Net-(I4-IN-)
- I4 pad 9: INA1 -> Net-(I4-IN-)
- I5 pad 1: unconnected-(I5-A1-Pad1) -> GND
- I5 pad 10: INA1 -> Net-(I5-IN+)
- I5 pad 2: unconnected-(I5-A0-Pad2) -> SCL_INA
- I5 pad 3: unconnected-(I5-Alert-Pad3) -> D2_3
- I5 pad 4: unconnected-(I5-SDA-Pad4) -> SDA_INA
- I5 pad 5: unconnected-(I5-SCL-Pad5) -> SCL_INA
- I5 pad 8: INA1 -> Net-(I5-IN-)
- I5 pad 9: INA1 -> Net-(I5-IN-)
- I6 pad 1: unconnected-(I6-A1-Pad1) -> GND
- I6 pad 10: INA1 -> Net-(I6-IN+)
- I6 pad 2: unconnected-(I6-A0-Pad2) -> SDA_INA
- I6 pad 3: unconnected-(I6-Alert-Pad3) -> D2_2
- I6 pad 4: unconnected-(I6-SDA-Pad4) -> SDA_INA
- I6 pad 5: unconnected-(I6-SCL-Pad5) -> SCL_INA
- I6 pad 8: INA1 -> Net-(I6-IN-)
- I6 pad 9: INA1 -> Net-(I6-IN-)
- I7 pad 1: unconnected-(I7-A1-Pad1) -> +5v
- I7 pad 10: INA1 -> Net-(I7-IN+)
- I7 pad 2: unconnected-(I7-A0-Pad2) -> +5v
- I7 pad 3: unconnected-(I7-Alert-Pad3) -> D2_1
- I7 pad 4: unconnected-(I7-SDA-Pad4) -> SDA_INA
- I7 pad 5: unconnected-(I7-SCL-Pad5) -> SCL_INA
- I7 pad 8: INA1 -> Net-(I7-IN-)
- I7 pad 9: INA1 -> Net-(I7-IN-)
- I8 pad 1: unconnected-(I8-A1-Pad1) -> SDA_INA
- I8 pad 10: INA1 -> Net-(I8-IN+)
- I8 pad 2: unconnected-(I8-A0-Pad2) -> +5v
- I8 pad 3: unconnected-(I8-Alert-Pad3) -> D2_6
- I8 pad 4: unconnected-(I8-SDA-Pad4) -> SDA_INA
- I8 pad 5: unconnected-(I8-SCL-Pad5) -> SCL_INA
- I8 pad 8: INA1 -> Net-(I8-IN-)
- I8 pad 9: INA1 -> Net-(I8-IN-)
- I9 pad 1: unconnected-(I9-A1-Pad1) -> +5v
- I9 pad 10: INA1 -> Net-(I9-IN+)
- I9 pad 2: unconnected-(I9-A0-Pad2) -> SDA_INA
- I9 pad 3: unconnected-(I9-Alert-Pad3) -> D2_4
- I9 pad 4: unconnected-(I9-SDA-Pad4) -> SDA_INA
- I9 pad 5: unconnected-(I9-SCL-Pad5) -> SCL_INA
- I9 pad 8: INA1 -> Net-(I9-IN-)
- I9 pad 9: INA1 -> Net-(I9-IN-)
- L1 pad 1: +5v -> Net-(D2-K)
- L1 pad 2: Net-(D1-K) -> +5v
- L2 pad 1: VBUS(PA9) -> Net-(D3-K)
- L2 pad 2: Net-(D2-K) -> +3v3
- L3 pad 1: +5v -> Net-(D6-K)
- L3 pad 2: Net-(D5-K) -> +5v
- M_Con1 pad 3: INA1 -> Net-(JP4-C)
- M_Con2 pad 3: INA1 -> Net-(JP5-C)
- M_Con3 pad 3: INA1 -> Net-(JP6-C)
- M_Con4 pad 3: INA1 -> Net-(JP7-C)
- M_Con5 pad 3: INA1 -> Net-(JP8-C)
- M_Con6 pad 3: INA1 -> Net-(JP9-C)
- R1 pad 2: INA1 -> +14.4v
- R15 pad 2: Net-(DRV1-FS#) -> Net-(U5-VSENSE)
- R16 pad 1: +5v -> Net-(U5-VSENSE)
- R16 pad 2: Net-(DRV2-FS#) -> GND
- R17 pad 2: Net-(DRV3-FS#) -> FS2
- R2 pad 1: INA1 -> +14.4v
- R21 pad 2: Net-(DRV4-FS#) -> FS6
- R22 pad 2: Net-(DRV5-FS#) -> FS4
- R23 pad 1: +5v -> Net-(I4-IN+)
- R23 pad 2: Net-(DRV6-FS#) -> +14.4v
- R4 pad 1: Net-(LED1-+) -> +5v
- R4 pad 2: +5v -> Net-(D1-A)
- R7 pad 2: INA1 -> +14.4v
- R8 pad 1: INA1 -> +14.4v
- U1 pad 4: VBUS(PA9) -> Net-(U1-VOUT)
- U1 pad 7: (no net) -> unconnected-(U1-EXP-Pad7)
- U2 pad 8: Net-(D1-K) -> Net-(D2-K)
- U3 pad 1: VBUS(PA9) -> +3v3
- U4 pad 5: unconnected-(U4-ENA-Pad5) -> ENA_U4
- U4 pad 8: Net-(D2-K) -> Net-(D3-K)
- U5 pad 5: unconnected-(U5-ENA-Pad5) -> ENA_U5
- U5 pad 7: Net-(I3-IN-) -> Net-(JP3-A)
- U5 pad 8: Net-(D5-K) -> Net-(D6-K)
Other:
- board outline removed

Commit message: Add files via upload
Parts:
- moved M_Con4 396.9 mm to (343.4, 228.0), turned to -90 degrees
- moved M_Con3 390.5 mm to (343.3, 182.2), turned to -90 degrees
- moved M_Con1 317.1 mm to (270.3, 34.2), turned to -90 degrees
- moved M_Con2 313.2 mm to (270.8, 80.7), turned to -90 degrees
- moved M_Con5 304.3 mm to (251.2, 228.8), turned to 180 degrees
- moved U9 263.9 mm to (194.5, -21.0)
- moved U6 261.0 mm to (195.5, -37.5)
- moved M_Con6 242.6 mm to (191.8, 227.3), turned to 180 degrees
- moved U12 242.4 mm to (154.5, -36.5)
- moved U8 228.1 mm to (107.8, -36.3)
- moved U17 224.0 mm to (196.0, 12.5)
- moved U14 219.5 mm to (195.5, -3.00)
- moved U15 216.6 mm to (155.0, -20.0)
- moved J2 213.8 mm to (87.8, -38.8)
- moved U7 213.8 mm to (155.5, -2.00)
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Connections:
- C13 pad 1: +3v3 -> +3,3v
- C25 pad 1: +3v3 -> +3,3v
- L2 pad 2: +3v3 -> +3,3v
- R10 pad 1: +3v3 -> +3,3v
- U2 pad 9: (no net) -> GND
- U3 pad 1: +3v3 -> +3,3v
- U4 pad 9: (no net) -> GND
- U5 pad 9: (no net) -> GND
Routing:
- net +14.4v: track 0.30 -> 124.2 mm
- net GND: track 0.00 -> 36.5 mm
- net +5v: track 0.00 -> 25.9 mm
- net Net-(D2-K): track 0.00 -> 16.9 mm
- net Net-(D5-A): track 0.00 -> 10.7 mm
- net Net-(D4-A): track 0.00 -> 6.71 mm
- net Net-(U2-BOOT): track 0.00 -> 4.06 mm
- net Net-(JP1-A): track 0.00 -> 3.71 mm
- net Net-(I2-IN-): track 0.00 -> 2.10 mm
- net Net-(I2-IN+): track 0.00 -> 2.08 mm
- net Net-(I6-IN-): track 0.00 -> 2.02 mm
- net Net-(I7-IN-): track 0.00 -> 1.94 mm
- net Net-(I1-IN+): track 0.00 -> 1.92 mm
- net Net-(I3-IN+): track 0.00 -> 1.92 mm
- net Net-(I9-IN+): track 0.00 -> 1.91 mm
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
Commit message: Add files via upload
Parts:
- C26: footprint Capacitor_Tantalum_SMD:CP_EIA-7343-31_Kemet-D_HandSolder -> Capacitor_SMD:C_0603_1608Metric
- C29: footprint Capacitor_SMD:C_0603_1608Metric -> Capacitor_Tantalum_SMD:CP_EIA-7343-31_Kemet-D_HandSolder
- moved R16 108.4 mm to (248.8, 132.5), turned to 0 degrees
- moved U5 97.0 mm to (241.3, 126.0)
- moved Con1 96.5 mm to (200.3, 143.8), turned to 0 degrees
- moved C3 96.4 mm to (201.4, 136.4), turned to 180 degrees
- moved C30 96.3 mm to (245.9, 125.0)
- moved U1 96.3 mm to (201.0, 140.8), turned to -90 degrees
- moved C13 96.1 mm to (205.0, 141.6), turned to 0 degrees
- moved U3 92.6 mm to (206.0, 137.0), turned to 90 degrees
- moved C4 92.6 mm to (201.4, 138.0), turned to 180 degrees
- moved C6 92.5 mm to (197.5, 143.6), turned to 180 degrees
- moved C5 92.0 mm to (198.3, 141.2), turned to 90 degrees
- moved C14 91.9 mm to (204.9, 132.5), turned to 0 degrees
- moved R4 91.2 mm to (201.6, 133.0)
- moved C28 90.1 mm to (236.8, 127.2), turned to 90 degrees
- moved D1 88.9 mm to (201.4, 134.8), turned to 0 degrees
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Connections:
- R10 pad 2: Net-(U4-VSENSE) -> GND
- R11 pad 1: Net-(U4-VSENSE) -> GND
- R15 pad 2: Net-(U5-VSENSE) -> GND
- R16 pad 1: Net-(U5-VSENSE) -> GND
- U4 pad 4: Net-(U4-VSENSE) -> GND
- U5 pad 4: Net-(U5-VSENSE) -> GND
Routing:
- net GND: track 36.5 -> 153.7 mm
- net +5v: track 25.9 -> 71.7 mm
- net Net-(D3-K): track 0.00 -> 21.4 mm
- net Net-(D6-K): track 0.00 -> 20.6 mm
- net +3,3v: track 0.00 -> 11.5 mm
- net Net-(JP3-A): track 1.71 -> 12.2 mm
- net Net-(JP2-A): track 1.81 -> 11.8 mm
- net Net-(JP1-A): track 3.71 -> 11.8 mm
- net +14.4v: track 124.2 -> 131.6 mm
- net Net-(U1-VOUT): track 0.00 -> 5.76 mm
- net Net-(I2-IN-): track 2.10 -> 7.84 mm
- net Net-(I1-IN-): track 1.91 -> 7.62 mm
- net Net-(I1-IN+): track 1.92 -> 7.60 mm
- net Net-(I3-IN+): track 1.92 -> 7.57 mm
- net Net-(D2-K): track 16.9 -> 22.5 mm
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
Commit message: Add files via upload
Parts:
- removed C13: 4.7uF, Capacitor_SMD:C_0603_1608Metric
- removed C14: 0.1uF, Capacitor_SMD:C_0603_1608Metric
- removed U3: KF33BD-TR, Package_SO:SOIC-8_3.9x4.9mm_P1.27mm
- DRV1, DRV2, DRV3, DRV4, DRV5, DRV6: footprint Package_SO:HSOP-20-1EP_11.0x15.9mm_P1.27mm_SlugDown -> Package_SO:HSOP-20-1EP_11.0x15.9mm_P1.27mm_SlugUp
- moved D18 173.8 mm to (18.1, 130.2)
- moved D30 173.8 mm to (19.7, 130.2)
- moved D17 159.0 mm to (38.1, 130.0), turned to 180 degrees
- moved D29 157.0 mm to (38.1, 128.4), turned to 0 degrees
- moved R42 153.0 mm to (28.7, 137.9)
- moved R45 152.6 mm to (31.2, 137.3), turned to -90 degrees
- moved R36 152.6 mm to (26.2, 137.2), turned to -90 degrees
- moved C53 151.9 mm to (28.7, 136.1)
- moved D16 151.7 mm to (48.4, 131.8)
- moved D28 151.7 mm to (50.0, 131.8)
- moved I8 146.6 mm to (28.8, 116.9), turned to 180 degrees
- moved R49 145.7 mm to (179.2, 82.6), turned to 180 degrees
- moved J2 138.4 mm to (161.2, 78.6), turned to 180 degrees
- moved D15 136.9 mm to (68.4, 131.0), turned to 180 degrees
- moved C38 136.8 mm to (144.9, 87.2), turned to 0 degrees
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Routing:
- net GND: track 153.7 -> 679.9 mm, vias 0 -> 53
- net +5v: track 71.7 -> 380.6 mm, vias 0 -> 26
- net +14.4v: track 131.6 -> 29.4 mm
- net INA2: track 1.72 -> 80.7 mm, vias 0 -> 3
- net INA3: track 1.70 -> 79.9 mm, vias 0 -> 3
- net INA5: track 1.71 -> 65.6 mm, vias 0 -> 3
- net INA4: track 1.71 -> 64.3 mm, vias 0 -> 3
- net INA6: track 1.70 -> 63.5 mm, vias 0 -> 3
- net INA1: track 1.71 -> 53.1 mm, vias 0 -> 3
- net FS1: track 0.00 -> 32.6 mm
- net IN2_M1: track 0.00 -> 31.5 mm
- net D2_6: track 0.00 -> 25.2 mm
- net D2_5: track 0.00 -> 25.1 mm
- net D2_4: track 0.00 -> 24.6 mm
- net D2_2: track 0.00 -> 24.0 mm
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
Commit message: Add files via upload
Parts:
- moved M_Con3 299.3 mm to (86.2, 28.9), turned to 180 degrees
- moved JP6 290.5 mm to (80.4, 43.8), turned to 0 degrees
- moved M_Con4 288.1 mm to (64.2, 156.5), turned to 0 degrees
- moved JP7 278.8 mm to (70.6, 141.6), turned to 180 degrees
- moved R36 171.6 mm to (197.2, 122.2), turned to 90 degrees
- moved R42 166.9 mm to (194.7, 121.0), turned to 180 degrees
- moved C53 166.5 mm to (194.7, 123.3), turned to 180 degrees
- moved C43 166.1 mm to (183.9, 136.7)
- moved C44 166.1 mm to (185.5, 136.7)
- moved D17 166.1 mm to (203.9, 139.6)
- moved D18 166.1 mm to (183.9, 139.8)
- moved D30 166.1 mm to (185.5, 139.8)
- moved DRV5 166.1 mm to (194.4, 136.5)
- moved I8 166.1 mm to (194.6, 126.5), turned to 0 degrees
- moved R21 166.1 mm to (184.6, 132.2)
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Routing:
- net GND: track 679.9 -> 1521.0 mm, vias 53 -> 51
- net +14.4v: track 29.4 -> 773.8 mm, vias 0 -> 29
- net +5v: track 380.6 -> 1067.9 mm, vias 26 -> 43
- net +3,3v: track 9.33 -> 511.9 mm, vias 0 -> 11
- net SCL_INA: track 6.47 -> 493.1 mm, vias 0 -> 10
- net SDA_INA: track 10.3 -> 434.3 mm
- net IN2_M3: track 0.00 -> 56.3 mm, vias 0 -> 2
- net IN2_M5: track 0.00 -> 55.8 mm, vias 0 -> 2
- net IN2_M2: track 0.00 -> 55.7 mm, vias 0 -> 2
- net IN2_M4: track 0.00 -> 54.1 mm, vias 0 -> 2
- net IN2_M6: track 0.00 -> 52.0 mm, vias 0 -> 2
- net IN2_M1: track 31.5 -> 56.0 mm, vias 0 -> 2
- net CONN_M4_2: track 5.32 -> 29.6 mm
- net CONN_M6_2: track 5.28 -> 28.4 mm
- net CONN_M2_2: track 5.16 -> 27.9 mm
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
Commit message: Add files via upload
Parts:
- removed C43, C45, C47: 10uF, Capacitor_SMD:C_0603_1608Metric
- removed C44, C46, C48, C49, C50, C51, C52, C53, C54: 100nF, Capacitor_SMD:C_0603_1608Metric
- removed U17: PC817, Package_DIP:DIP-4_W7.62mm_SMDSocket_SmallPads
- added C13: 100nF, Capacitor_SMD:C_0603_1608Metric, F.Cu at (202.4, 92.3)
- added C14: 100nF, Capacitor_SMD:C_0603_1608Metric, F.Cu at (195.5, 106.0)
- added REF**: Arduino_UNO_R2, Module:Arduino_UNO_R2, F.Cu at (353.0, 55.8)
- added U3: TPS5450, Package_SO:SOIC-8-1EP_3.9x4.9mm_P1.27mm_EP2.29x3mm, F.Cu at (131.9, 97.6)
- C10, C16: value 100nF -> 10nF
- C11, C17: value 100nF -> 330uF; footprint Capacitor_SMD:C_0603_1608Metric -> Capacitor_Tantalum_SMD:CP_EIA-7343-31_Kemet-D_HandSolder
- C12, C18: value 100nF -> 4.7uF
- C20, C28: value 10nF -> 100nF
- C22, C24, C31, C33, C35: value 100nF -> 10uF
- C25, C29: value 330uF -> 100nF; footprint Capacitor_Tantalum_SMD:CP_EIA-7343-31_Kemet-D_HandSolder -> Capacitor_SMD:C_0603_1608Metric
- C26: value 4.7uF -> 10uF
- C30: value 4.7uF -> 100nF
- C34, C36, C38: value 10uF -> 100nF
- Con2: renamed from con2; value KF202 -> DG125-5.0-02P-14-00A(H); footprint Library_footprints:con_klemnic -> TerminalBlock_Phoenix:TerminalBlock_Phoenix_MKDS-1,5-2_1x02_P5.00mm_Horizontal
- D4, D5: footprint Diode_SMD:D_0603_1608Metric -> Diode_SMD:D_SMC
- J1, J2, J3, J4, J5, J6: footprint Connector_PinHeader_1.00mm:PinHeader_1x05_P1.00mm_Vertical -> Connector_PinHeader_2.54mm:PinHeader_1x05_P2.54mm_Vertical
- U5: value TPS5450 -> PC817; footprint Package_SO:SOIC-8-1EP_3.9x4.9mm_P1.27mm_EP2.29x3mm -> Package_DIP:DIP-4_W7.62mm_SMDSocket_SmallPads
- con3: renamed from Con3; value DG125-5.0-02P-14-00A(H) -> KF202; footprint TerminalBlock_Phoenix:TerminalBlock_Phoenix_MKDS-1,5-2_1x02_P5.00mm_Horizontal -> Library_footprints:con_klemnic
- moved C24 167.0 mm to (113.8, 78.1)
- moved C32 155.2 mm to (194.8, 126.7), turned to 0 degrees
- moved C19 153.7 mm to (128.2, 69.3)
- moved C10 153.5 mm to (126.9, 98.8), turned to 90 degrees
- moved C9 146.7 mm to (136.9, 91.8)
- moved C22 141.4 mm to (146.5, 75.0), turned to 180 degrees
- moved C23 139.6 mm to (146.5, 73.4), turned to 180 degrees
- moved C12 139.1 mm to (136.5, 96.6), turned to 90 degrees
- moved C11 136.9 mm to (140.7, 109.4), turned to 90 degrees
- moved C16 134.7 mm to (148.9, 98.6), turned to 90 degrees
- moved U16 120.7 mm to (184.7, 134.1)
- moved C18 120.6 mm to (158.4, 96.5), turned to 90 degrees
- moved U13 120.6 mm to (178.8, 134.1)
- moved C21 118.7 mm to (175.9, 69.5)
- moved C17 117.5 mm to (162.7, 109.4), turned to 90 degrees
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Connections:
- C10 pad 1: VDD -> Net-(U3-BOOT)
- C10 pad 2: GND -> Net-(D3-K)
- C11 pad 1: VDD -> +3,3v
- C12 pad 1: VDD -> GND
- C12 pad 2: GND -> Net-(JP2-A)
- C15 pad 1: Net-(I2-IN+) -> Net-(I3-IN+)
- C15 pad 2: Net-(I2-IN-) -> Net-(I3-IN-)
- C16 pad 1: VDD -> Net-(U4-BOOT)
- C16 pad 2: GND -> Net-(D6-K)
- C17 pad 1: VDD -> +5v
- C18 pad 1: VDD -> GND
- C18 pad 2: GND -> Net-(JP3-A)
- C19 pad 1: VDD -> Net-(DRV1-CCP)
- C20 pad 1: Net-(U4-BOOT) -> Net-(DRV2-CCP)
- C20 pad 2: Net-(D3-K) -> GND
- C21 pad 1: VDD -> Net-(DRV3-CCP)
- C22 pad 1: VDD -> INA2
- C23 pad 1: VDD -> INA2
- C24 pad 1: VDD -> INA3
- C25 pad 1: +3,3v -> INA3
- C26 pad 1: GND -> INA1
- C26 pad 2: Net-(JP2-A) -> GND
- C27 pad 1: Net-(I3-IN+) -> INA1
- C27 pad 2: Net-(I3-IN-) -> GND
- C28 pad 1: Net-(U5-BOOT) -> Net-(DRV4-CCP)
- C28 pad 2: Net-(D6-K) -> GND
- C29 pad 1: +5v -> Net-(DRV5-CCP)
- C30 pad 1: GND -> Net-(DRV6-CCP)
- C30 pad 2: Net-(JP3-A) -> GND
- C31 pad 1: Net-(DRV1-CCP) -> INA6
- C32 pad 1: Net-(DRV2-CCP) -> INA6
- C33 pad 1: Net-(DRV3-CCP) -> INA5
- C34 pad 1: INA2 -> INA5
- C35 pad 1: INA2 -> INA4
- C36 pad 1: INA3 -> INA4
- C37 pad 1: INA3 -> Net-(I4-IN+)
- C37 pad 2: GND -> Net-(I4-IN-)
- C38 pad 1: INA1 -> Net-(I5-IN+)
- C38 pad 2: GND -> Net-(I5-IN-)
- C39 pad 1: INA1 -> Net-(I6-IN+)
- C39 pad 2: GND -> Net-(I6-IN-)
- C40 pad 1: Net-(DRV4-CCP) -> Net-(I7-IN+)
- C40 pad 2: GND -> Net-(I7-IN-)
- C41 pad 1: Net-(DRV5-CCP) -> Net-(I8-IN+)
- C41 pad 2: GND -> Net-(I8-IN-)
- C42 pad 1: Net-(DRV6-CCP) -> Net-(I9-IN+)
- C42 pad 2: GND -> Net-(I9-IN-)
- C9 pad 1: VDD -> Net-(I2-IN+)
- C9 pad 2: GND -> Net-(I2-IN-)
- Con2 pad 1: Net-(D5-A) -> +14.4v
- D4 pad 1: +14.4v -> Net-(D4-K)
- D4 pad 2: Net-(D4-A) -> +14.4v
- D5 pad 2: Net-(D5-A) -> GND
- U10 pad 1: Net-(R54-Pad2) -> Net-(R55-Pad2)
- U10 pad 3: ENC_B_M5_mk -> ENC_B_M1_mk
- U11 pad 1: Net-(R55-Pad2) -> Net-(R59-Pad2)
- U11 pad 3: ENC_B_M1_mk -> ENC_A_M2_mk
- U12 pad 1: Net-(R59-Pad2) -> Net-(R60-Pad2)
- U12 pad 3: ENC_A_M2_mk -> ENC_A_M4_mk
- U13 pad 1: Net-(R60-Pad2) -> Net-(R61-Pad2)
- U13 pad 3: ENC_A_M4_mk -> ENC_A_M6_mk
- U14 pad 1: Net-(R61-Pad2) -> Net-(R65-Pad2)
- U14 pad 3: ENC_A_M6_mk -> ENC_B_M2_mk
- U15 pad 1: Net-(R65-Pad2) -> Net-(R66-Pad2)
- U15 pad 3: ENC_B_M2_mk -> ENC_B_M4_mk
- U16 pad 1: Net-(R66-Pad2) -> Net-(R67-Pad2)
- U16 pad 3: ENC_B_M4_mk -> ENC_B_M6_mk
- U4 pad 5: ENA_U4 -> ENA_U5
- U4 pad 7: Net-(JP2-A) -> Net-(JP3-A)
- U4 pad 8: Net-(D3-K) -> Net-(D6-K)
- U5 pad 1: Net-(U5-BOOT) -> Net-(R47-Pad2)
- U5 pad 2: unconnected-(U5-NC-Pad2) -> GND
- U5 pad 3: unconnected-(U5-NC-Pad3) -> ENC_A_M3_mk
- U5 pad 4: GND -> +5v
- U6 pad 1: Net-(R47-Pad2) -> Net-(R48-Pad2)
- U6 pad 3: ENC_A_M3_mk -> ENC_A_M5_mk
- U7 pad 1: Net-(R48-Pad2) -> Net-(R49-Pad2)
- U7 pad 3: ENC_A_M5_mk -> ENC_A_M1_mk
- U8 pad 1: Net-(R49-Pad2) -> Net-(R53-Pad2)
- U8 pad 3: ENC_A_M1_mk -> ENC_B_M3_mk
- U9 pad 1: Net-(R53-Pad2) -> Net-(R54-Pad2)
- U9 pad 3: ENC_B_M3_mk -> ENC_B_M5_mk
- con3 pad 1: Net-(D4-A) -> Net-(D4-K)
Routing:
- net +5v: track 1067.9 -> 93.6 mm, vias 43 -> 5
- net GND: track 1521.0 -> 2029.1 mm, vias 51 -> 20
- net +3,3v: track 511.9 -> 29.2 mm, vias 11 -> 2
- net SCL_INA: track 493.1 -> 297.5 mm, vias 10 -> 11
- net SDA_INA: track 434.3 -> 283.1 mm, vias 0 -> 13
- net +14.4v: track 773.8 -> 629.5 mm, vias 29 -> 0
- net INA1: track 63.6 -> 0.00 mm, vias 3 -> 0
- net INA2: track 62.6 -> 0.00 mm, vias 3 -> 0
- net IN2_M1: track 56.0 -> 0.00 mm, vias 2 -> 0
- net IN2_M2: track 55.7 -> 0.00 mm, vias 2 -> 0
- net D2_1: track 24.0 -> 0.00 mm
- net D2_2: track 23.5 -> 0.00 mm
- net CONN_M2_2: track 27.9 -> 6.04 mm
- net IN1_M2: track 20.7 -> 0.00 mm
- net CONN_M1_2: track 26.7 -> 6.04 mm
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
Commit message: Add files via upload
Parts:
- moved REF** 186.2 mm to (168.7, 82.1)
- moved J6 10.2 mm to (162.8, 75.4), turned to -90 degrees
- moved J2 10.2 mm to (210.8, 75.4), turned to -90 degrees
- moved C19 0.34 mm to (128.2, 69.6)
- moved C21 0.32 mm to (175.9, 69.8)
- moved Con4 0.20 mm to (164.6, 82.5)
Routing:
- net +5v: track 93.6 -> 960.5 mm, vias 5 -> 52
- net +3,3v: track 29.2 -> 459.6 mm, vias 2 -> 10
- net INA1: track 0.00 -> 59.8 mm, vias 0 -> 2
- net INA2: track 0.00 -> 58.1 mm, vias 0 -> 2
- net IN2_M1: track 0.00 -> 40.4 mm, vias 0 -> 2
- net IN2_M2: track 0.00 -> 39.4 mm, vias 0 -> 2
- net D2_2: track 0.00 -> 36.9 mm, vias 0 -> 2
- net D2_1: track 0.00 -> 36.6 mm, vias 0 -> 2
- net SDA_INA: track 283.1 -> 318.1 mm, vias 13 -> 28
- net CONN_M1_1: track 6.04 -> 31.4 mm, vias 0 -> 1
- net IN1_M2: track 0.00 -> 24.0 mm, vias 0 -> 2
- net IN1_M1: track 0.00 -> 23.8 mm, vias 0 -> 2
- net CONN_M2_2: track 6.04 -> 29.8 mm, vias 0 -> 1
- net FS2: track 0.00 -> 22.5 mm, vias 0 -> 2
- net CONN_M2_1: track 6.04 -> 27.8 mm, vias 0 -> 1
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
Commit message: Add files via upload
Parts:
- removed REF**: Arduino_UNO_R2, Module:Arduino_UNO_R2
- con1: renamed from Con1; footprint Connector_PinHeader_1.00mm:PinHeader_1x02_P1.00mm_Vertical -> Connector_PinHeader_1.00mm:PinHeader_1x03_P1.00mm_Vertical
- moved con1 2.92 mm to (194.5, 111.1)
Connections:
- con1 pad 1: Net-(U1-VOUT) -> GND
- con1 pad 2: GND -> +5v
Routing:
- net +5v: track 960.5 -> 975.3 mm
- net GND: track 2031.9 -> 2035.9 mm
- net Net-(U1-VOUT): track 9.71 -> 11.1 mm
