File: plat_power.kicad_pcb (KiCad board)
At the start: 2 copper layers, 201 parts, among them Con2 DG125-5.0-02P-14-00A(H), J1 Conn_01x05_Pin, J2 Conn_01x05_Pin, J3 Conn_01x05_Pin, J4 Conn_01x05_Pin, J5 Conn_01x05_Pin, J6 Conn_01x05_Pin, U1 LD39050PU33R, U10 PC817, U11 PC817, U12 PC817, U13 PC817, U14 PC817, U15 PC817, U16 PC817, U2 TPS5450, U3 TPS5450, U4 TPS5450, U5 PC817, U6 PC817, U7 PC817, U8 PC817, U9 PC817, con3 KF202

Commit message: Add files via upload
Parts:
- Con4: footprint Connector_PinHeader_1.00mm:PinHeader_1x02_P1.00mm_Vertical -> Connector_PinHeader_2.54mm:PinHeader_1x02_P2.54mm_Vertical
- con1: footprint Connector_PinHeader_1.00mm:PinHeader_1x03_P1.00mm_Vertical -> Connector_PinHeader_2.54mm:PinHeader_1x03_P2.54mm_Vertical
- moved con1 5.37 mm to (199.2, 113.7), turned to -90 degrees
- moved Con2 4.95 mm to (209.0, 108.7), turned to 90 degrees
- moved C14 0.40 mm to (195.5, 105.6), turned to 90 degrees
- moved D5 0.40 mm to (199.7, 105.6), turned to 90 degrees
Routing:
- net +14.4v: track 629.5 -> 636.2 mm
- net GND: track 2035.9 -> 2034.0 mm
- net +5v: track 975.3 -> 977.0 mm
- net SDA_INA: track 318.1 -> 318.9 mm, vias 28 -> 27
- net SCL_INA: track 317.1 -> 316.4 mm
- net Net-(U1-VOUT): track 11.1 -> 10.5 mm
- added copper zone on B.Cu, net GND
Other:
- board outline added: 147.3 x 123.8 mm
- board text added: "3v3"
- board text added: "3v3_mk"
- board text added: "5v"
- board text added: "ENC_A"
- board text added: "ENC_B"
- board text added: "FS"
- board text added: "GND"
- board text added: "IN1"
- board text added: "IN2"
- board text added: "M+"
- board text added: "M-"
- board text added: "SCL"
- board text added: "SDA"
- board text added: "ch_A"
- board text added: "ch_B"

Commit message: trass
Parts:
- removed Con4: ~, Connector_PinHeader_2.54mm:PinHeader_1x02_P2.54mm_Vertical
- removed DRV1, DRV2, DRV3, DRV4, DRV5, DRV6: MC33886PVW, Package_SO:HSOP-20-1EP_11.0x15.9mm_P1.27mm_SlugUp
- removed I4, I5, I6, I7, I8, I9: INA226, Package_SO:TSSOP-10_3x3mm_P0.5mm
- removed J4, J5, J6: Conn_01x05_Pin, Connector_PinHeader_2.54mm:PinHeader_1x05_P2.54mm_Vertical
- removed R25, R32, R33, R34, R35, R36, R37, R44, R45, R46: 1, Resistor_SMD:R_0603_1608Metric
- removed R26, R27, R29, R38, R39, R41, R50, R51, R52, R56, R57, R58, R62, R63, R64, R68, R69, R70: 10k, Resistor_SMD:R_0805_2012Metric
- removed R28, R30, R31, R40, R42, R43: 10m, Resistor_SMD:R_0805_2012Metric
- removed R47, R48, R49, R53, R54, R55, R59, R60, R61, R65, R66, R67: 1k, Resistor_SMD:R_0805_2012Metric
- removed con3: KF202, Library_footprints:con_klemnic
- added ADC1: ~, Package_SO:TSSOP-38_4.4x9.7mm_P0.5mm, F.Cu at (160.2, 76.3)
- added C43: 1uF, Capacitor_SMD:C_0603_1608Metric, F.Cu at (159.8, 101.2)
- added C44: 10uF, Capacitor_SMD:C_0603_1608Metric, F.Cu at (159.8, 104.6)
- added C45: 1uF, Capacitor_SMD:C_0603_1608Metric, F.Cu at (88.6, 42.9)
- added C46: 10uF, Capacitor_SMD:C_0603_1608Metric, F.Cu at (88.6, 39.4)
- added C47: 1uF, Capacitor_SMD:C_0603_1608Metric, F.Cu at (96.3, 101.2)
- added C48: 10uF, Capacitor_SMD:C_0603_1608Metric, F.Cu at (96.3, 104.9)
- added C49: 0.1uF, Capacitor_SMD:C_0603_1608Metric, F.Cu at (159.8, 103.1)
- added C50: 0.1uF, Capacitor_SMD:C_0603_1608Metric, F.Cu at (88.6, 40.9)
- added C51: 0.1uF, Capacitor_SMD:C_0603_1608Metric, F.Cu at (96.3, 103.3)
- added C52: 0.1uF, Capacitor_SMD:C_0603_1608Metric, F.Cu at (151.3, 103.9)
- added C53: 0.1uF, Capacitor_SMD:C_0603_1608Metric, F.Cu at (97.0, 40.1)
- added C54: 0.1uF, Capacitor_SMD:C_0603_1608Metric, F.Cu at (87.9, 104.2)
- added C55: 47nF, Capacitor_SMD:C_1210_3225Metric, F.Cu at (169.6, 73.9)
- added C56: 10uF, Capacitor_SMD:C_0603_1608Metric, F.Cu at (174.2, 69.0)
- added C57: 100nF, Capacitor_SMD:C_0603_1608Metric, F.Cu at (160.3, 82.4)
- added C58: 100nF, Capacitor_SMD:C_0603_1608Metric, F.Cu at (166.2, 77.2)
- added C59: 100nF, Capacitor_SMD:C_0603_1608Metric, F.Cu at (162.6, 69.6)
- added C60: 10uF, Capacitor_SMD:C_0603_1608Metric, F.Cu at (167.5, 66.0)
- added C61: 0.1uF, Capacitor_SMD:C_0603_1608Metric, F.Cu at (159.2, 65.2)
- added C62: 1nF, Capacitor_SMD:C_0603_1608Metric, F.Cu at (159.9, 70.1)
- added Con3: DG125-5.0-02P-14-00A(H), TerminalBlock_Phoenix:TerminalBlock_Phoenix_MKDS-1,5-2_1x02_P5.00mm_Horizontal, F.Cu at (84.4, 65.2)
- added Con5: ~, Connector_PinHeader_2.54mm:PinHeader_1x02_P2.54mm_Vertical, F.Cu at (125.3, 83.7)
- added Kontur2: ~, Library_footprints:JetBot_AI_Kit_3x18650_Hole_Pattern, F.Cu at (79.1, 29.6)
- added U17: ISO7762FDBQ, Package_SO:SSOP-16_3.9x4.9mm_P0.635mm, F.Cu at (194.7, 76.6)
- added U18: ISO7762FDBQ, Package_SO:SSOP-16_3.9x4.9mm_P0.635mm, F.Cu at (194.7, 83.1)
- added U19: ISO7762FDBQ, Package_SO:SSOP-16_3.9x4.9mm_P0.635mm, F.Cu at (195.3, 89.5)
- added U20: ISO7762FDBQ, Package_SO:SSOP-16_3.9x4.9mm_P0.635mm, F.Cu at (233.0, 86.2)
- added con4: KF202, Library_footprints:con_klemnic, F.Cu at (79.1, 74.7)
- C12, C18, C8: footprint Capacitor_SMD:C_0603_1608Metric -> Capacitor_SMD:C_1206_3216Metric
- C19, C20, C21, C25, C27, C29, C37, C38, C39: value 100nF -> 1uF
- C22, C24: value 10uF -> 47nF; footprint Capacitor_SMD:C_0603_1608Metric -> Capacitor_SMD:C_1210_3225Metric
- C23, C40, C41, C42: value 100nF -> 47nF; footprint Capacitor_SMD:C_0603_1608Metric -> Capacitor_SMD:C_1210_3225Metric
- C28, C30: value 100nF -> 10uF
- C31, C33, C35: value 10uF -> 0.1uF
- C32, C34, C36: value 100nF -> 0.1uF
- Con2: value DG125-5.0-02P-14-00A(H) -> ~; footprint TerminalBlock_Phoenix:TerminalBlock_Phoenix_MKDS-1,5-2_1x02_P5.00mm_Horizontal -> Connector_PinHeader_2.54mm:PinHeader_1x02_P2.54mm_Vertical
- J1, J2: value Conn_01x05_Pin -> Conn_01x18_Pin; footprint Connector_PinHeader_2.54mm:PinHeader_1x05_P2.54mm_Vertical -> Connector_PinHeader_2.54mm:PinHeader_2x09_P2.54mm_Vertical
- J3: value Conn_01x05_Pin -> Conn_01x06_Pin; footprint Connector_PinHeader_2.54mm:PinHeader_1x05_P2.54mm_Vertical -> Connector_PinHeader_2.54mm:PinHeader_1x06_P2.54mm_Vertical
- JP1, JP2, JP3, JP4, JP5, JP6, JP7, JP8, JP9: footprint Jumper:SolderJumper-3_P1.3mm_Bridged123_Pad1.0x1.5mm -> Connector_PinHeader_2.54mm:PinHeader_1x03_P2.54mm_Vertical
- R17, R18, R19, R20, R21, R22: value 1k -> 10k
- R24: value 1 -> 10; footprint Resistor_SMD:R_0603_1608Metric -> Resistor_SMD:R_0805_2012Metric
- U10, U11, U6, U7, U8, U9: value PC817 -> DRV8873SPWPRQ1; footprint Package_DIP:DIP-4_W7.62mm_SMDSocket_SmallPads -> Library_footprints:C2150678_HTSSOP-24_L7_8-W4_4-P0_65-LS6_4-TL-EP
- U12: value PC817 -> REF5025AD; footprint Package_DIP:DIP-4_W7.62mm_SMDSocket_SmallPads -> Package_SO:SOIC-8_3.9x4.9mm_P1.27mm
- U13, U14, U15: value PC817 -> ISO7762FDBQ; footprint Package_DIP:DIP-4_W7.62mm_SMDSocket_SmallPads -> Package_SO:SSOP-16_3.9x4.9mm_P0.635mm
- U16: value PC817 -> TLV9061xDBV; footprint Package_DIP:DIP-4_W7.62mm_SMDSocket_SmallPads -> Package_TO_SOT_SMD:SOT-23-5
- U3: value TPS5450 -> ISO1540; footprint Package_SO:SOIC-8-1EP_3.9x4.9mm_P1.27mm_EP2.29x3mm -> Package_SO:SOIC-8_3.9x4.9mm_P1.27mm
- U5: value PC817 -> TPS5450; footprint Package_DIP:DIP-4_W7.62mm_SMDSocket_SmallPads -> Package_SO:SOIC-8-1EP_3.9x4.9mm_P1.27mm_EP2.29x3mm
- moved M_Con5 140.1 mm to (101.1, 23.1), turned to 180 degrees
- moved C41 136.3 mm to (88.5, 49.0), turned to -90 degrees
- moved R21 128.6 mm to (88.7, 55.5)
- moved D29 127.6 mm to (90.2, 103.3), turned to 180 degrees
- moved D13 125.0 mm to (182.6, 43.4), turned to 0 degrees
- moved D27 118.1 mm to (94.8, 41.0)
- moved J1 114.8 mm to (228.5, 66.8), turned to -90 degrees
- moved D5 112.4 mm to (93.5, 68.5), turned to -90 degrees
- moved D17 112.3 mm to (150.9, 43.2), turned to 0 degrees
- moved C14 112.3 mm to (91.7, 62.8), turned to 0 degrees
- moved D14 112.1 mm to (182.6, 41.8)
- moved D28 111.3 mm to (94.8, 39.4), turned to 0 degrees
- moved JP8 110.5 mm to (100.2, 39.3), turned to 90 degrees
- moved U10 110.2 mm to (94.2, 48.9), turned to 90 degrees
- moved D30 109.9 mm to (90.2, 105.0), turned to 180 degrees
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Connections:
- C10 pad 1: Net-(U3-BOOT) -> Net-(U4-BOOT)
- C14 pad 1: +14.4v -> +14.4v*
- C14 pad 2: GND -> GND*
- C16 pad 1: Net-(U4-BOOT) -> Net-(U5-BOOT)
- C19 pad 1: Net-(DRV1-CCP) -> GND
- C19 pad 2: GND -> Net-(U6-DVDD)
- C20 pad 1: Net-(DRV2-CCP) -> GND
- C20 pad 2: GND -> Net-(U7-DVDD)
- C21 pad 1: Net-(DRV3-CCP) -> GND
- C21 pad 2: GND -> Net-(U8-DVDD)
- C22 pad 1: INA2 -> Net-(U6-CPL)
- C22 pad 2: GND -> Net-(U6-CPH)
- C23 pad 1: INA2 -> Net-(U7-CPL)
- C23 pad 2: GND -> Net-(U7-CPH)
- C24 pad 1: INA3 -> Net-(U8-CPL)
- C24 pad 2: GND -> Net-(U8-CPH)
- C25 pad 1: INA3 -> Net-(U6-VCP)
- C25 pad 2: GND -> +14.4v
- C26 pad 1: INA1 -> +14.4v
- C27 pad 1: INA1 -> Net-(U7-VCP)
- C27 pad 2: GND -> +14.4v
- C28 pad 1: Net-(DRV4-CCP) -> +14.4v
- C29 pad 1: Net-(DRV5-CCP) -> Net-(U8-VCP)
- C29 pad 2: GND -> +14.4v
- C3 pad 1: +5v -> +5v*
- C3 pad 2: GND -> GND*
- C30 pad 1: Net-(DRV6-CCP) -> +14.4v
- C31 pad 1: INA6 -> GND
- C31 pad 2: GND -> +14.4v
- C32 pad 1: INA6 -> GND
- C32 pad 2: GND -> +14.4v
- C33 pad 1: INA5 -> GND
- C33 pad 2: GND -> +14.4v
- C34 pad 1: INA5 -> GND
- C34 pad 2: GND -> +14.4v
- C35 pad 1: INA4 -> GND
- C35 pad 2: GND -> +14.4v
- C36 pad 1: INA4 -> GND
- C36 pad 2: GND -> +14.4v
- C37 pad 1: Net-(I4-IN+) -> GND
- C37 pad 2: Net-(I4-IN-) -> Net-(U9-DVDD)
- C38 pad 1: Net-(I5-IN+) -> GND
- C38 pad 2: Net-(I5-IN-) -> Net-(U10-DVDD)
- C39 pad 1: Net-(I6-IN+) -> GND
- C39 pad 2: Net-(I6-IN-) -> Net-(U11-DVDD)
- C4 pad 1: +5v -> +5v*
- C4 pad 2: GND -> GND*
- C40 pad 1: Net-(I7-IN+) -> Net-(U9-CPL)
- C40 pad 2: Net-(I7-IN-) -> Net-(U9-CPH)
- C41 pad 1: Net-(I8-IN+) -> Net-(U10-CPL)
- C41 pad 2: Net-(I8-IN-) -> Net-(U10-CPH)
- C42 pad 1: Net-(I9-IN+) -> Net-(U11-CPL)
- C42 pad 2: Net-(I9-IN-) -> Net-(U11-CPH)
- C5 pad 1: Net-(U1-VOUT) -> +3,3v*
- C5 pad 2: GND -> GND*
- C6 pad 1: Net-(U1-VOUT) -> +3,3v*
- C6 pad 2: GND -> GND*
- C7 pad 1: +5v -> +5v*
- C7 pad 2: GND -> GND*
- C8 pad 1: GND -> GND*
- Con2 pad 1: +14.4v -> Net-(U3-SDA2)
- Con2 pad 2: GND -> Net-(U3-SCL2)
- D1 pad 1: GND -> GND*
- D10 pad 2: CONN_M2_1 -> CONN_1_M2
- D11 pad 1: +14.4v -> CONN_1_M3
- D11 pad 2: CONN_M3_2 -> GND
- D12 pad 2: CONN_M3_1 -> CONN_1_M3
- D13 pad 1: +14.4v -> CONN_2_M1
- D13 pad 2: CONN_M4_2 -> GND
- D14 pad 2: CONN_M4_1 -> CONN_2_M1
- D15 pad 1: +14.4v -> CONN_2_M2
- D15 pad 2: CONN_M5_2 -> GND
- D16 pad 2: CONN_M5_1 -> CONN_2_M2
- D17 pad 1: +14.4v -> CONN_2_M3
- D17 pad 2: CONN_M6_2 -> GND
- D18 pad 2: CONN_M6_1 -> CONN_2_M3
- D19 pad 1: CONN_M1_2 -> CONN_1_M4
- D2 pad 2: GND -> GND*
- D20 pad 1: CONN_M1_1 -> +14.4v
- D20 pad 2: GND -> CONN_1_M4
- D21 pad 1: CONN_M2_2 -> CONN_1_M5
- D22 pad 1: CONN_M2_1 -> +14.4v
- D22 pad 2: GND -> CONN_1_M5
- D23 pad 1: CONN_M3_2 -> CONN_1_M6
- D24 pad 1: CONN_M3_1 -> +14.4v
- D24 pad 2: GND -> CONN_1_M6
- D25 pad 1: CONN_M4_2 -> CONN_2_M4
- D26 pad 1: CONN_M4_1 -> +14.4v
- D26 pad 2: GND -> CONN_2_M4
- D27 pad 1: CONN_M5_2 -> CONN_2_M5
- D28 pad 1: CONN_M5_1 -> +14.4v
- D28 pad 2: GND -> CONN_2_M5
- D29 pad 1: CONN_M6_2 -> CONN_2_M6
- D30 pad 1: CONN_M6_1 -> +14.4v
- D30 pad 2: GND -> CONN_2_M6
- D5 pad 1: +14.4v -> +14.4v*
- D5 pad 2: GND -> GND*
- D7 pad 1: +14.4v -> CONN_1_M1
- D7 pad 2: CONN_M1_2 -> GND
- D8 pad 2: CONN_M1_1 -> CONN_1_M1
- D9 pad 1: +14.4v -> CONN_1_M2
- D9 pad 2: CONN_M2_2 -> GND
- I1 pad 1: GND -> GND*
- I1 pad 2: GND -> GND*
- I1 pad 6: +5v -> +5v*
- I1 pad 7: GND -> GND*
- J1 pad 1: IN1_M3 -> nSCS_mk_1
- J1 pad 2: IN2_M3 -> EN/IN1_mk_1
- J1 pad 3: FS3 -> PH/IN2_mk_1
- J1 pad 4: ENC_A_M3_mk -> DISABLE_mk_1
- J1 pad 5: ENC_B_M3_mk -> ENC_A_M1_mk
- J2 pad 1: IN1_M1 -> nSCS_mk_4
- J2 pad 2: IN2_M1 -> EN/IN1_mk_4
- J2 pad 3: FS1 -> PH/IN2_mk_4
- J2 pad 4: ENC_A_M1_mk -> DISABLE_mk_4
- J2 pad 5: ENC_B_M1_mk -> ENC_A_M4_mk
- J3 pad 1: IN1_M5 -> Net-(J3-Pin_1)
- J3 pad 2: IN2_M5 -> Net-(J3-Pin_2)
- J3 pad 3: FS5 -> Net-(J3-Pin_3)
- J3 pad 4: ENC_A_M5_mk -> Net-(J3-Pin_4)
- J3 pad 5: ENC_B_M5_mk -> unconnected-(J3-Pin_5-Pad5)
- L1 pad 2: +5v -> +5v*
- M_Con1 pad 1: CONN_M1_2 -> CONN_2_M1
- M_Con1 pad 2: CONN_M1_1 -> CONN_1_M1
- M_Con2 pad 1: CONN_M2_2 -> CONN_2_M2
- M_Con2 pad 2: CONN_M2_1 -> CONN_1_M2
- M_Con3 pad 1: CONN_M3_2 -> CONN_2_M3
- M_Con3 pad 2: CONN_M3_1 -> CONN_1_M3
- M_Con4 pad 1: CONN_M4_2 -> CONN_2_M4
- M_Con4 pad 2: CONN_M4_1 -> CONN_1_M4
- M_Con5 pad 1: CONN_M5_2 -> CONN_2_M5
- M_Con5 pad 2: CONN_M5_1 -> CONN_1_M5
- M_Con6 pad 1: CONN_M6_2 -> CONN_2_M6
- M_Con6 pad 2: CONN_M6_1 -> CONN_1_M6
- R1 pad 2: +14.4v -> +14.4v*
- R11 pad 1: GND -> Net-(U4-VSENSE)
- R16 pad 1: GND -> Net-(U5-VSENSE)
- R17 pad 1: +5v -> +3,3v
- R17 pad 2: FS2 -> nFault_ISO
- R18 pad 1: +5v -> +3,3v
- R18 pad 2: FS3 -> nFault_ISO
- R19 pad 1: +5v -> +3,3v
- R19 pad 2: FS1 -> nFault_ISO
- R2 pad 1: +14.4v -> +14.4v*
- R20 pad 1: +5v -> +3,3v
- R20 pad 2: FS5 -> nFault_ISO
- R21 pad 1: +5v -> +3,3v
- R21 pad 2: FS6 -> nFault_ISO
- R22 pad 1: +5v -> +3,3v
- R22 pad 2: FS4 -> nFault_ISO
- R23 pad 1: Net-(I4-IN+) -> Net-(ADC1-REFP)
- R23 pad 2: +14.4v -> Net-(C55-Pad1)
- R24 pad 1: Net-(I5-IN+) -> Net-(U16--)
- R24 pad 2: +14.4v -> Net-(ADC1-AINP)
- R4 pad 1: +5v -> +5v*
- R5 pad 1: +5v -> +5v*
- R5 pad 2: GND -> GND*
- R6 pad 1: GND -> Net-(U2-VSENSE)
- R6 pad 2: GND -> GND*
- U1 pad 1: +5v -> +5v*
- U1 pad 2: GND -> GND*
- U1 pad 4: Net-(U1-VOUT) -> +3,3v*
- U1 pad 6: +5v -> +5v*
- U10 pad 1: Net-(R55-Pad2) -> Net-(U10-DVDD)
- U10 pad 2: GND -> nFault_ISO
- U10 pad 3: ENC_B_M1_mk -> SDO_ISO
- U10 pad 4: +5v -> SDI_ISO
- U11 pad 1: Net-(R59-Pad2) -> Net-(U11-DVDD)
- U11 pad 2: GND -> nFault_ISO
- U11 pad 3: ENC_A_M2_mk -> SDO_ISO
- U11 pad 4: +5v -> SDI_ISO
- U12 pad 1: Net-(R60-Pad2) -> unconnected-(U12-DNC-Pad1)
- U12 pad 2: GND -> +3,3v*
- U12 pad 3: ENC_A_M4_mk -> unconnected-(U12-Temp-Pad3)
- U12 pad 4: +5v -> GND*
- U13 pad 1: Net-(R61-Pad2) -> +3,3v*
- U13 pad 2: GND -> nSCS_mk_1
- U13 pad 3: ENC_A_M6_mk -> EN/IN1_mk_1
- U13 pad 4: +5v -> PH/IN2_mk_1
- U14 pad 1: Net-(R65-Pad2) -> +3,3v*
- U14 pad 2: GND -> nSCS_mk_2
- U14 pad 3: ENC_B_M2_mk -> EN/IN1_mk_2
- U14 pad 4: +5v -> PH/IN2_mk_2
- U15 pad 1: Net-(R66-Pad2) -> +3,3v*
- U15 pad 2: GND -> nSCS_mk_3
- U15 pad 3: ENC_B_M4_mk -> EN/IN1_mk_3
- U15 pad 4: +5v -> PH/IN2_mk_3
- U16 pad 1: Net-(R67-Pad2) -> Net-(U16--)
- U16 pad 2: GND -> GND*
- U16 pad 3: ENC_B_M6_mk -> Net-(ADC1-MXO)
- U16 pad 4: +5v -> Net-(U16--)
- U2 pad 4: GND -> Net-(U2-VSENSE)
- U2 pad 6: GND -> GND*
- U2 pad 9: GND -> GND*
- U3 pad 1: Net-(U3-BOOT) -> +3,3v
- U3 pad 2: unconnected-(U3-NC-Pad2) -> SDA_INA
- U3 pad 3: unconnected-(U3-NC-Pad3) -> SCL_INA
- U3 pad 5: ENA_U4 -> GND*
- U3 pad 6: GND -> Net-(U3-SCL2)
- U3 pad 7: Net-(JP2-A) -> Net-(U3-SDA2)
- U3 pad 8: Net-(D3-K) -> +3,3v*
- U4 pad 4: GND -> Net-(U4-VSENSE)
- U4 pad 5: ENA_U5 -> ENA_U4
- U4 pad 7: Net-(JP3-A) -> Net-(JP2-A)
- U4 pad 8: Net-(D6-K) -> Net-(D3-K)
- U5 pad 1: Net-(R47-Pad2) -> Net-(U5-BOOT)
- U5 pad 2: GND -> unconnected-(U5-NC-Pad2)
- U5 pad 3: ENC_A_M3_mk -> unconnected-(U5-NC-Pad3)
- U5 pad 4: +5v -> Net-(U5-VSENSE)
- U6 pad 1: Net-(R48-Pad2) -> Net-(U6-DVDD)
- U6 pad 2: GND -> nFault_ISO
- U6 pad 3: ENC_A_M5_mk -> SDO_ISO
- U6 pad 4: +5v -> SDI_ISO
- U7 pad 1: Net-(R49-Pad2) -> Net-(U7-DVDD)
- U7 pad 2: GND -> nFault_ISO
- U7 pad 3: ENC_A_M1_mk -> SDO_ISO
- U7 pad 4: +5v -> SDI_ISO
- U8 pad 1: Net-(R53-Pad2) -> Net-(U8-DVDD)
- U8 pad 2: GND -> nFault_ISO
- U8 pad 3: ENC_B_M3_mk -> SDO_ISO
- U8 pad 4: +5v -> SDI_ISO
- U9 pad 1: Net-(R54-Pad2) -> Net-(U9-DVDD)
- U9 pad 2: GND -> nFault_ISO
- U9 pad 3: ENC_B_M5_mk -> SDO_ISO
- U9 pad 4: +5v -> SDI_ISO
- con1 pad 1: GND -> GND*
- con1 pad 2: +5v -> +3,3v*
- con1 pad 3: Net-(U1-VOUT) -> +5v*
Routing:
- net GND: track 2034.0 -> 0.00 mm, vias 20 -> 0
- net +5v: track 977.0 -> 0.00 mm, vias 52 -> 0
- net +14.4v: track 636.2 -> 0.00 mm
- net +3,3v: track 459.6 -> 0.00 mm, vias 10 -> 0
- net SDA_INA: track 318.9 -> 0.00 mm, vias 27 -> 0
- net SCL_INA: track 316.4 -> 0.00 mm, vias 22 -> 0
- net INA5: track 61.5 -> 0.00 mm, vias 2 -> 0
- net INA6: track 61.4 -> 0.00 mm, vias 2 -> 0
- net INA4: track 60.4 -> 0.00 mm, vias 2 -> 0
- net INA3: track 60.0 -> 0.00 mm, vias 2 -> 0
- net INA1: track 59.8 -> 0.00 mm, vias 2 -> 0
- net INA2: track 58.1 -> 0.00 mm, vias 2 -> 0
- net IN2_M3: track 43.2 -> 0.00 mm, vias 2 -> 0
- net IN2_M6: track 41.1 -> 0.00 mm, vias 2 -> 0
- net IN2_M5: track 40.4 -> 0.00 mm, vias 2 -> 0
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- removed copper zone on B.Cu, net GND
Other:
- board text removed: "3v3"
- board text removed: "3v3_mk"
- board text removed: "5v"
- board text removed: "ENC_A"
- board text removed: "ENC_B"
- board text removed: "FS"
- board text removed: "GND"
- board text removed: "IN1"
- board text removed: "IN2"
- board text removed: "M+"
- board text removed: "M-"
- board text removed: "SCL"
- board text removed: "SDA"
- board text removed: "ch_A"
- board text removed: "ch_B"

Commit message: tray
Parts:
- removed Con2, Con5: ~, Connector_PinHeader_2.54mm:PinHeader_1x02_P2.54mm_Vertical
- removed Con3: DG125-5.0-02P-14-00A(H), TerminalBlock_Phoenix:TerminalBlock_Phoenix_MKDS-1,5-2_1x02_P5.00mm_Horizontal
- removed Kontur2: ~, Library_footprints:JetBot_AI_Kit_3x18650_Hole_Pattern
- removed U10, U11, U6, U7, U8, U9: DRV8873SPWPRQ1, Library_footprints:C2150678_HTSSOP-24_L7_8-W4_4-P0_65-LS6_4-TL-EP
- removed U12: REF5025AD, Package_SO:SOIC-8_3.9x4.9mm_P1.27mm
- removed U13, U14, U15, U17, U18, U19, U20: ISO7762FDBQ, Package_SO:SSOP-16_3.9x4.9mm_P0.635mm
- removed U16: TLV9061xDBV, Package_TO_SOT_SMD:SOT-23-5
- removed U5: TPS5450, Package_SO:SOIC-8-1EP_3.9x4.9mm_P1.27mm_EP2.29x3mm
- removed con1: ~, Connector_PinHeader_2.54mm:PinHeader_1x03_P2.54mm_Vertical
- removed con4: KF202, Library_footprints:con_klemnic
- added DRV1: DRV8873SPWPRQ1, Library_footprints:C2150678_HTSSOP-24_L7_8-W4_4-P0_65-LS6_4-TL-EP, F.Cu at (166.7, 77.6)
- added DRV2: DRV8873SPWPRQ1, Library_footprints:C2150678_HTSSOP-24_L7_8-W4_4-P0_65-LS6_4-TL-EP, F.Cu at (157.3, 122.9)
- added DRV3: DRV8873SPWPRQ1, Library_footprints:C2150678_HTSSOP-24_L7_8-W4_4-P0_65-LS6_4-TL-EP, F.Cu at (153.4, 77.8)
- added DRV4: DRV8873SPWPRQ1, Library_footprints:C2150678_HTSSOP-24_L7_8-W4_4-P0_65-LS6_4-TL-EP, F.Cu at (143.8, 122.9)
- added DRV5: DRV8873SPWPRQ1, Library_footprints:C2150678_HTSSOP-24_L7_8-W4_4-P0_65-LS6_4-TL-EP, F.Cu at (140.2, 78.0)
- added DRV6: DRV8873SPWPRQ1, Library_footprints:C2150678_HTSSOP-24_L7_8-W4_4-P0_65-LS6_4-TL-EP, F.Cu at (130.7, 122.8)
- added ISO1: ISO7762FDBQ, Package_SO:SSOP-16_3.9x4.9mm_P0.635mm, F.Cu at (168.0, 86.8)
- added ISO2: ISO7762FDBQ, Package_SO:SSOP-16_3.9x4.9mm_P0.635mm, F.Cu at (155.9, 113.2)
- added ISO3: ISO7762FDBQ, Package_SO:SSOP-16_3.9x4.9mm_P0.635mm, F.Cu at (154.5, 86.9)
- added ISO4: ISO7762FDBQ, Package_SO:SSOP-16_3.9x4.9mm_P0.635mm, F.Cu at (142.4, 113.2)
- added ISO5: ISO7762FDBQ, Package_SO:SSOP-16_3.9x4.9mm_P0.635mm, F.Cu at (131.0, 112.3)
- added ISO6: ISO7762FDBQ, Package_SO:SSOP-16_3.9x4.9mm_P0.635mm, F.Cu at (141.4, 86.9)
- added ISO7: ISO7762FDBQ, Package_SO:SSOP-16_3.9x4.9mm_P0.635mm, F.Cu at (146.2, 95.5)
- added ISO8: ISO1540, Package_SO:SOIC-8_3.9x4.9mm_P1.27mm, F.Cu at (146.0, 101.1)
- added Klem_clear1: DG125-5.0-02P-14-00A(H), TerminalBlock_Phoenix:TerminalBlock_Phoenix_MKDS-1,5-2_1x02_P5.00mm_Horizontal, F.Cu at (200.9, 86.5)
- added Klem_dirty1: KF202, Library_footprints:con_klemnic, F.Cu at (86.0, 86.3)
- added Kontur1: ~, Library_footprints:JetBot_AI_Kit_3x18650_Hole_Pattern, F.Cu at (86.0, 58.4)
- added OPER1: TLV9061xDBV, Package_TO_SOT_SMD:SOT-23-5, F.Cu at (174.2, 99.1)
- added REF1: REF5025AD, Package_SO:SOIC-8_3.9x4.9mm_P1.27mm, F.Cu at (169.5, 99.8)
- J3: value Conn_01x06_Pin -> Conn_01x12_Pin; footprint Connector_PinHeader_2.54mm:PinHeader_1x06_P2.54mm_Vertical -> Connector_PinHeader_2.54mm:PinHeader_2x06_P2.54mm_Vertical
- U3: value ISO1540 -> TPS5450; footprint Package_SO:SOIC-8_3.9x4.9mm_P1.27mm -> Package_SO:SOIC-8-1EP_3.9x4.9mm_P1.27mm_EP2.29x3mm
- moved R1 108.7 mm to (204.6, 104.8), turned to 90 degrees
- moved C14 106.2 mm to (194.4, 89.9), turned to -90 degrees
- moved R2 105.3 mm to (202.1, 104.3), turned to 180 degrees
- moved C1 104.9 mm to (202.1, 106.0), turned to 180 degrees
- moved I1 104.5 mm to (202.1, 108.6), turned to 0 degrees
- moved C2 103.2 mm to (199.8, 100.5), turned to -90 degrees
- moved R3 101.7 mm to (199.6, 104.8), turned to 90 degrees
- moved D5 99.3 mm to (191.7, 83.4), turned to 90 degrees
- moved U3 99.2 mm to (110.1, 112.0), turned to 90 degrees
- moved D2 99.0 mm to (195.0, 94.5), turned to 180 degrees
- moved R6 98.5 mm to (195.2, 96.2), turned to 180 degrees
- moved U2 98.2 mm to (196.3, 101.0), turned to -90 degrees
- moved C8 97.1 mm to (196.5, 106.0), turned to 0 degrees
- moved JP4 95.1 mm to (96.1, 67.8)
- moved JP5 94.7 mm to (95.4, 132.9)
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Connections:
- ADC1 pad 13: IPROPI1_2 -> IPROPI1_3
- ADC1 pad 14: IPROPI2_2 -> IPROPI2_3
- ADC1 pad 15: IPROPI1_3 -> IPROPI2_5
- ADC1 pad 16: IPROPI2_3 -> IPROPI1_5
- ADC1 pad 25: IPROPI2_5 -> IPROPI2_4
- ADC1 pad 26: IPROPI1_5 -> IPROPI1_4
- ADC1 pad 27: IPROPI2_4 -> IPROPI2_2
- ADC1 pad 28: IPROPI1_4 -> IPROPI1_2
- C10 pad 1: Net-(U4-BOOT) -> Net-(U3-BOOT)
- C16 pad 1: Net-(U5-BOOT) -> Net-(U4-BOOT)
- J1 pad 10: DISABLE_mk_2 -> DISABLE_mk_3
- J1 pad 11: ENC_A_M2_mk -> ENC_A_M3_mk
- J1 pad 12: ENC_B_M2_mk -> ENC_B_M3_mk
- J1 pad 13: nSCS_mk_3 -> nSCS_mk_5
- J1 pad 14: EN/IN1_mk_3 -> EN/IN1_mk_5
- J1 pad 15: PH/IN2_mk_3 -> PH/IN2_mk_5
- J1 pad 16: DISABLE_mk_3 -> DISABLE_mk_5
- J1 pad 17: ENC_A_M3_mk -> ENC_A_M5_mk
- J1 pad 18: ENC_B_M3_mk -> ENC_B_M5_mk
- J1 pad 7: nSCS_mk_2 -> nSCS_mk_3
- J1 pad 8: EN/IN1_mk_2 -> EN/IN1_mk_3
- J1 pad 9: PH/IN2_mk_2 -> PH/IN2_mk_3
- J2 pad 1: nSCS_mk_4 -> nSCS_mk_2
- J2 pad 10: DISABLE_mk_5 -> DISABLE_mk_4
- J2 pad 11: ENC_A_M5_mk -> ENC_A_M4_mk
- J2 pad 12: ENC_B_M5_mk -> ENC_B_M4_mk
- J2 pad 2: EN/IN1_mk_4 -> EN/IN1_mk_2
- J2 pad 3: PH/IN2_mk_4 -> PH/IN2_mk_2
- J2 pad 4: DISABLE_mk_4 -> DISABLE_mk_2
- J2 pad 5: ENC_A_M4_mk -> ENC_A_M2_mk
- J2 pad 6: ENC_B_M4_mk -> ENC_B_M2_mk
- J2 pad 7: nSCS_mk_5 -> nSCS_mk_4
- J2 pad 8: EN/IN1_mk_5 -> EN/IN1_mk_4
- J2 pad 9: PH/IN2_mk_5 -> PH/IN2_mk_4
- J3 pad 5: unconnected-(J3-Pin_5-Pad5) -> Net-(ISO8-SDA2)
- M_Con1 pad 1: CONN_2_M1 -> Net-(JP4-C)
- M_Con1 pad 2: CONN_1_M1 -> GND
- M_Con1 pad 3: Net-(JP4-C) -> CONN_1_M1
- M_Con1 pad 4: ENC_B_M1 -> CONN_2_M1
- M_Con1 pad 6: GND -> ENC_B_M1
- M_Con2 pad 1: CONN_2_M2 -> ENC_A_M2
- M_Con2 pad 2: CONN_1_M2 -> ENC_B_M2
- M_Con2 pad 3: Net-(JP5-C) -> CONN_1_M2
- M_Con2 pad 4: ENC_B_M2 -> CONN_2_M2
- M_Con2 pad 5: ENC_A_M2 -> GND
- M_Con2 pad 6: GND -> Net-(JP5-C)
- M_Con3 pad 1: CONN_2_M3 -> Net-(JP6-C)
- M_Con3 pad 2: CONN_1_M3 -> GND
- M_Con3 pad 3: Net-(JP6-C) -> CONN_1_M3
- M_Con3 pad 4: ENC_B_M3 -> CONN_2_M3
- M_Con3 pad 6: GND -> ENC_B_M3
- M_Con4 pad 1: CONN_2_M4 -> ENC_A_M4
- M_Con4 pad 2: CONN_1_M4 -> ENC_B_M4
- M_Con4 pad 3: Net-(JP7-C) -> CONN_1_M4
- M_Con4 pad 4: ENC_B_M4 -> CONN_2_M4
- M_Con4 pad 5: ENC_A_M4 -> GND
- M_Con4 pad 6: GND -> Net-(JP7-C)
- M_Con5 pad 1: CONN_2_M5 -> Net-(JP8-C)
- M_Con5 pad 2: CONN_1_M5 -> GND
- M_Con5 pad 3: Net-(JP8-C) -> CONN_1_M5
- M_Con5 pad 4: ENC_B_M5 -> CONN_2_M5
- M_Con5 pad 6: GND -> ENC_B_M5
- M_Con6 pad 1: CONN_2_M6 -> ENC_A_M6
- M_Con6 pad 2: CONN_1_M6 -> ENC_B_M6
- M_Con6 pad 3: Net-(JP9-C) -> CONN_1_M6
- M_Con6 pad 4: ENC_B_M6 -> CONN_2_M6
- M_Con6 pad 5: ENC_A_M6 -> GND
- M_Con6 pad 6: GND -> Net-(JP9-C)
- R11 pad 1: Net-(U4-VSENSE) -> Net-(U3-VSENSE)
- R16 pad 1: Net-(U5-VSENSE) -> Net-(U4-VSENSE)
- U3 pad 1: +3,3v -> Net-(U3-BOOT)
- U3 pad 2: SDA_INA -> unconnected-(U3-NC-Pad2)
- U3 pad 3: SCL_INA -> unconnected-(U3-NC-Pad3)
- U3 pad 4: GND -> Net-(U3-VSENSE)
- U3 pad 5: GND* -> ENA_U4
- U3 pad 6: Net-(U3-SCL2) -> GND
- U3 pad 7: Net-(U3-SDA2) -> Net-(JP2-A)
- U3 pad 8: +3,3v* -> Net-(D3-K)
- U4 pad 5: ENA_U4 -> ENA_U5
- U4 pad 7: Net-(JP2-A) -> Net-(JP3-A)
- U4 pad 8: Net-(D3-K) -> Net-(D6-K)
Routing:
- net +14.4v: track 0.00 -> 444.8 mm
- net +3,3v: track 0.00 -> 307.8 mm, vias 0 -> 3
- net +5v: track 0.00 -> 243.5 mm, vias 0 -> 2
- net +3,3v*: track 0.00 -> 186.4 mm, vias 0 -> 4
- net SCLK_ISO: track 0.00 -> 153.1 mm, vias 0 -> 9
- net SDI_ISO: track 0.00 -> 152.3 mm, vias 0 -> 8
- net nFault_ISO: track 0.00 -> 150.6 mm, vias 0 -> 12
- net SDO_ISO: track 0.00 -> 132.3 mm, vias 0 -> 8
- net SDA_INA: track 0.00 -> 98.4 mm, vias 0 -> 5
- net Net-(JP4-C): track 0.00 -> 94.5 mm
- net Net-(JP5-C): track 0.00 -> 91.0 mm
- net ENC_A_M2: track 0.00 -> 90.3 mm, vias 0 -> 1
- net GND*: track 0.00 -> 88.7 mm, vias 0 -> 4
- net SCL_INA: track 0.00 -> 88.4 mm, vias 0 -> 4
- net ENC_B_M2: track 0.00 -> 83.6 mm, vias 0 -> 1
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Other:
- board size 147.3 x 123.8 mm -> 133.8 x 103.9 mm

Commit message: trass
Parts:
- removed C62: 1nF, Capacitor_SMD:C_0603_1608Metric
- removed Klem_clear1: DG125-5.0-02P-14-00A(H), TerminalBlock_Phoenix:TerminalBlock_Phoenix_MKDS-1,5-2_1x02_P5.00mm_Horizontal
- added F1: Fuse, Fuse:Fuseholder_Clip-5x20mm_Bel_FC-203-22_Lateral_P17.80x5.00mm_D1.17mm_Horizontal, F.Cu at (93.0, 88.7)
- added R25: 10, Resistor_SMD:R_0805_2012Metric, F.Cu at (190.6, 88.3)
- C15: value 100nF -> 10nF
- C16: value 10nF -> 330uF; footprint Capacitor_SMD:C_0603_1608Metric -> Capacitor_Tantalum_SMD:CP_EIA-7343-31_Kemet-D_HandSolder
- C17: value 330uF -> 4.7uF; footprint Capacitor_Tantalum_SMD:CP_EIA-7343-31_Kemet-D_HandSolder -> Capacitor_SMD:C_1206_3216Metric
- C18: value 4.7uF -> 1uF; footprint Capacitor_SMD:C_1206_3216Metric -> Capacitor_SMD:C_0603_1608Metric
- C21, C39: value 1uF -> 47nF; footprint Capacitor_SMD:C_0603_1608Metric -> Capacitor_SMD:C_1210_3225Metric
- C24, C42: value 47nF -> 1uF; footprint Capacitor_SMD:C_1210_3225Metric -> Capacitor_SMD:C_0603_1608Metric
- C25, C27, C29, C43, C45, C47: value 1uF -> 10uF
- C26, C28, C44, C46: value 10uF -> 1uF
- C30, C48, C60: value 10uF -> 0.1uF
- C36: value 0.1uF -> 1uF
- C54: value 0.1uF -> 47nF; footprint Capacitor_SMD:C_0603_1608Metric -> Capacitor_SMD:C_1210_3225Metric
- C55: value 47nF -> 10uF; footprint Capacitor_SMD:C_1210_3225Metric -> Capacitor_SMD:C_0603_1608Metric
- C56: value 10uF -> 100nF
- C59: value 100nF -> 10uF
- C61: value 0.1uF -> 1nF
- D4: value SS54L -> Green; footprint Diode_SMD:D_SMC -> LED_SMD:LED_0603_1608Metric
- J3: value Conn_01x12_Pin -> Conn_01x10_Pin; footprint Connector_PinHeader_2.54mm:PinHeader_2x06_P2.54mm_Vertical -> Connector_PinHeader_2.54mm:PinHeader_2x05_P2.54mm_Vertical
- R11: value 6.8K -> 2.2k; footprint Resistor_SMD:R_0805_2012Metric -> Resistor_SMD:R_0603_1608Metric
- R12: value 1 -> 6.8K; footprint Resistor_SMD:R_0603_1608Metric -> Resistor_SMD:R_0805_2012Metric
- R13: value 10m -> 1; footprint Resistor_SMD:R_0805_2012Metric -> Resistor_SMD:R_0603_1608Metric
- R14: value 1 -> 10m; footprint Resistor_SMD:R_0603_1608Metric -> Resistor_SMD:R_0805_2012Metric
- R15: value 10k -> 1; footprint Resistor_SMD:R_0805_2012Metric -> Resistor_SMD:R_0603_1608Metric
- R16: value 3.3k -> 10k
- R17: value 10k -> 3.3k
- R23: value 1 -> 10k; footprint Resistor_SMD:R_0603_1608Metric -> Resistor_SMD:R_0805_2012Metric
- R24: value 10 -> 1; footprint Resistor_SMD:R_0805_2012Metric -> Resistor_SMD:R_0603_1608Metric
- moved D5 96.1 mm to (97.8, 103.9), turned to -90 degrees
- moved R1 93.0 mm to (113.3, 122.9), turned to -90 degrees
- moved R2 88.3 mm to (115.8, 123.4), turned to 0 degrees
- moved C1 87.6 mm to (115.8, 121.7), turned to 0 degrees
- moved I1 87.0 mm to (115.8, 119.1), turned to 180 degrees
- moved C2 86.0 mm to (118.1, 127.2), turned to 90 degrees
- moved R3 83.3 mm to (118.3, 122.9), turned to -90 degrees
- moved D2 81.9 mm to (122.9, 133.2), turned to 0 degrees
- moved R6 80.6 mm to (122.7, 131.4), turned to 0 degrees
- moved C14 80.1 mm to (115.2, 78.1), turned to 0 degrees
- moved U2 79.0 mm to (121.6, 126.6), turned to 90 degrees
- moved C8 76.7 mm to (121.5, 121.7), turned to 180 degrees
- moved C54 75.7 mm to (194.4, 97.3), turned to 0 degrees
- moved JP1 75.2 mm to (121.7, 118.7), turned to 180 degrees
- moved J3 72.6 mm to (204.2, 102.8), turned to 180 degrees
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Connections:
- ADC1 pad 10: GND* -> GND
- ADC1 pad 19: GND* -> GND
- ADC1 pad 20: GND* -> GND
- ADC1 pad 29: +3,3v* -> +3,3v
- ADC1 pad 3: GND* -> GND
- ADC1 pad 30: GND* -> GND
- ADC1 pad 35: GND* -> GND
- ADC1 pad 36: +3,3v* -> +3,3v
- ADC1 pad 5: +3,3v* -> +3,3v
- ADC1 pad 6: GND* -> GND
- ADC1 pad 9: GND* -> GND
- C13 pad 1: Net-(D4-K) -> Net-(Klem_dirty1-VIN)
- C14 pad 1: +14.4v* -> Net-(I3-IN+)
- C14 pad 2: GND* -> Net-(I3-IN-)
- C15 pad 1: Net-(I3-IN+) -> Net-(U4-BOOT)
- C15 pad 2: Net-(I3-IN-) -> Net-(D6-K)
- C16 pad 1: Net-(U4-BOOT) -> +5v
- C16 pad 2: Net-(D6-K) -> GND
- C17 pad 1: +5v -> GND
- C17 pad 2: GND -> Net-(JP3-A)
- C18 pad 2: Net-(JP3-A) -> Net-(DRV1-DVDD)
- C19 pad 2: Net-(DRV1-DVDD) -> Net-(DRV2-DVDD)
- C20 pad 2: Net-(DRV2-DVDD) -> Net-(DRV3-DVDD)
- C21 pad 1: GND -> Net-(DRV1-CPL)
- C21 pad 2: Net-(DRV3-DVDD) -> Net-(DRV1-CPH)
- C22 pad 1: Net-(DRV1-CPL) -> Net-(DRV2-CPL)
- C22 pad 2: Net-(DRV1-CPH) -> Net-(DRV2-CPH)
- C23 pad 1: Net-(DRV2-CPL) -> Net-(DRV3-CPL)
- C23 pad 2: Net-(DRV2-CPH) -> Net-(DRV3-CPH)
- C24 pad 1: Net-(DRV3-CPL) -> Net-(DRV1-VCP)
- C24 pad 2: Net-(DRV3-CPH) -> +14.4v
- C25 pad 1: Net-(DRV1-VCP) -> +14.4v
- C25 pad 2: +14.4v -> GND
- C26 pad 1: +14.4v -> Net-(DRV2-VCP)
- C26 pad 2: GND -> +14.4v
- C27 pad 1: Net-(DRV2-VCP) -> +14.4v
- C27 pad 2: +14.4v -> GND
- C28 pad 1: +14.4v -> Net-(DRV3-VCP)
- C28 pad 2: GND -> +14.4v
- C29 pad 1: Net-(DRV3-VCP) -> +14.4v
- C29 pad 2: +14.4v -> GND
- C3 pad 1: +5v* -> +5v
- C3 pad 2: GND* -> GND
- C30 pad 1: +14.4v -> GND
- C30 pad 2: GND -> +14.4v
- C36 pad 2: +14.4v -> Net-(DRV4-DVDD)
- C37 pad 2: Net-(DRV4-DVDD) -> Net-(DRV5-DVDD)
- C38 pad 2: Net-(DRV5-DVDD) -> Net-(DRV6-DVDD)
- C39 pad 1: GND -> Net-(DRV4-CPL)
- C39 pad 2: Net-(DRV6-DVDD) -> Net-(DRV4-CPH)
- C4 pad 1: +5v* -> +5v
- C4 pad 2: GND* -> GND
- C40 pad 1: Net-(DRV4-CPL) -> Net-(DRV5-CPL)
- C40 pad 2: Net-(DRV4-CPH) -> Net-(DRV5-CPH)
- C41 pad 1: Net-(DRV5-CPL) -> Net-(DRV6-CPL)
- C41 pad 2: Net-(DRV5-CPH) -> Net-(DRV6-CPH)
- C42 pad 1: Net-(DRV6-CPL) -> Net-(DRV4-VCP)
- C42 pad 2: Net-(DRV6-CPH) -> +14.4v
- C43 pad 1: Net-(DRV4-VCP) -> +14.4v
- C43 pad 2: +14.4v -> GND
- C44 pad 1: +14.4v -> Net-(DRV5-VCP)
- C44 pad 2: GND -> +14.4v
- C45 pad 1: Net-(DRV5-VCP) -> +14.4v
- C45 pad 2: +14.4v -> GND
- C46 pad 1: +14.4v -> Net-(DRV6-VCP)
- C46 pad 2: GND -> +14.4v
- C47 pad 1: Net-(DRV6-VCP) -> +14.4v
- C47 pad 2: +14.4v -> GND
- C48 pad 1: +14.4v -> GND
- C48 pad 2: GND -> +14.4v
- C5 pad 1: +3,3v* -> +3,3v
- C5 pad 2: GND* -> GND
- C54 pad 1: GND -> Net-(C54-Pad1)
- C54 pad 2: +14.4v -> GND
- C55 pad 1: Net-(C55-Pad1) -> +3,3v
- C55 pad 2: GND* -> GND
- C56 pad 1: +3,3v* -> +3,3v
- C56 pad 2: GND* -> GND
- C57 pad 1: +3,3v* -> +3,3v
- C57 pad 2: GND* -> GND
- C58 pad 1: +3,3v* -> +3,3v
- C58 pad 2: GND* -> GND
- C59 pad 1: +3,3v* -> Net-(ADC1-REFP)
- C59 pad 2: GND* -> GND
- C6 pad 1: +3,3v* -> +3,3v
- C6 pad 2: GND* -> GND
- C60 pad 1: Net-(ADC1-REFP) -> GND
- C60 pad 2: GND* -> +3,3v
- C61 pad 1: GND* -> GND
- C61 pad 2: +3,3v* -> Net-(ADC1-AINP)
- C7 pad 1: +5v* -> +5v
- C7 pad 2: GND* -> GND
- C8 pad 1: GND* -> GND
- D1 pad 1: GND* -> GND
- D2 pad 2: GND* -> GND
- D4 pad 2: +14.4v -> GND
- D5 pad 1: +14.4v* -> +14.4v
- D5 pad 2: GND* -> GND
- I1 pad 1: GND* -> GND
- I1 pad 2: GND* -> GND
- I1 pad 6: +5v* -> +5v
- I1 pad 7: GND* -> GND
- ISO1 pad 1: +3,3v* -> +3,3v
- ISO1 pad 8: GND* -> GND
- ISO2 pad 1: +3,3v* -> +3,3v
- ISO2 pad 8: GND* -> GND
- ISO3 pad 1: +3,3v* -> +3,3v
- ISO3 pad 8: GND* -> GND
- ISO4 pad 1: +3,3v* -> +3,3v
- ISO4 pad 8: GND* -> GND
- ISO5 pad 1: +3,3v* -> +3,3v
- ISO5 pad 8: GND* -> GND
- ISO6 pad 1: +3,3v* -> +3,3v
- ISO6 pad 8: GND* -> GND
- ISO7 pad 1: +3,3v* -> +3,3v
- ISO7 pad 8: GND* -> GND
- ISO8 pad 5: GND* -> GND
- ISO8 pad 8: +3,3v* -> +3,3v
- J3 pad 1: Net-(ISO7-INA) -> Net-(ISO8-SDA2)
- J3 pad 10: +3,3v* -> Net-(ISO7-OUTF)
- J3 pad 2: Net-(ISO7-INB) -> Net-(ISO7-INA)
- J3 pad 3: Net-(ISO7-INC) -> Net-(ISO8-SCL2)
- J3 pad 4: Net-(ISO7-IND) -> Net-(ISO7-INB)
- J3 pad 5: Net-(ISO8-SDA2) -> +5v
- J3 pad 6: Net-(ISO7-OUTF) -> Net-(ISO7-INC)
- J3 pad 7: Net-(ISO8-SCL2) -> +3,3v
- J3 pad 8: +5v* -> Net-(ISO7-IND)
- J3 pad 9: +5v -> GND
- Klem_dirty1 pad 1: Net-(D4-K) -> Net-(Klem_dirty1-VIN)
- L1 pad 2: +5v* -> +5v
- OPER1 pad 2: GND* -> GND
- OPER1 pad 5: +3,3v* -> +3,3v
- R1 pad 2: +14.4v* -> +14.4v
- R11 pad 1: Net-(U3-VSENSE) -> +14.4v
- R11 pad 2: GND -> Net-(D4-K)
- R12 pad 1: Net-(I3-IN+) -> Net-(U3-VSENSE)
- R12 pad 2: +14.4v -> GND
- R13 pad 1: +14.4v -> Net-(I3-IN+)
- R13 pad 2: Net-(JP3-A) -> +14.4v
- R14 pad 1: Net-(I3-IN-) -> +14.4v
- R15 pad 1: +5v -> Net-(I3-IN-)
- R15 pad 2: GND -> Net-(JP3-A)
- R16 pad 1: Net-(U4-VSENSE) -> +5v
- R17 pad 1: +3,3v -> Net-(U4-VSENSE)
- R17 pad 2: nFault_ISO -> GND
- R2 pad 1: +14.4v* -> +14.4v
- R23 pad 1: Net-(ADC1-REFP) -> +3,3v
- R23 pad 2: Net-(C55-Pad1) -> nFault_ISO
- R24 pad 1: Net-(OPER1--) -> Net-(ADC1-REFP)
- R24 pad 2: Net-(ADC1-AINP) -> Net-(C54-Pad1)
- R4 pad 1: +5v* -> +5v
- R5 pad 1: +5v* -> +5v
- R5 pad 2: GND* -> GND
- R6 pad 2: GND* -> GND
- REF1 pad 2: +3,3v* -> +3,3v
- REF1 pad 4: GND* -> GND
- U1 pad 1: +5v* -> +5v
- U1 pad 2: GND* -> GND
- U1 pad 4: +3,3v* -> +3,3v
- U1 pad 6: +5v* -> +5v
- U2 pad 6: GND* -> GND
- U2 pad 9: GND* -> GND
Routing:
- net +14.4v: track 444.8 -> 0.00 mm
- net +3,3v: track 307.8 -> 0.00 mm, vias 3 -> 0
- net +5v: track 243.5 -> 0.00 mm, vias 2 -> 0
- net +3,3v*: track 186.4 -> 0.00 mm, vias 4 -> 0
- net SCLK_ISO: track 153.1 -> 0.00 mm, vias 9 -> 0
- net SDI_ISO: track 152.3 -> 0.00 mm, vias 8 -> 0
- net nFault_ISO: track 150.6 -> 0.00 mm, vias 12 -> 0
- net SDO_ISO: track 132.3 -> 0.00 mm, vias 8 -> 0
- net SDA_INA: track 98.4 -> 0.00 mm, vias 5 -> 0
- net Net-(JP4-C): track 94.5 -> 0.00 mm
- net Net-(JP5-C): track 91.0 -> 0.00 mm
- net ENC_A_M2: track 90.3 -> 0.00 mm, vias 1 -> 0
- net GND*: track 88.7 -> 0.00 mm, vias 4 -> 0
- net SCL_INA: track 88.4 -> 0.00 mm, vias 4 -> 0
- net ENC_B_M2: track 83.6 -> 0.00 mm, vias 1 -> 0
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
Commit message: trassing
Parts:
- added XT60M1: Klem2, Connector_AMASS:AMASS_XT60-M_1x02_P7.20mm_Vertical, F.Cu at (97.8, 90.2)
- moved JP7 104.3 mm to (199.1, 118.9)
- moved JP9 104.3 mm to (199.2, 115.2)
- moved JP5 104.3 mm to (199.2, 122.5)
- moved JP4 103.2 mm to (199.2, 73.4)
- moved JP8 103.2 mm to (199.1, 80.7)
- moved JP6 103.2 mm to (199.2, 77.1)
- moved C17 43.4 mm to (121.5, 121.6)
- moved D6 43.4 mm to (122.8, 133.2)
- moved R13 43.4 mm to (113.2, 122.7)
- moved C14 43.4 mm to (115.7, 121.4)
- moved C15 43.4 mm to (118.1, 127.2)
- moved C16 43.4 mm to (133.6, 118.2)
- moved I3 43.4 mm to (115.9, 118.8)
- moved L3 43.4 mm to (131.3, 127.4)
- moved R14 43.4 mm to (115.7, 123.2)
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Routing:
- net +14.4v: track 0.00 -> 537.6 mm
- net +5v: track 0.00 -> 57.2 mm
- net GND: track 0.00 -> 48.2 mm
- net Net-(Klem_dirty1-VIN): track 0.00 -> 34.5 mm
- net Net-(D3-K): track 0.00 -> 26.7 mm
- net +3,3v: track 0.00 -> 25.1 mm
- net Net-(D2-K): track 0.00 -> 24.2 mm
- net Net-(JP3-A): track 0.00 -> 23.7 mm
- net Net-(D6-K): track 0.00 -> 23.6 mm
- net Net-(I3-Alert): track 0.00 -> 21.1 mm
- net CONN_2_M4: track 0.00 -> 18.0 mm, vias 0 -> 1
- net CONN_1_M6: track 0.00 -> 17.5 mm, vias 0 -> 1
- net CONN_1_M4: track 0.00 -> 16.8 mm, vias 0 -> 1
- net CONN_2_M6: track 0.00 -> 15.8 mm, vias 0 -> 1
- net ENA_U5: track 0.00 -> 15.0 mm
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