File: plat_power.kicad_pcb (KiCad board)
At the start: 2 copper layers, 133.8 x 103.9 mm, 165 parts, among them J1 Conn_01x18_Pin, J2 Conn_01x18_Pin, J3 Conn_01x10_Pin, U1 LD39050PU33R, U2 TPS5450, U3 TPS5450, U4 TPS5450

Commit message: I2C
Parts:
- moved ISO8 47.7 mm to (147.0, 97.8)
- moved C60 40.1 mm to (201.3, 95.0), turned to -90 degrees
- moved C61 36.3 mm to (198.4, 90.1), turned to 180 degrees
- moved R25 35.8 mm to (198.7, 91.9), turned to 180 degrees
- moved OPER1 35.0 mm to (198.8, 95.1), turned to -90 degrees
- moved C56 28.0 mm to (194.6, 100.2), turned to 0 degrees
- moved JP8 26.6 mm to (174.5, 70.6)
- moved JP6 26.6 mm to (174.6, 67.0)
- moved REF1 25.7 mm to (194.1, 95.7), turned to 90 degrees
- moved J2 25.2 mm to (184.0, 122.2), turned to 90 degrees
- moved J1 23.8 mm to (183.7, 75.3), turned to 90 degrees
- moved C59 19.6 mm to (189.7, 91.0), turned to 180 degrees
- moved JP7 19.3 mm to (183.0, 129.5)
- moved JP9 19.3 mm to (183.0, 125.8)
- moved JP5 19.3 mm to (183.0, 133.1)
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Connections:
- ISO7 pad 11: SDO_ISO -> CS_ISO
- ISO7 pad 12: unconnected-(ISO7-OUTD-Pad12) -> SDO_ISO
- ISO7 pad 13: CS_ISO -> SDI_ISO
- ISO7 pad 15: SDI_ISO -> unconnected-(ISO7-OUTA-Pad15)
- J1 pad 1: nSCS_mk_1 -> EN/IN1_mk_1
- J1 pad 11: ENC_A_M3_mk -> nSCS_mk_3
- J1 pad 12: ENC_B_M3_mk -> EN/IN1_mk_3
- J1 pad 13: nSCS_mk_5 -> EN/IN1_mk_5
- J1 pad 14: EN/IN1_mk_5 -> nSCS_mk_5
- J1 pad 15: PH/IN2_mk_5 -> DISABLE_mk_5
- J1 pad 16: DISABLE_mk_5 -> PH/IN2_mk_5
- J1 pad 17: ENC_A_M5_mk -> ENC_B_M5_mk
- J1 pad 18: ENC_B_M5_mk -> ENC_A_M5_mk
- J1 pad 2: EN/IN1_mk_1 -> nSCS_mk_1
- J1 pad 3: PH/IN2_mk_1 -> DISABLE_mk_1
- J1 pad 4: DISABLE_mk_1 -> PH/IN2_mk_1
- J1 pad 5: ENC_A_M1_mk -> ENC_B_M1_mk
- J1 pad 6: ENC_B_M1_mk -> ENC_A_M1_mk
- J1 pad 7: nSCS_mk_3 -> ENC_A_M3_mk
- J1 pad 8: EN/IN1_mk_3 -> ENC_B_M3_mk
- J2 pad 1: nSCS_mk_2 -> ENC_A_M2_mk
- J2 pad 10: DISABLE_mk_4 -> PH/IN2_mk_4
- J2 pad 11: ENC_A_M4_mk -> ENC_B_M4_mk
- J2 pad 12: ENC_B_M4_mk -> ENC_A_M4_mk
- J2 pad 13: nSCS_mk_6 -> EN/IN1_mk_6
- J2 pad 14: EN/IN1_mk_6 -> nSCS_mk_6
- J2 pad 15: PH/IN2_mk_6 -> DISABLE_mk_6
- J2 pad 16: DISABLE_mk_6 -> PH/IN2_mk_6
- J2 pad 17: ENC_A_M6_mk -> ENC_B_M6_mk
- J2 pad 18: ENC_B_M6_mk -> ENC_A_M6_mk
- J2 pad 2: EN/IN1_mk_2 -> ENC_B_M2_mk
- J2 pad 5: ENC_A_M2_mk -> nSCS_mk_2
- J2 pad 6: ENC_B_M2_mk -> EN/IN1_mk_2
- J2 pad 7: nSCS_mk_4 -> EN/IN1_mk_4
- J2 pad 8: EN/IN1_mk_4 -> nSCS_mk_4
- J2 pad 9: PH/IN2_mk_4 -> DISABLE_mk_4
Routing:
- net SCLK_ISO: track 0.00 -> 203.3 mm, vias 0 -> 7
- net SDI_ISO: track 0.00 -> 199.6 mm, vias 0 -> 7
- net SDO_ISO: track 0.00 -> 195.6 mm, vias 0 -> 7
- net nFault_ISO: track 0.00 -> 185.0 mm, vias 0 -> 9
- net ENC_A_M5_mk: track 0.00 -> 82.5 mm
- net PH/IN2_mk_5: track 0.00 -> 81.3 mm
- net nSCS_mk_5: track 0.00 -> 80.1 mm
- net ENC_B_M5_mk: track 0.00 -> 79.7 mm
- net ENC_B_M6_mk: track 0.00 -> 79.3 mm
- net DISABLE_mk_5: track 0.00 -> 78.5 mm
- net EN/IN1_mk_5: track 0.00 -> 77.3 mm
- net DISABLE_mk_6: track 0.00 -> 74.8 mm
- net ENC_A_M6_mk: track 0.00 -> 73.8 mm
- net EN/IN1_mk_6: track 0.00 -> 70.1 mm
- net PH/IN2_mk_6: track 0.00 -> 69.1 mm
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
Commit message: 3v3MK
Parts:
- moved JP9 92.2 mm to (91.0, 120.4)
- moved JP5 92.2 mm to (91.0, 127.7)
- moved JP7 92.2 mm to (91.0, 124.0)
- moved JP4 88.3 mm to (95.0, 66.1)
- moved JP6 79.5 mm to (95.1, 69.8)
- moved JP8 79.5 mm to (95.0, 73.4)
- moved C13 10.3 mm to (89.2, 115.1), turned to 0 degrees
- moved C55 5.38 mm to (194.8, 100.2)
- moved C56 5.20 mm to (189.6, 98.9)
- moved C57 2.73 mm to (188.2, 88.7), turned to 0 degrees
- moved C60 0.78 mm to (201.2, 95.8)
- moved ISO8 0.52 mm to (147.4, 98.1)
Connections:
- M_Con1 pad 3: CONN_1_M1 -> CONN_2_M1
- M_Con1 pad 4: CONN_2_M1 -> CONN_1_M1
- M_Con6 pad 3: CONN_1_M6 -> CONN_2_M6
- M_Con6 pad 4: CONN_2_M6 -> CONN_1_M6
Routing:
- net +3,3v: track 28.3 -> 442.4 mm, vias 0 -> 13
- net +5v: track 57.2 -> 220.9 mm, vias 0 -> 4
- net Net-(JP5-C): track 0.00 -> 110.2 mm
- net Net-(ISO8-SDA2): track 0.00 -> 105.0 mm, vias 0 -> 1
- net Net-(ISO8-SCL2): track 0.00 -> 101.9 mm, vias 0 -> 1
- net SDA_INA: track 0.00 -> 98.7 mm, vias 0 -> 4
- net Net-(JP4-C): track 0.00 -> 97.0 mm
- net GND: track 52.0 -> 143.0 mm
- net SCL_INA: track 0.00 -> 78.8 mm, vias 0 -> 4
- net ENC_B_M1: track 2.51 -> 69.5 mm
- net ENC_A_M2: track 7.99 -> 71.9 mm
- net ENC_A_M1: track 2.83 -> 66.7 mm
- net ENC_B_M2: track 7.99 -> 65.3 mm
- net Net-(JP7-C): track 0.00 -> 54.1 mm, vias 0 -> 2
- net CONN_1_M6: track 17.5 -> 66.2 mm
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