File: plat_power.kicad_sch (KiCad schematic)
At the start: 54 parts, among them U3 LD39050PU33R, U5 DG125-5.0-02P-14-00A(H)

Commit message: footprint, symbols kicad
Parts:
- removed U3: LD39050PU33R, symbol LD39050PU33R
- removed U5: DG125-5.0-02P-14-00A(H), symbol DG125-5.0-02P-14-00A(H)
- added Con1: DG125-5.0-02P-14-00A(H), TerminalBlock_Phoenix:TerminalBlock_Phoenix_MKDS-1,5-2_1x02_P5.00mm_Horizontal, symbol MyLIB:Con_power
- added D26: SS54L, Diode_SMD:D_0603_1608Metric, symbol SS54L
- added U1: LD39050PU33R, Package_DFN_QFN:DFN-6-1EP_3x3mm_P0.95mm_EP1.7x2.6mm, symbol MyLIB:LD39050PU33R
- added con2: (no value), Connector_PinHeader_1.00mm:PinHeader_1x04_P1.00mm_Horizontal, symbol MyLIB:Waga256_402
- C10, C12, C13, C14, C15, C16, C17, C18, C19, C20, C21, C22, C23, C24: footprint (none) -> Capacitor_SMD:C_0402_1005Metric
- C11, C60, C9: footprint (none) -> Capacitor_SMD:C_0603_1608Metric
- C62: value 2.2uF -> 4.7uF; footprint (none) -> Capacitor_SMD:C_1206_3216Metric
- D25, D28, D29, D30: footprint (none) -> Diode_SMD:D_0603_1608Metric
- I11, I2, I3: value (none) -> INA226; footprint (none) -> Package_SO:TSSOP-10_3x3mm_P0.5mm
- R14: footprint (none) -> Resistor_SMD:R_0805_2012Metric
- U10: value (none) -> KF33BD-TR; footprint (none) -> Package_SO:SOIC-8_3.9x4.9mm_P1.27mm
- U11, U12, U14: value (none) -> TPS5450; footprint (none) -> Package_SO:SOIC-8-1EP_3.9x4.9mm_P1.27mm_EP2.29x3mm
Connections:
- net +14.4v: now also D26.1 (K)
- net +3v3: now also U1.4 (VOUT)
- net +5v: now also U1.1 (EN), U1.6 (VIN)
- net GND: now also Con1.2, U1.2 (GND), U1.7 (GND), con2.3 (GND), con2.4 (GND)
- net at D25.2 (A): now also Con1.1
- new net: D26.2 (A), con2.1 (VIN), con2.2 (VIN)
- no-connect marks 3 -> 29
Other:
- moved on the sheet: R14

Commit message: Add files via upload
Parts:
- removed C45, C53, C58: C_US, symbol Device:C_US
- removed I11: INA226, Package_SO:TSSOP-10_3x3mm_P0.5mm, symbol MyLIB:INA226
- removed R62, R67: R, symbol Device:R
- added C1, C15, C42: 100nF, Capacitor_SMD:C_0603_1608Metric, symbol 0805_C9900012713_1
- added C26: 4.7uF, Capacitor_Tantalum_SMD:CP_EIA-7343-31_Kemet-D_HandSolder, symbol Device:C
- added C29, C8: 4.7uF, Capacitor_SMD:C_0603_1608Metric, symbol Device:C
- added I2: INA226, Package_SO:TSSOP-10_3x3mm_P0.5mm, symbol MyLIB:INA226
- added JP1, JP2, JP3: Jumper_3_Open, Jumper:SolderJumper-3_P1.3mm_Bridged123_Pad1.0x1.5mm, symbol Jumper:Jumper_3_Open
- added R1, R3, R33, R34, R7, R9: 1, Resistor_SMD:R_0603_1608Metric, symbol Device:R
- added R35, R8: 10m, Resistor_SMD:R_0805_2012Metric, symbol Device:R
- C10: renamed from C14; footprint Capacitor_SMD:C_0402_1005Metric -> Capacitor_SMD:C_0603_1608Metric
- C11: renamed from C15; footprint Capacitor_SMD:C_0402_1005Metric -> Capacitor_SMD:C_0603_1608Metric
- C12: renamed from C16; footprint Capacitor_SMD:C_0402_1005Metric -> Capacitor_SMD:C_1206_3216Metric
- C13: renamed from C62; footprint Capacitor_SMD:C_1206_3216Metric -> Capacitor_SMD:C_0603_1608Metric
- C16: renamed from C17; footprint Capacitor_SMD:C_0402_1005Metric -> Capacitor_SMD:C_0603_1608Metric
- C17: renamed from C18; footprint Capacitor_SMD:C_0402_1005Metric -> Capacitor_SMD:C_0603_1608Metric
- C18: renamed from C19; footprint Capacitor_SMD:C_0402_1005Metric -> Capacitor_SMD:C_0603_1608Metric
- C19: renamed from C20; footprint Capacitor_SMD:C_0402_1005Metric -> Capacitor_SMD:C_0603_1608Metric
- C2: renamed from C54; footprint (none) -> Capacitor_SMD:C_0603_1608Metric
- C20: renamed from C57; footprint (none) -> Capacitor_SMD:C_0603_1608Metric
- C21, C22, C24: footprint Capacitor_SMD:C_0402_1005Metric -> Capacitor_SMD:C_0603_1608Metric
- C23: footprint Capacitor_SMD:C_0402_1005Metric -> Capacitor_Tantalum_SMD:CP_EIA-7343-31_Kemet-D_HandSolder
- C25: renamed from C59; value C_US -> 330uF; footprint (none) -> Capacitor_Tantalum_SMD:CP_EIA-7343-31_Kemet-D_HandSolder
- C27: renamed from C55; footprint (none) -> Capacitor_SMD:C_0603_1608Metric
- C28: renamed from C56; value C_US -> 330uF; footprint (none) -> Capacitor_SMD:C_0603_1608Metric
- C4: renamed from C12; footprint Capacitor_SMD:C_0402_1005Metric -> Capacitor_SMD:C_0603_1608Metric
- C6: renamed from C10; footprint Capacitor_SMD:C_0402_1005Metric -> Capacitor_Tantalum_SMD:CP_EIA-7343-31_Kemet-D_HandSolder
- C7: renamed from C46; value C_US -> 330uF; footprint (none) -> Capacitor_Tantalum_SMD:CP_EIA-7343-31_Kemet-D_HandSolder
- C9: renamed from C13; footprint Capacitor_SMD:C_0402_1005Metric -> Capacitor_SMD:C_0603_1608Metric
- L1: renamed from L2; footprint Inductors:IND_0402 -> Inductor_SMD:L_12x12mm_H4.5mm
- L2: renamed from L10; footprint Inductors:IND_0402 -> Inductor_SMD:L_12x12mm_H4.5mm
- L3: footprint Inductors:IND_0402 -> Inductor_SMD:L_12x12mm_H4.5mm
- LED1: footprint (none) -> LED_SMD:LED_0603_1608Metric
- R10: renamed from R59; value R -> 10k; footprint (none) -> Resistor_SMD:R_0805_2012Metric
- R11: renamed from R58; value R -> 6.8K; footprint (none) -> Resistor_SMD:R_0805_2012Metric
- R13: renamed from R61; value R -> 10k; footprint (none) -> Resistor_SMD:R_0805_2012Metric
- R14: renamed from R60; value R -> 3.3k; footprint (none) -> Resistor_SMD:R_0805_2012Metric
- R2: renamed from R49; value R -> 10m; footprint (none) -> Resistor_SMD:R_0805_2012Metric
- R5: renamed from R57; value R -> 10k; footprint (none) -> Resistor_SMD:R_0805_2012Metric
- R6: renamed from R50; value R -> 3.3k; footprint (none) -> Resistor_SMD:R_0805_2012Metric
- con1: renamed from con2; value (none) -> KF202; footprint Connector_PinHeader_1.00mm:PinHeader_1x04_P1.00mm_Horizontal -> Library_footprints:con_klemnic
- renumbered C60 to C14, C11 to C3, C9 to C5, Con1 to Con2, D28 to D1, D30 to D2, D25 to D3, D26 to D4, D29 to D5, I2 to I1, R14 to R4, U11 to U2, U10 to U3, U12 to U4, U14 to U5
Connections:
- net +14.4v: now also R1.2, R34.2, R35.1, R7.2, R8.1; no longer I1.10 (IN+), I1.8 (VBUS), I1.9 (IN-), I3.10 (IN+), I3.8 (VBUS), I3.9 (IN-), R2.2, U2.7 (VIN), U4.7 (VIN), U5.7 (VIN)
- net +5v: now also I3.1 (A1), I2.2 (A0), I2.6 (VS)
- net GND: now also I1.1 (A1), I1.2 (A0), I3.2 (A0), con1.2 (GND), C26.1, C29.1, C8.1, I2.1 (A1), I2.7 (GND); no longer U1.7 (GND), con1.3 (GND), con1.4 (GND)
- net ENA_U2: now reaches U2.5 (ENA)
- net ENA_U2: now also JP1.3 (B)
- net at I1.3 (Alert): now also JP1.2 (C)
- net SDA_INA: now reaches I1.4 (SDA)
- net SDA_INA: now also I3.4 (SDA), I2.4 (SDA)
- net SCL_INA: now reaches I1.5 (SCL)
- net SCL_INA: now also I3.5 (SCL), I2.5 (SCL)
- net ENA_U5: now reaches U5.5 (ENA)
- net ENA_U5: now also JP3.3 (B)
- net at D4.2 (A), con1.1 (VIN): no longer con1.2 (VIN)
- net ENA_U4: now reaches U4.5 (ENA)
- net ENA_U4: now also JP2.3 (B)
- net at I3.3 (Alert): now also JP3.2 (C)
- new net: C26.2, JP2.1 (A), R8.2, R9.2, U4.7 (VIN)
- new net: I2.3 (Alert), JP2.2 (C)
- new net: C8.2, JP1.1 (A), R2.2, R3.2, U2.7 (VIN)
- new net: C1.1, I1.10 (IN+), R1.1
- new net: C1.2, I1.8 (VBUS), I1.9 (IN-), R3.1
- new net: C29.2, JP3.1 (A), R33.2, R35.2, U5.7 (VIN)
- new net: C15.1, I2.10 (IN+), R7.1
- new net: C15.2, I2.8 (VBUS), I2.9 (IN-), R9.1
- new net: C42.1, I3.10 (IN+), R34.1
- new net: C42.2, I3.8 (VBUS), I3.9 (IN-), R33.1
- no-connect marks 29 -> 10
Other:
- note added: "2) Добавить оптопары в разрыв ENC_A|B (гальваническая развязка) 1) Коннекторы. Проработать все лог. подключения 3) Разместить компонеты в редакторе плат 4) Прикинуть как дорожки будут идти"
- moved on the sheet: C2, C20, C25, C27, C28, C7, D1, D2, D5, I1, I3, L1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

Commit message: Add files via upload
Parts:
- removed C1, C15, C4, C42: 100nF, Capacitor_SMD:C_0603_1608Metric, symbol 0805_C9900012713_1
- removed C10: 100nF, Capacitor_SMD:C_0603_1608Metric, symbol 0805_C9900012713_14
- removed C11: 100nF, Capacitor_SMD:C_0603_1608Metric, symbol 0805_C9900012713_13
- removed C12: 100nF, Capacitor_SMD:C_1206_3216Metric, symbol 0805_C9900012713_12
- removed C13: 4.7uF, Capacitor_SMD:C_0603_1608Metric, symbol 0805_C9900012713_2
- removed C14: 0.1uF, Capacitor_SMD:C_0603_1608Metric, symbol 0805_C9900012713_2
- removed C16: 100nF, Capacitor_SMD:C_0603_1608Metric, symbol 0805_C9900012713_8
- removed C17: 100nF, Capacitor_SMD:C_0603_1608Metric, symbol 0805_C9900012713_9
- removed C18: 100nF, Capacitor_SMD:C_0603_1608Metric, symbol 0805_C9900012713_10
- removed C19: 100nF, Capacitor_SMD:C_0603_1608Metric, symbol 0805_C9900012713_11
- removed C21: 100nF, Capacitor_SMD:C_0603_1608Metric, symbol 0805_C9900012713_4
- removed C22: 100nF, Capacitor_SMD:C_0603_1608Metric, symbol 0805_C9900012713_5
- removed C23: 100nF, Capacitor_Tantalum_SMD:CP_EIA-7343-31_Kemet-D_HandSolder, symbol 0805_C9900012713_6
- removed C24: 100nF, Capacitor_SMD:C_0603_1608Metric, symbol 0805_C9900012713_7
- removed C3: 1uF, Capacitor_SMD:C_0603_1608Metric, symbol 0805_C9900012713
- removed C5: 1uF, Capacitor_SMD:C_0603_1608Metric, symbol 0805_C9900012713_2
- removed C6: 100nF, Capacitor_Tantalum_SMD:CP_EIA-7343-31_Kemet-D_HandSolder, symbol 0805_C9900012713_3
- removed C9: 100nF, Capacitor_SMD:C_0603_1608Metric, symbol 0805_C9900012713_15
- removed D1, D2, D5: BAS70, Diode_SMD:D_0603_1608Metric, symbol SS54L_19
- removed D3, D4: SS54L, Diode_SMD:D_0603_1608Metric, symbol SS54L
- removed L1, L2, L3: 10uH, Inductor_SMD:L_12x12mm_H4.5mm, symbol Tittar_kl:L
- removed LED1: Green, LED_SMD:LED_0603_1608Metric, symbol LED0805
- removed R4: 1K, Resistor_SMD:R_0805_2012Metric, symbol 0805
- added C1, C10, C11, C12, C15, C16, C17, C18, C19, C21, C22, C23, C24, C27, C4, C6, C9: 100nF, Capacitor_SMD:C_0603_1608Metric, symbol Device:C
- added C13: 4.7uF, Capacitor_SMD:C_0603_1608Metric, symbol Device:C
- added C14: 0.1uF, Capacitor_SMD:C_0603_1608Metric, symbol Device:C
- added C3, C5: 1uF, Capacitor_SMD:C_0603_1608Metric, symbol Device:C
- added Con1: (no value), Connector_PinHeader_1.00mm:PinHeader_1x02_P1.00mm_Vertical, symbol MyLIB:Con_power
- added D1: Green, LED_SMD:LED_0603_1608Metric, symbol Device:LED
- added D2, D3, D6: BAS70, Diode_SMD:D_0603_1608Metric, symbol Diode:PMEG60T30ELR
- added D4, D5: SS54L, Diode_SMD:D_0603_1608Metric, symbol Diode:PMEG60T30ELR
- added L1, L2, L3: 10uH, Inductor_SMD:L_12x12mm_H4.5mm, symbol Device:L
- added R4: 1k, Resistor_SMD:R_0805_2012Metric, symbol Device:R
- renumbered C27 to C28, C28 to C29, C29 to C30, Con2 to Con3, R34 to R12, R35 to R13, R33 to R14, R13 to R15, R14 to R16, con1 to con2
Connections:
- net +14.4v: now also D4.1 (K), D5.1 (K)
- net +3v3: now also C13.1, L2.2; no longer U1.4 (VOUT)
- net +5v: now also C14.1, C3.1, C4.1, L1.2, L3.2, R4.1
- net GND: now also C10.2, C11.2, C12.2, C13.2, C14.2, C16.2, C17.2, C18.2, C19.2, C21.2, C22.2, C23.2, C24.2, C3.2, C4.2, C5.2, C6.2, C9.2, Con1.2, D1.1 (K), D2.2 (A), D3.2 (A), D6.2 (A)
- net VDD: now also C10.1, C11.1, C12.1, C16.1, C17.1, C18.1, C19.1, C21.1, C22.1, C23.1, C24.1, C9.1
- net at C28.2, U5.8 (PH): now also D6.1 (K), L3.1
- net at C2.2, U2.8 (PH): now also D2.1 (K), L1.1
- net at I1.10 (IN+), R1.1: now also C1.1
- net at I1.8 (VBUS), I1.9 (IN-), R3.1: now also C1.2
- net at C20.2, U4.8 (PH): now also D3.1 (K), L2.1
- net at I2.10 (IN+), R7.1: now also C15.1
- net at I2.8 (VBUS), I2.9 (IN-), R9.1: now also C15.2
- net at con2.1 (VIN): now also D5.2 (A)
- net at Con3.1: now also D4.2 (A)
- net at I3.10 (IN+), R12.1: now also C27.1
- net at I3.8 (VBUS), I3.9 (IN-), R14.1: now also C27.2
- new net: C5.1, C6.1, Con1.1, U1.4 (VOUT)
- new net: D1.2 (A), R4.2
- no-connect marks 10 -> 11
Other:
- note added: "1) Разместить компонеты в редакторе плат 2) Прикинуть как дорожки будут идти"
- note added: "Питание на логическую плату"
- note removed: "2) Добавить оптопары в разрыв ENC_A|B (гальваническая развязка) 1) Коннекторы. Проработать все лог. подключения 3) Разместить компонеты в редакторе плат 4) Прикинуть как дорожки будут идти"

Commit message: Add files via upload
Connections:
- net GND: now also U2.9 (GND), U4.9 (GND), U5.9 (GND)
- net +3v3 renamed +3,3v

Commit message: Add files via upload
Parts:
- C26: footprint Capacitor_Tantalum_SMD:CP_EIA-7343-31_Kemet-D_HandSolder -> Capacitor_SMD:C_0603_1608Metric
- C29: footprint Capacitor_SMD:C_0603_1608Metric -> Capacitor_Tantalum_SMD:CP_EIA-7343-31_Kemet-D_HandSolder
Connections:
- net GND: now also R10.2, R11.1, R15.2, R16.1, U4.4 (VSENSE), U5.4 (VSENSE)
Other:
- moved on the sheet: R3

Commit message: Add files via upload
Parts:
- removed C13: 4.7uF, Capacitor_SMD:C_0603_1608Metric, symbol Device:C
- removed C14: 0.1uF, Capacitor_SMD:C_0603_1608Metric, symbol Device:C
- removed U3: KF33BD-TR, Package_SO:SOIC-8_3.9x4.9mm_P1.27mm, symbol MyLIB:KF33BD-TR
Connections:
- no-connect marks 11 -> 9
Other:
- note removed: "Оставить LD39050 или KF33DB-TR"

Commit message: Add files via upload
Parts:
- removed C10, C11, C12, C16, C17, C18, C19, C23, C24, C9: 100nF, Capacitor_SMD:C_0603_1608Metric, symbol Device:C
- D4: renamed from D5; footprint Diode_SMD:D_0603_1608Metric -> Diode_SMD:D_SMC
- D5: renamed from D4; footprint Diode_SMD:D_0603_1608Metric -> Diode_SMD:D_SMC
- renumbered C20 to C10, C25 to C11, C26 to C12, C22 to C13, C21 to C14, C27 to C15, C28 to C16, C29 to C17, C30 to C18, C15 to C9, Con3 to Con2, U4 to U3, U5 to U4, con2 to con3
Connections:
- net +14.4v: now also C14.1, Con2.1, D4.2 (A); no longer D4.1 (K)
- net GND: now also D5.2 (A)
- net at con3.1 (VIN): now also C13.1, D4.1 (K); no longer D4.2 (A)
- removed net VDD: C13.1, C14.1
Other:
- note added: "Diode_SMD:D_SMC (done) Connector_PinHeader_2.54mm:PinHeader_1x05_P2.54mm_Vertical (J1-J6) (done) Arduino_UNO_R2 - для примерки (done)"
- note removed: "1) Разместить компонеты в редакторе плат 2) Прикинуть как дорожки будут идти"
- moved on the sheet: C13, C14, Con2, D4, D5

Commit message: Add files via upload
Parts:
- removed Con1: (no value), Connector_PinHeader_1.00mm:PinHeader_1x02_P1.00mm_Vertical, symbol MyLIB:Con_power
- added con1: (no value), Connector_PinHeader_1.00mm:PinHeader_1x03_P1.00mm_Vertical, symbol MyLIB:con_3
Connections:
- net +5v: now also con1.2
- net GND: now also con1.1
- net at C5.1, C6.1, U1.4 (VOUT): now also con1.3
