File: plat_power.kicad_sch (KiCad schematic)
At the start: 56 parts, among them Con2 DG125-5.0-02P-14-00A(H), U1 LD39050PU33R, U2 TPS5450, U3 TPS5450, U4 TPS5450, con3 KF202

Commit message: Add files via upload
Parts:
- con1: footprint Connector_PinHeader_1.00mm:PinHeader_1x03_P1.00mm_Vertical -> Connector_PinHeader_2.54mm:PinHeader_1x03_P2.54mm_Vertical
Other:
- note added: "Diode_SMD:D_SMC (done)"
- note removed: "Diode_SMD:D_SMC (done) Connector_PinHeader_2.54mm:PinHeader_1x05_P2.54mm_Vertical (J1-J6) (done) Arduino_UNO_R2 - для примерки (done)"
Changed lines of the file:
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@@
 		)
 	)
-	(text "Diode_SMD:D_SMC (done)\n\nConnector_PinHeader_2.54mm:PinHeader_1x05_P2.54mm_Vertical (J1-J6) (done)\n\nArduino_UNO_R2 - для примерки (done)"
+	(text "Diode_SMD:D_SMC (done)\n"
 		(exclude_from_sim no)
 		(at 323.85 228.092 0)
@@
 			)
 		)
-		(property "Footprint" "Connector_PinHeader_1.00mm:PinHeader_1x03_P1.00mm_Vertical"
+		(property "Footprint" "Connector_PinHeader_2.54mm:PinHeader_1x03_P2.54mm_Vertical"
 			(at 261.62 53.34 0)
 			(hide yes)

Commit message: trass
Parts:
- added Con2, Con5: (no value), Connector_PinHeader_2.54mm:PinHeader_1x02_P2.54mm_Vertical, symbol MyLIB:Con_power
- added U3: ISO1540, Package_SO:SOIC-8_3.9x4.9mm_P1.27mm, symbol Isolator:ISO1540
- C12, C18, C8: footprint Capacitor_SMD:C_0603_1608Metric -> Capacitor_SMD:C_1206_3216Metric
- JP1, JP2, JP3: footprint Jumper:SolderJumper-3_P1.3mm_Bridged123_Pad1.0x1.5mm -> Connector_PinHeader_2.54mm:PinHeader_1x03_P2.54mm_Vertical
- renumbered Con2 to Con3, U3 to U4, U4 to U5, con3 to con4
Connections:
- net +14.4v: no longer C14.1, Con3.1, D5.1 (K), R1.2, R2.1
- net +3,3v: now also U3.1 (VCC1)
- net +5v: now also Con5.1; no longer C3.1, C4.1, C7.1, I1.6 (VS), L1.2, R4.1, R5.1, U1.1 (EN), U1.6 (VIN), con1.2
- net GND: now also Con5.2, U3.4 (GND1); no longer C14.2, C3.2, C4.2, C5.2, C6.2, C7.2, C8.1, Con3.2, D1.1 (K), D2.2 (A), D5.2 (A), I1.1 (A1), I1.2 (A0), I1.7 (GND), R11.1, R16.1, R5.2, R6.1, R6.2, U1.2 (GND), U2.4 (VSENSE), U2.6 (GND), U2.9 (GND), U4.4 (VSENSE), U5.4 (VSENSE), con1.1
- net SCL_INA: now also U3.3 (SCL1)
- net SDA_INA: now also U3.2 (SDA1)
- net +3,3v*: now reaches C5.1, C6.1, U1.4 (VOUT)
- net +3,3v*: now also con1.2, U3.8 (VCC2); no longer con1.3
- new net: R6.1, U2.4 (VSENSE)
- new net: R16.1, U5.4 (VSENSE)
- new net: R11.1, U4.4 (VSENSE)
- new net: Con2.2, U3.6 (SCL2)
- new net: Con2.1, U3.7 (SDA2)
- new net +14.4v*: C14.1, Con3.1, D5.1 (K), R1.2, R2.1
- new net +5v*: C3.1, C4.1, C7.1, I1.6 (VS), L1.2, R4.1, R5.1, U1.1 (EN), U1.6 (VIN), con1.3
- new net GND*: C14.2, C3.2, C4.2, C5.2, C6.2, C7.2, C8.1, Con3.2, D1.1 (K), D2.2 (A), D5.2 (A), I1.1 (A1), I1.2 (A0), I1.7 (GND), R5.2, R6.2, U1.2 (GND), U2.6 (GND), U2.9 (GND), U3.5 (GND2), con1.1
Other:
- note removed: "Diode_SMD:D_SMC (done)"

Commit message: tray
Parts:
- removed Con2, Con5: (no value), Connector_PinHeader_2.54mm:PinHeader_1x02_P2.54mm_Vertical, symbol MyLIB:Con_power
- removed U3: ISO1540, Package_SO:SOIC-8_3.9x4.9mm_P1.27mm, symbol Isolator:ISO1540
- removed con1: (no value), Connector_PinHeader_2.54mm:PinHeader_1x03_P2.54mm_Vertical, symbol MyLIB:con_3
- renumbered Con3 to Klem_clear1, con4 to Klem_dirty1, U4 to U3, U5 to U4
Other:
- note removed: "Питание на логическую плату"

Commit message: trass
Parts:
- removed C14: 100nF, Capacitor_SMD:C_0603_1608Metric, symbol Device:C
- removed D5: SS54L, Diode_SMD:D_SMC, symbol Diode:PMEG60T30ELR
- removed Klem_clear1: DG125-5.0-02P-14-00A(H), TerminalBlock_Phoenix:TerminalBlock_Phoenix_MKDS-1,5-2_1x02_P5.00mm_Horizontal, symbol MyLIB:Con_power
- added D4: Green, LED_SMD:LED_0603_1608Metric, symbol Device:LED
- added F1: Fuse, Fuseholder_Clip-5x20mm_Bel_FC-203-22_Lateral_P17.80x5.00mm_D1.17mm_Horizontal, symbol Device:Fuse
- added R11: 2.2k, Resistor_SMD:R_0603_1608Metric, symbol Device:R
- renumbered C15 to C14, C16 to C15, C17 to C16, C18 to C17, D4 to D5, R11 to R12, R12 to R13, R13 to R14, R14 to R15, R15 to R16, R16 to R17
Connections:
- net +14.4v* is gone; now on net +14.4v: R1.2, R2.1
- net +3,3v* is gone; now on net +3,3v: C5.1, C6.1, U1.4 (VOUT)
- net +5v* is gone; now on net +5v: C3.1, C4.1, C7.1, I1.6 (VS), L1.2, R4.1, R5.1, U1.1 (EN), U1.6 (VIN)
- net GND* is gone; now on net GND: C3.2, C4.2, C5.2, C6.2, C7.2, C8.1, D1.1 (K), D2.2 (A), I1.1 (A1), I1.2 (A0), I1.7 (GND), R5.2, R6.2, U1.2 (GND), U2.6 (GND), U2.9 (GND)
- net +14.4v: now also D5.1 (K), F1.1, R11.1; no longer D5.2 (A)
- net GND: now also D5.2 (A), D4.2 (A)
- net at C13.1, Klem_dirty1.1 (VIN): now also F1.2; no longer D5.1 (K)
- new net: D4.1 (K), R11.2
Other:
- moved on the sheet: D5

Commit message: trassing
Parts:
- added XT60M1: Klem2, Connector_AMASS:AMASS_XT60-M_1x02_P7.20mm_Vertical, symbol Connector:Conn_01x02_Pin
Connections:
- net GND: now also XT60M1.2 (Pin_2)
- net at C13.1, F1.2, Klem_dirty1.1 (VIN): now also XT60M1.1 (Pin_1)
Changed lines of the file:
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@@
 	)
 	(junction
+		(at 297.18 198.12)
+		(diameter 0)
+		(color 0 0 0 0)
+	)
+	(junction
 		(at 86.36 33.02)
 		(diameter 0)
@@
 	)
 	(junction
+		(at 316.23 198.12)
+		(diameter 0)
+		(color 0 0 0 0)
+	)
+	(junction
 		(at 114.3 115.57)
 		(diameter 0)
@@
 	(wire
 		(pts
+			(xy 294.64 204.47) (xy 297.18 204.47)
+		)
+		(stroke
+			(width 0)
+			(type default)
+		)
+	)
+	(wire
+		(pts
 			(xy 96.52 109.22) (xy 96.52 105.41)
 		)
@@
 	(wire
 		(pts
-			(xy 293.37 198.12) (xy 299.72 198.12)
+			(xy 293.37 198.12) (xy 297.18 198.12)
 		)
 		(stroke
@@
 	(wire
 		(pts
+			(xy 297.18 204.47) (xy 297.18 198.12)
+		)
+		(stroke
+			(width 0)
+			(type default)
+		)
+	)
+	(wire
+		(pts
 			(xy 111.76 20.32) (xy 111.76 25.4)
 		)
@@
 	(wire
 		(pts
+			(xy 294.64 207.01) (xy 316.23 207.01)
+		)
+		(stroke
+			(width 0)
+			(type default)
+		)
+	)
+	(wire
+		(pts
 			(xy 132.08 63.5) (xy 138.43 63.5)
 		)
@@
 	(wire
 		(pts
+			(xy 316.23 207.01) (xy 316.23 198.12)
+		)
+		(stroke
+			(width 0)
+			(type default)
+		)
+	)
+	(wire
+		(pts
 			(xy 73.66 158.75) (xy 71.12 158.75)
 		)
@@
 	(wire
 		(pts
+			(xy 316.23 198.12) (xy 318.77 198.12)
+		)
+		(stroke
+			(width 0)
+			(type default)
+		)
+	)
+	(wire
+		(pts
 			(xy 43.18 203.2) (xy 43.18 207.01)
 		)
@@
 	(wire
 		(pts
-			(xy 314.96 198.12) (xy 318.77 198.12)
+			(xy 314.96 198.12) (xy 316.23 198.12)
 		)
 		(stroke
@@
 	(wire
 		(pts
+			(xy 297.18 198.12) (xy 299.72 198.12)
+		)
+		(stroke
+			(width 0)
+			(type default)
+		)
+	)
+	(wire
+		(pts
 			(xy 114.3 130.81) (xy 114.3 143.51)
 		)
@@
 					(unit 1)
 				)
+			)
+		)
+	)
+	(symbol
+		(lib_id "Connector:Conn_01x02_Pin")
+		(at 289.56 204.47 0)
+		(unit 1)
+		(body_style 1)
+		(exclude_from_sim no)
+		(in_bom yes)
+		(on_board yes)
+		(in_pos_files yes)
+		(dnp no)
+		(property "Reference" "XT60M1"
+			(at 285.75 204.47 0)
+			(show_name no)
+			(do_not_autoplace no)
+			(effects
+				(font
+					(size 1.27 1.27)
+				)
+			)
+		)
+		(property "Value" "Klem2"
+			(at 286.004 206.502 0)
+			(show_name no)
+			(do_not_autoplace no)
+			(effects
+				(font
+					(size 1.27 1.27)
+				)
+			)
+		)
+		(property "Footprint" "Connector_AMASS:AMASS_XT60-M_1x02_P7.20mm_Vertical"
+			(at 289.56 204.47 0)
+			(hide yes)
+			(show_name no)
+			(do_not_autoplace no)
+			(effects
+				(font
+					(size 1.27 1.27)
+				)
+			)
+		)
+		(property "Datasheet" ""
+			(at 289.56 204.47 0)
+			(hide yes)
+			(show_name no)
+			(do_not_autoplace no)
+			(effects
+				(font
+					(size 1.27 1.27)
+				)
+			)
+		)
+		(property "Description" "Generic connector, single row, 01x02, script generated"
+			(at 289.56 204.47 0)
+			(hide yes)
+			(show_name no)
+			(do_not_autoplace no)
+			(effects
+				(font
+					(size 1.27 1.27)
+				)
+			)
+		)
+		(pin "1"
+		)
+		(pin "2"
+		)
+		(instances
+			(project "plat_power"
+				(path "/d8484589-1448-4c11-9029-5047a0584288"
+					(reference "XT60M1")
+					(unit 1)
+				)
