File: motor_control.kicad_sch (KiCad schematic)
At the start: 75 parts, among them U6 DRV8873SPWPR, U7 TB67H451FNG,EL, U8 DRV8231DDAR

Commit message: footprint, symbols kicad
Parts:
- removed DRV1: MC33886PVW, symbol MC33886PVW
- removed DRV2: MC33886PVW, symbol MC33886PVW_2
- removed DRV3: MC33886PVW, symbol MC33886PVW_1
- removed DRV4: MC33886PVW, symbol MC33886PVW_3
- removed DRV5: MC33886PVW, symbol MC33886PVW_4
- removed DRV6: MC33886PVW, symbol MC33886PVW_5
- added DRV1, DRV2, DRV3, DRV4, DRV5, DRV7: MC33886PVW, Package_SO:HSOP-20-1EP_11.0x15.9mm_P1.27mm_SlugDown, symbol MyLIB:Driver
- added M_Con1, M_Con2, M_Con3, M_Con4, M_Con5, M_Con6: ZX-PH2.0-6PWZ-Y, Connector_PinHeader_2.00mm:PinHeader_1x06_P2.00mm_Vertical, symbol MyLIB:motor_con
- C25, C26, C29, C30, C35, C36: footprint (none) -> Capacitor_SMD:C_0402_1005Metric
- C27, C28, C31, C32, C37, C38: value 33nF -> 100nF; footprint (none) -> Capacitor_SMD:C_0402_1005Metric
- C3_TANTAL1, C4_TANTAL1, C5_TANTAL1, C6_TANTAL1, C8_TANTAL1, C9_TANTAL1: footprint (none) -> Capacitor_SMD:C_0603_1608Metric
- D1, D10, D11, D12, D13, D14, D15, D16, D17, D18, D19, D2, D20, D21, D22, D23, D24, D3, D4, D5, D6, D7, D8, D9: footprint (none) -> Diode_SMD:D_0603_1608Metric
- I10, I5, I6, I7, I8, I9: value (none) -> INA226; footprint (none) -> Package_SO:TSSOP-10_3x3mm_P0.5mm
- R17, R18, R21, R22, R37, R38: footprint (none) -> Resistor_SMD:R_0805_2012Metric
Connections:
- net +14.4v: now also DRV1.16 (V+), DRV1.4 (V+), DRV1.5 (V+), DRV2.16 (V+), DRV2.4 (V+), DRV2.5 (V+), DRV3.16 (V+), DRV3.4 (V+), DRV3.5 (V+), DRV4.16 (V+), DRV4.4 (V+), DRV4.5 (V+), DRV5.16 (V+), DRV5.4 (V+), DRV5.5 (V+), DRV7.16 (V+), DRV7.4 (V+), DRV7.5 (V+), M_Con1.3, M_Con2.3, M_Con3.3, M_Con4.3, M_Con5.3, M_Con6.3
- net +5v: now also DRV1.13 (D2#), DRV2.13 (D2#), DRV3.13 (D2#), DRV4.13 (D2#), DRV5.13 (D2#), DRV7.13 (D2#)
- net CONN_M1_1: now also DRV7.6 (OUT1), DRV7.7 (OUT1), M_Con1.2
- net CONN_M1_2: now also DRV7.14 (OUT2), DRV7.15 (OUT2), M_Con1.1
- net CONN_M2_1: now also DRV1.6 (OUT1), DRV1.7 (OUT1), M_Con2.2
- net CONN_M2_2: now also DRV1.14 (OUT2), DRV1.15 (OUT2), M_Con2.1
- net CONN_M3_1: now also DRV2.6 (OUT1), DRV2.7 (OUT1), M_Con3.2
- net CONN_M3_2: now also DRV2.14 (OUT2), DRV2.15 (OUT2), M_Con3.1
- net CONN_M4_1: now also DRV3.6 (OUT1), DRV3.7 (OUT1), M_Con4.2
- net CONN_M4_2: now also DRV3.14 (OUT2), DRV3.15 (OUT2), M_Con4.1
- net CONN_M5_1: now also DRV4.6 (OUT1), DRV4.7 (OUT1), M_Con5.2
- net CONN_M5_2: now also DRV4.14 (OUT2), DRV4.15 (OUT2), M_Con5.1
- net CONN_M6_1: now also DRV5.6 (OUT1), DRV5.7 (OUT1), M_Con6.2
- net CONN_M6_2: now also DRV5.14 (OUT2), DRV5.15 (OUT2), M_Con6.1
- net GND: now also DRV1.1 (AGND), DRV1.10 (PGND), DRV1.11 (PGND), DRV1.12 (PGND), DRV1.18 (D1), DRV1.9 (PGND), DRV2.1 (AGND), DRV2.10 (PGND), DRV2.11 (PGND), DRV2.12 (PGND), DRV2.18 (D1), DRV2.9 (PGND), DRV3.1 (AGND), DRV3.10 (PGND), DRV3.11 (PGND), DRV3.12 (PGND), DRV3.18 (D1), DRV3.9 (PGND), DRV4.1 (AGND), DRV4.10 (PGND), DRV4.11 (PGND), DRV4.12 (PGND), DRV4.18 (D1), DRV4.9 (PGND), DRV5.1 (AGND), DRV5.10 (PGND), DRV5.11 (PGND), DRV5.12 (PGND), DRV5.18 (D1), DRV5.9 (PGND), DRV7.1 (AGND), DRV7.10 (PGND), DRV7.11 (PGND), DRV7.12 (PGND), DRV7.18 (D1), DRV7.9 (PGND), M_Con1.6, M_Con2.6, M_Con3.6, M_Con4.6, M_Con5.6, M_Con6.6
- net IN1_M1: now also DRV7.3 (IN1)
- net IN1_M2: now also DRV1.3 (IN1)
- net IN1_M3: now also DRV2.3 (IN1)
- net IN1_M4: now also DRV3.3 (IN1)
- net IN1_M5: now also DRV4.3 (IN1)
- net IN1_M6: now also DRV5.3 (IN1)
- net IN2_M1: now also DRV7.19 (IN2)
- net IN2_M2: now also DRV1.19 (IN2)
- net IN2_M3: now also DRV2.19 (IN2)
- net IN2_M4: now also DRV3.19 (IN2)
- net IN2_M5: now also DRV4.19 (IN2)
- net IN2_M6: now also DRV5.19 (IN2)
- net at C38.2: now also DRV5.17 (CCP)
- net at R19.2, R21.2: now also DRV4.2 (FS#)
- net at R35.2, R37.2: now also DRV2.2 (FS#)
- net at C37.2: now also DRV2.17 (CCP)
- net at C28.2: now also DRV7.17 (CCP)
- net at R15.2, R17.2: now also DRV3.2 (FS#)
- net at R36.2, R38.2: now also DRV5.2 (FS#)
- net at R20.2, R22.2: now also DRV1.2 (FS#)
- net at R16.2, R18.2: now also DRV7.2 (FS#)
- net at C31.2: now also DRV4.17 (CCP)
- net at C32.2: now also DRV1.17 (CCP)
- net at C27.2: now also DRV3.17 (CCP)
- new net ENC_A_M1: M_Con1.5
- new net ENC_A_M2: M_Con2.5
- new net ENC_A_M3: M_Con3.5
- new net ENC_A_M4: M_Con4.5
- new net ENC_A_M5: M_Con5.5
- new net ENC_A_M6: M_Con6.5
- new net ENC_B_M1: M_Con1.4
- new net ENC_B_M2: M_Con2.4
- new net ENC_B_M3: M_Con3.4
- new net ENC_B_M4: M_Con4.4
- new net ENC_B_M5: M_Con5.4
- new net ENC_B_M6: M_Con6.4
- no-connect marks 12 -> 48
Other:
- moved on the sheet: U6, U7, U8

Commit message: Add files via upload
Parts:
- removed I6, I7, I8, I9: INA226, Package_SO:TSSOP-10_3x3mm_P0.5mm, symbol MyLIB:INA226
- removed R15: 0, symbol R_0603_EU_3
- removed R16: 0, symbol R_0603_EU
- removed R19: 0, symbol R_0603_EU_4
- removed R20: 0, symbol R_0603_EU_2
- removed R35: 0, symbol R_0603_EU_1
- removed R36: 0, symbol R_0603_EU_5
- removed R68, R69, R70, R71, R72, R73: R, symbol Device:R
- removed U6: DRV8873SPWPR, symbol DRV8873SPWPR
- removed U7: TB67H451FNG,EL, symbol TB67H451FNG,EL
- removed U8: DRV8231DDAR, symbol DRV8231DDAR
- added C43, C44, C45, C46, C47, C48: 100nF, Capacitor_SMD:C_0603_1608Metric, symbol 0805_C9900012713_1
- added I11, I12, I13, I14: INA226, Package_SO:TSSOP-10_3x3mm_P0.5mm, symbol MyLIB:INA226
- added JP4: Jumper_3_Open, Jumper:SolderJumper-3_P1.3mm_Bridged123_Pad1.0x1.5mm, symbol Jumper:Jumper_3_Open
- added R12, R32, R36, R40, R43, R44, R47, R48, R51, R52, R55, R56: 1, Resistor_SMD:R_0603_1608Metric, symbol Device:R
- added R18, R19: 1k, Resistor_SMD:R_0805_2012Metric, symbol 0805_1
- added R37, R41, R45, R49, R53, R57: 10m, Resistor_SMD:R_0805_2012Metric, symbol Device:R
- added R38, R39, R42, R46, R50, R54, R58, R59: 10k, Resistor_SMD:R_0805_2012Metric, symbol 0805
- added U7, U8: PC817, Package_DIP:DIP-4_W7.62mm_SMDSocket_SmallPads, symbol Isolator:PC817
- C30: renamed from C32; footprint Capacitor_SMD:C_0402_1005Metric -> Capacitor_SMD:C_0603_1608Metric
- C31: renamed from C37; footprint Capacitor_SMD:C_0402_1005Metric -> Capacitor_SMD:C_0603_1608Metric
- C32: renamed from C28; footprint Capacitor_SMD:C_0402_1005Metric -> Capacitor_SMD:C_0603_1608Metric
- C33: renamed from C29; footprint Capacitor_SMD:C_0402_1005Metric -> Capacitor_SMD:C_0603_1608Metric
- C34: renamed from C36; footprint Capacitor_SMD:C_0402_1005Metric -> Capacitor_SMD:C_0603_1608Metric
- C35: renamed from C26; footprint Capacitor_SMD:C_0402_1005Metric -> Capacitor_SMD:C_0603_1608Metric
- C36: renamed from C31; footprint Capacitor_SMD:C_0402_1005Metric -> Capacitor_SMD:C_0603_1608Metric
- C37: renamed from C38; footprint Capacitor_SMD:C_0402_1005Metric -> Capacitor_SMD:C_0603_1608Metric
- C38: renamed from C27; footprint Capacitor_SMD:C_0402_1005Metric -> Capacitor_SMD:C_0603_1608Metric
- C39: renamed from C35; footprint Capacitor_SMD:C_0402_1005Metric -> Capacitor_SMD:C_0603_1608Metric
- C40: renamed from C30; footprint Capacitor_SMD:C_0402_1005Metric -> Capacitor_SMD:C_1206_3216Metric
- C41: renamed from C25; footprint Capacitor_SMD:C_0402_1005Metric -> Capacitor_SMD:C_1206_3216Metric
- renumbered D17 to D10, D19 to D11, D21 to D12, D23 to D13, D1 to D14, D3 to D15, D5 to D16, D7 to D17, D10 to D18, D12 to D19, D14 to D20, D16 to D21, D18 to D22, D20 to D23, D22 to D24, D24 to D25, D2 to D26, D4 to D27, D6 to D28, D8 to D29, D9 to D6, D11 to D7, D13 to D8, D15 to D9, DRV7 to DRV3, DRV3 to DRV6, I5 to I8, R22 to R15, R37 to R16, R18 to R17, R38 to R22, R17 to R23
Connections:
- net +14.4v: now also R12.2, R32.2, R36.2, R37.1, R37.2, R40.2, R41.1, R41.2, R43.2, R44.2, R45.1, R45.2, R47.2, R48.2, R49.1, R49.2, R51.2, R52.2, R53.1, R53.2, R55.2, R56.2, R57.1, R57.2; no longer I10.10 (IN+), I10.8 (VBUS), I10.9 (IN-), I8.10 (IN+), I8.8 (VBUS), I8.9 (IN-), M_Con1.3
- net +5v: now also I8.1 (A1), I8.2 (A0), I11.6 (VS), I12.1 (A1), I12.6 (VS), I13.1 (A1), I13.6 (VS), I14.2 (A0), I14.6 (VS), JP4.1 (A), R38.1, R39.1, R42.1, R46.1, R50.1, R54.1, U7.4, U8.4; no longer DRV1.13 (D2#), DRV2.13 (D2#), DRV3.13 (D2#), DRV4.13 (D2#), DRV5.13 (D2#), DRV6.13 (D2#)
- net ENC_A_M1: now also R59.1, U8.3
- net ENC_B_M1: now also R58.1, U7.3
- net FS1: now also DRV3.2 (FS#), R17.2
- net GND: now also I10.1 (A1), I11.1 (A1), I11.7 (GND), I12.7 (GND), I13.7 (GND), I14.7 (GND), R58.2, R59.2, U7.2, U8.2
- net FS5: now reaches DRV4.2 (FS#), R21.2
- net FS3: now reaches DRV2.2 (FS#), R16.2
- net D2_1: now reaches I8.3 (Alert)
- net D2_1: now also DRV3.13 (D2#), R38.2
- net SDA_INA: now reaches I8.4 (SDA)
- net SDA_INA: now also I10.2 (A0), I10.4 (SDA), I11.4 (SDA), I12.2 (A0), I12.4 (SDA), I13.4 (SDA), I14.1 (A1), I14.4 (SDA)
- net SCL_INA: now reaches I8.5 (SCL)
- net SCL_INA: now also I10.5 (SCL), I11.2 (A0), I11.5 (SCL), I12.5 (SCL), I13.2 (A0), I13.5 (SCL), I14.5 (SCL)
- net FS6: now reaches DRV5.2 (FS#), R22.2
- net FS4: now reaches DRV6.2 (FS#), R23.2
- net D2_2: now reaches I10.3 (Alert)
- net D2_2: now also DRV1.13 (D2#), R39.2
- net FS2: now reaches DRV1.2 (FS#), R15.2
- new net: C44.1, I10.10 (IN+), R40.1
- new net: C44.2, I10.8 (VBUS), I10.9 (IN-), R32.1
- new net: C46.1, I12.10 (IN+), R48.1
- new net: C46.2, I12.8 (VBUS), I12.9 (IN-), R47.1
- new net: C45.2, I11.8 (VBUS), I11.9 (IN-), R43.1
- new net: C43.1, I8.10 (IN+), R36.1
- new net: C48.1, I14.10 (IN+), R56.1
- new net: C48.2, I14.8 (VBUS), I14.9 (IN-), R55.1
- new net: R19.2, U8.1
- new net: C45.1, I11.10 (IN+), R44.1
- new net: C43.2, I8.8 (VBUS), I8.9 (IN-), R12.1
- new net: C47.1, I13.10 (IN+), R52.1
- new net: R18.2, U7.1
- new net: C47.2, I13.8 (VBUS), I13.9 (IN-), R51.1
- new net +3,3v: JP4.3 (B)
- new net D2_3: DRV2.13 (D2#), I11.3 (Alert), R42.2
- new net D2_4: DRV6.13 (D2#), I12.3 (Alert), R46.2
- new net D2_5: DRV4.13 (D2#), I13.3 (Alert), R50.2
- new net D2_6: DRV5.13 (D2#), I14.3 (Alert), R54.2
- new net VS_ENC_M1: JP4.2 (C), R18.1, R19.1
- no-connect marks 48 -> 18
Other:
- moved on the sheet: C30, C31, C32, C33, C34, C35, C36, C37, C38, C39, C3_TANTAL1, C40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

Commit message: Add files via upload
Parts:
- removed C30: 100nF, Capacitor_SMD:C_0603_1608Metric, symbol 0805_C9900012713_5
- removed C31: 100nF, Capacitor_SMD:C_0603_1608Metric, symbol 0805_C9900012713_2
- removed C32, C43, C44, C45, C46, C47, C48: 100nF, Capacitor_SMD:C_0603_1608Metric, symbol 0805_C9900012713_1
- removed C33: 100nF, Capacitor_SMD:C_0603_1608Metric, symbol 0805_C9900012713_4
- removed C34: 100nF, Capacitor_SMD:C_0603_1608Metric, symbol 0805_C9900012713_3
- removed C35: 100nF, Capacitor_SMD:C_0603_1608Metric, symbol 0805_C9900012713
- removed C36: 100nF, Capacitor_SMD:C_0603_1608Metric, symbol 0805_C9900012713_8
- removed C37: 100nF, Capacitor_SMD:C_0603_1608Metric, symbol 0805_C9900012713_11
- removed C38: 100nF, Capacitor_SMD:C_0603_1608Metric, symbol 0805_C9900012713_7
- removed C39: 100nF, Capacitor_SMD:C_0603_1608Metric, symbol 0805_C9900012713_10
- removed C3_TANTAL1: 10uF, Capacitor_SMD:C_0603_1608Metric, symbol TANTALUM SMT CAPACITOR 330UF C
- removed C40: 100nF, Capacitor_SMD:C_1206_3216Metric, symbol 0805_C9900012713_9
- removed C41: 100nF, Capacitor_SMD:C_1206_3216Metric, symbol 0805_C9900012713_6
- removed C4_TANTAL1: 10uF, Capacitor_SMD:C_0603_1608Metric, symbol TANTALUM SMT CAPACITOR 330UF C_3
- removed C5_TANTAL1: 10uF, Capacitor_SMD:C_0603_1608Metric, symbol TANTALUM SMT CAPACITOR 330UF C_4
- removed C6_TANTAL1: 10uF, Capacitor_SMD:C_0603_1608Metric, symbol TANTALUM SMT CAPACITOR 330UF C_2
- removed C8_TANTAL1: 10uF, Capacitor_SMD:C_0603_1608Metric, symbol TANTALUM SMT CAPACITOR 330UF C_5
- removed C9_TANTAL1: 10uF, Capacitor_SMD:C_0603_1608Metric, symbol TANTALUM SMT CAPACITOR 330UF C_1
- removed D10: SS54L, Diode_SMD:D_0603_1608Metric, symbol SS54L
- removed D11: SS54L, Diode_SMD:D_0603_1608Metric, symbol SS54L_18
- removed D12: SS54L, Diode_SMD:D_0603_1608Metric, symbol SS54L_20
- removed D13: SS54L, Diode_SMD:D_0603_1608Metric, symbol SS54L_21
- removed D14: SS54L, Diode_SMD:D_0603_1608Metric, symbol SS54L_19
- removed D15: SS54L, Diode_SMD:D_0603_1608Metric, symbol SS54L_1
- removed D16: SS54L, Diode_SMD:D_0603_1608Metric, symbol SS54L_12
- removed D17: SS54L, Diode_SMD:D_0603_1608Metric, symbol SS54L_9
- removed D18: SS54L, Diode_SMD:D_0603_1608Metric, symbol SS54L_5
- removed D19: SS54L, Diode_SMD:D_0603_1608Metric, symbol SS54L_4
- removed D20: SS54L, Diode_SMD:D_0603_1608Metric, symbol SS54L_10
- removed D21: SS54L, Diode_SMD:D_0603_1608Metric, symbol SS54L_15
- removed D22: SS54L, Diode_SMD:D_0603_1608Metric, symbol SS54L_2
- removed D23: SS54L, Diode_SMD:D_0603_1608Metric, symbol SS54L_16
- removed D24: SS54L, Diode_SMD:D_0603_1608Metric, symbol SS54L_22
- removed D25: SS54L, Diode_SMD:D_0603_1608Metric, symbol SS54L_23
- removed D26: SS54L, Diode_SMD:D_0603_1608Metric, symbol SS54L_17
- removed D27: SS54L, Diode_SMD:D_0603_1608Metric, symbol SS54L_3
- removed D28: SS54L, Diode_SMD:D_0603_1608Metric, symbol SS54L_14
- removed D29: SS54L, Diode_SMD:D_0603_1608Metric, symbol SS54L_11
- removed D6: SS54L, Diode_SMD:D_0603_1608Metric, symbol SS54L_7
- removed D7: SS54L, Diode_SMD:D_0603_1608Metric, symbol SS54L_6
- removed D8: SS54L, Diode_SMD:D_0603_1608Metric, symbol SS54L_8
- removed D9: SS54L, Diode_SMD:D_0603_1608Metric, symbol SS54L_13
- removed R15: 1k, Resistor_SMD:R_0805_2012Metric, symbol 0805_2
- removed R16, R18, R19: 1k, Resistor_SMD:R_0805_2012Metric, symbol 0805_1
- removed R17: 1k, Resistor_SMD:R_0805_2012Metric, symbol 0805
- removed R21: 1k, Resistor_SMD:R_0805_2012Metric, symbol 0805_4
- removed R22: 1k, Resistor_SMD:R_0805_2012Metric, symbol 0805_5
- removed R23: 1k, Resistor_SMD:R_0805_2012Metric, symbol 0805_3
- removed R38, R39, R42, R46, R50, R54, R58, R59: 10k, Resistor_SMD:R_0805_2012Metric, symbol 0805
- added C31, C32, C33, C35, C37, C39, C40, C41, C42, C44, C46, C48, C49, C50, C51, C52, C53, C54: 100nF, Capacitor_SMD:C_0603_1608Metric, symbol Device:C
- added C34, C36, C38, C43, C45, C47: 10uF, Capacitor_SMD:C_0603_1608Metric, symbol Device:C_Polarized
- added Con4: (no value), Connector_PinHeader_1.00mm:PinHeader_1x02_P1.00mm_Vertical, symbol MyLIB:Con_power
- added D10, D11, D12, D13, D14, D15, D16, D17, D18, D19, D20, D21, D22, D23, D24, D25, D26, D27, D28, D29, D30, D7, D8, D9: SS54L, Diode_SMD:D_0603_1608Metric, symbol Diode:PMEG60T30ELR
- added J1, J2, J3, J4, J5, J6: Conn_01x05_Pin, Connector_PinHeader_1.00mm:PinHeader_1x05_P1.00mm_Vertical, symbol Connector:Conn_01x05_Pin
- added JP5, JP6, JP7, JP8, JP9: Jumper_3_Open, Jumper:SolderJumper-3_P1.3mm_Bridged123_Pad1.0x1.5mm, symbol Jumper:Jumper_3_Open
- added R17, R18, R19, R20, R21, R22, R47, R48, R49, R53, R54, R55, R59, R60, R61, R65, R66, R67: 1k, Resistor_SMD:R_0805_2012Metric, symbol Device:R
- added R26, R27, R29, R38, R39, R41, R50, R51, R52, R56, R57, R58, R62, R63, R64, R68, R69, R70: 10k, Resistor_SMD:R_0805_2012Metric, symbol Device:R
- added U10, U12, U13, U14, U15, U16, U17, U6, U7, U9: PC817, Package_DIP:DIP-4_W7.62mm_SMDSocket_SmallPads, symbol Isolator:PC817
- M_Con1, M_Con2, M_Con3, M_Con4, M_Con5, M_Con6: footprint Connector_PinHeader_2.00mm:PinHeader_1x06_P2.00mm_Vertical -> Library_footprints:KF202-7.5-6P
- renumbered I13 to I4, I11 to I5, I10 to I6, I8 to I7, I14 to I8, I12 to I9, R52 to R23, R44 to R24, R40 to R25, R53 to R28, R45 to R30, R41 to R31, R51 to R32, R43 to R33, R32 to R34, R36 to R35, R56 to R36, R48 to R37, R37 to R40, R57 to R42, R49 to R43, R12 to R44, R55 to R45, R47 to R46, U7 to U11
Connections:
- net VS_ENC_M1 is gone; now on an unnamed net: JP4.2 (C)
- net +14.4v: now also D10.1 (K), D11.1 (K), D12.1 (K), D13.1 (K), D14.1 (K), D15.1 (K), D16.1 (K), D17.1 (K), D18.1 (K), D7.1 (K), D8.1 (K), D9.1 (K); no longer DRV1.16 (V+), DRV1.4 (V+), DRV1.5 (V+), DRV2.16 (V+), DRV2.4 (V+), DRV2.5 (V+), DRV3.16 (V+), DRV3.4 (V+), DRV3.5 (V+), DRV4.16 (V+), DRV4.4 (V+), DRV4.5 (V+), DRV5.16 (V+), DRV5.4 (V+), DRV5.5 (V+), DRV6.16 (V+), DRV6.4 (V+), DRV6.5 (V+), M_Con2.3, M_Con3.3, M_Con4.3, M_Con5.3, M_Con6.3, R28.2, R30.2, R31.2, R32.2, R33.2, R34.2, R40.2, R42.2, R43.2, R44.2, R45.2, R46.2
- net +3,3v: now also JP5.3 (B), JP6.3 (B), JP7.3 (B), JP8.3 (B), JP9.3 (B)
- net +5v: now also JP5.1 (A), JP6.1 (A), JP7.1 (A), JP8.1 (A), JP9.1 (A), R17.1, R18.1, R19.1, R20.1, R21.1, R22.1, R26.1, R27.1, R29.1, R38.1, R39.1, R41.1, U10.4, U12.4, U13.4, U14.4, U15.4, U16.4, U17.4, U6.4, U7.4, U9.4
- net CONN_M1_1: now also D20.1 (K), D8.2 (A)
- net CONN_M1_2: now also D19.1 (K), D7.2 (A)
- net CONN_M2_1: now also D10.2 (A), D22.1 (K)
- net CONN_M2_2: now also D21.1 (K), D9.2 (A)
- net CONN_M3_1: now also D12.2 (A), D24.1 (K)
- net CONN_M3_2: now also D11.2 (A), D23.1 (K)
- net CONN_M4_1: now also D14.2 (A), D26.1 (K)
- net CONN_M4_2: now also D13.2 (A), D25.1 (K)
- net CONN_M5_1: now also D16.2 (A), D28.1 (K)
- net CONN_M5_2: now also D15.2 (A), D27.1 (K)
- net CONN_M6_1: now also D18.2 (A), D30.1 (K)
- net CONN_M6_2: now also D17.2 (A), D29.1 (K)
- net D2_1: now also R38.2
- net D2_2: now also R29.2
- net D2_3: now also R27.2
- net D2_4: now also R41.2
- net D2_5: now also R26.2
- net D2_6: now also R39.2
- net ENC_A_M1: now also R49.1; no longer U8.3
- net ENC_A_M2: now also R59.1
- net ENC_A_M3: now also R47.1
- net ENC_A_M4: now also R60.1
- net ENC_A_M5: now also R48.1
- net ENC_A_M6: now also R61.1
- net ENC_B_M1: now also R55.1; no longer U11.3
- net ENC_B_M2: now also R65.1
- net ENC_B_M3: now also R53.1
- net ENC_B_M4: now also R66.1
- net ENC_B_M5: now also R54.1
- net ENC_B_M6: now also R67.1
- net FS1: now also J2.3 (Pin_3), R19.2
- net FS2: now also J6.3 (Pin_3), R17.2
- net FS3: now also J1.3 (Pin_3), R18.2
- net FS4: now also J4.3 (Pin_3), R22.2
- net FS5: now also J3.3 (Pin_3), R20.2
- net FS6: now also J5.3 (Pin_3), R21.2
- net GND: now also C31.2, C32.2, C33.2, C34.2, C35.2, C36.2, C37.2, C38.2, C39.2, C40.2, C41.2, C42.2, C43.2, C44.2, C45.2, C46.2, C47.2, C48.2, D19.2 (A), D20.2 (A), D21.2 (A), D22.2 (A), D23.2 (A), D24.2 (A), D25.2 (A), D26.2 (A), D27.2 (A), D28.2 (A), D29.2 (A), D30.2 (A), R50.2, R51.2, R52.2, R56.2, R57.2, R58.2, R62.2, R63.2, R64.2, R68.2, R69.2, R70.2, U10.2, U12.2, U13.2, U14.2, U15.2, U16.2, U17.2, U6.2, U7.2, U9.2
- net IN1_M1: now also J2.1 (Pin_1)
- net IN1_M2: now also J6.1 (Pin_1)
- net IN1_M3: now also J1.1 (Pin_1)
- net IN1_M4: now also J4.1 (Pin_1)
- net IN1_M5: now also J3.1 (Pin_1)
- net IN1_M6: now also J5.1 (Pin_1)
- net IN2_M1: now also J2.2 (Pin_2)
- net IN2_M2: now also J6.2 (Pin_2)
- net IN2_M3: now also J1.2 (Pin_2)
- net IN2_M4: now also J4.2 (Pin_2)
- net IN2_M5: now also J3.2 (Pin_2)
- net IN2_M6: now also J5.2 (Pin_2)
- net SCL_INA: now also Con4.2
- net SDA_INA: now also Con4.1
- net at I6.10 (IN+), R25.1: now also C51.1
- net at I6.8 (VBUS), I6.9 (IN-), R34.1: now also C51.2
- net at I9.10 (IN+), R37.1: now also C54.1
- net at I9.8 (VBUS), I9.9 (IN-), R46.1: now also C54.2
- net at I5.8 (VBUS), I5.9 (IN-), R33.1: now also C50.2
- net at DRV5.17 (CCP): now also C41.1
- net at I7.10 (IN+), R35.1: now also C52.1
- net at I8.10 (IN+), R36.1: now also C53.1
- net at I8.8 (VBUS), I8.9 (IN-), R45.1: now also C53.2
- net at U8.1: now also R49.2
- net at I5.10 (IN+), R24.1: now also C50.1
- net at I7.8 (VBUS), I7.9 (IN-), R44.1: now also C52.2
- net at DRV3.17 (CCP): now also C33.1
- net at DRV4.17 (CCP): now also C40.1
- net at DRV2.17 (CCP): now also C32.1
- net at I4.10 (IN+), R23.1: now also C49.1
- net at U11.1: now also R55.2
- net at DRV6.17 (CCP): now also C42.1
- net at DRV1.17 (CCP): now also C31.1
- net at I4.8 (VBUS), I4.9 (IN-), R32.1: now also C49.2
- new net: JP8.2 (C), M_Con5.3
- new net: R48.2, U7.1
- new net: R53.2, U9.1
- new net: R60.2, U13.1
- new net: R65.2, U15.1
- new net: JP5.2 (C), M_Con2.3
- new net: JP6.2 (C), M_Con3.3
- new net: JP7.2 (C), M_Con4.3
- new net: R61.2, U14.1
- new net: R47.2, U6.1
- new net: R67.2, U17.1
- new net: R66.2, U16.1
- new net: JP9.2 (C), M_Con6.3
- new net: R59.2, U12.1
- new net: R54.2, U10.1
- new net ENC_A_M1_mk: J2.4 (Pin_4), R52.1, U8.3
- new net ENC_A_M2_mk: J6.4 (Pin_4), R62.1, U12.3
- new net ENC_A_M3_mk: J1.4 (Pin_4), R50.1, U6.3
- new net ENC_A_M4_mk: J4.4 (Pin_4), R63.1, U13.3
- new net ENC_A_M5_mk: J3.4 (Pin_4), R51.1, U7.3
- new net ENC_A_M6_mk: J5.4 (Pin_4), R64.1, U14.3
- new net ENC_B_M1_mk: J2.5 (Pin_5), R58.1, U11.3
- new net ENC_B_M2_mk: J6.5 (Pin_5), R68.1, U15.3
- new net ENC_B_M3_mk: J1.5 (Pin_5), R56.1, U9.3
- new net ENC_B_M4_mk: J4.5 (Pin_5), R69.1, U16.3
- new net ENC_B_M5_mk: J3.5 (Pin_5), R57.1, U10.3
- new net ENC_B_M6_mk: J5.5 (Pin_5), R70.1, U17.3
- new net INA1: C38.1, C39.1, DRV3.16 (V+), DRV3.4 (V+), DRV3.5 (V+), R40.2, R44.2
- new net INA2: C34.1, C35.1, DRV1.16 (V+), DRV1.4 (V+), DRV1.5 (V+), R31.2, R34.2
- new net INA3: C36.1, C37.1, DRV2.16 (V+), DRV2.4 (V+), DRV2.5 (V+), R30.2, R33.2
- new net INA4: C47.1, C48.1, DRV6.16 (V+), DRV6.4 (V+), DRV6.5 (V+), R43.2, R46.2
- new net INA5: C45.1, C46.1, DRV4.16 (V+), DRV4.4 (V+), DRV4.5 (V+), R28.2, R32.2
- new net INA6: C43.1, C44.1, DRV5.16 (V+), DRV5.4 (V+), DRV5.5 (V+), R42.2, R45.2
Other:
- note added: "I2C с INA226 на логическую плату"
- note added: "Сигналы с драйверов на физическое подключение моторов к силовой плате"
- note added: "Сигналы, идущие на логическую плату (по группам)"
- note added: "Физическое подключение моторов и энкодеров к силовой плате через клеммные колодки KF202 с пружинным зажимом"
- moved on the sheet: I4, I5, I6, I7, I8, I9, JP4, M_Con1, M_Con2, M_Con3, M_Con4, M_Con5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

Commit message: Add files via upload
Parts:
- DRV1, DRV2, DRV3, DRV4, DRV5, DRV6: footprint Package_SO:HSOP-20-1EP_11.0x15.9mm_P1.27mm_SlugDown -> Package_SO:HSOP-20-1EP_11.0x15.9mm_P1.27mm_SlugUp
Changed lines of the file:
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@@
 			)
 		)
-		(property "Footprint" "Package_SO:HSOP-20-1EP_11.0x15.9mm_P1.27mm_SlugDown"
+		(property "Footprint" "Package_SO:HSOP-20-1EP_11.0x15.9mm_P1.27mm_SlugUp"
 			(at 166.37 120.65 0)
 			(hide yes)
@@
 			)
 		)
-		(property "Footprint" "Package_SO:HSOP-20-1EP_11.0x15.9mm_P1.27mm_SlugDown"
+		(property "Footprint" "Package_SO:HSOP-20-1EP_11.0x15.9mm_P1.27mm_SlugUp"
 			(at 262.89 120.65 0)
 			(hide yes)
@@
 			)
 		)
-		(property "Footprint" "Package_SO:HSOP-20-1EP_11.0x15.9mm_P1.27mm_SlugDown"
+		(property "Footprint" "Package_SO:HSOP-20-1EP_11.0x15.9mm_P1.27mm_SlugUp"
 			(at 262.89 53.34 0)
 			(hide yes)
@@
 			)
 		)
-		(property "Footprint" "Package_SO:HSOP-20-1EP_11.0x15.9mm_P1.27mm_SlugDown"
+		(property "Footprint" "Package_SO:HSOP-20-1EP_11.0x15.9mm_P1.27mm_SlugUp"
 			(at 167.64 52.07 0)
 			(hide yes)
@@
 			)
 		)
-		(property "Footprint" "Package_SO:HSOP-20-1EP_11.0x15.9mm_P1.27mm_SlugDown"
+		(property "Footprint" "Package_SO:HSOP-20-1EP_11.0x15.9mm_P1.27mm_SlugUp"
 			(at 71.12 121.92 0)
 			(hide yes)
@@
 			)
 		)
-		(property "Footprint" "Package_SO:HSOP-20-1EP_11.0x15.9mm_P1.27mm_SlugDown"
+		(property "Footprint" "Package_SO:HSOP-20-1EP_11.0x15.9mm_P1.27mm_SlugUp"
 			(at 74.93 55.88 0)
 			(hide yes)

Commit message: Add files via upload
Parts:
- J1, J2, J3, J4, J5, J6: footprint Connector_PinHeader_1.00mm:PinHeader_1x05_P1.00mm_Vertical -> Connector_PinHeader_2.54mm:PinHeader_1x05_P2.54mm_Vertical
- renumbered C31 to C19, C32 to C20, C33 to C21, C34 to C22, C35 to C23, C36 to C24, C37 to C25, C38 to C26, C39 to C27, C40 to C28, C41 to C29, C42 to C30, C43 to C31, C44 to C32, C45 to C33, C46 to C34, C47 to C35, C48 to C36, C49 to C37, C50 to C38, C51 to C39, C52 to C40, C53 to C41, C54 to C42, U11 to U10, U12 to U11, U13 to U12, U14 to U13, U15 to U14, U16 to U15, U17 to U16, U6 to U5, U7 to U6, U8 to U7, U9 to U8, U10 to U9

Commit message: Add files via upload
Parts:
- Con4: footprint Connector_PinHeader_1.00mm:PinHeader_1x02_P1.00mm_Vertical -> Connector_PinHeader_2.54mm:PinHeader_1x02_P2.54mm_Vertical
Changed lines of the file:
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@@
 			)
 		)
-		(property "Footprint" "Connector_PinHeader_1.00mm:PinHeader_1x02_P1.00mm_Vertical"
+		(property "Footprint" "Connector_PinHeader_2.54mm:PinHeader_1x02_P2.54mm_Vertical"
 			(at 482.6 270.51 0)
 			(hide yes)
