File: motor_control.kicad_sch (KiCad schematic)
At the start: 145 parts, among them J1 Conn_01x05_Pin, J2 Conn_01x05_Pin, J3 Conn_01x05_Pin, J4 Conn_01x05_Pin, J5 Conn_01x05_Pin, J6 Conn_01x05_Pin, U10 PC817, U11 PC817, U12 PC817, U13 PC817, U14 PC817, U15 PC817, U16 PC817, U5 PC817, U6 PC817, U7 PC817, U8 PC817, U9 PC817

Commit message: trass
Parts:
- removed C22, C24, C31, C33, C35: 10uF, Capacitor_SMD:C_0603_1608Metric, symbol Device:C_Polarized
- removed C28, C30: 100nF, Capacitor_SMD:C_0603_1608Metric, symbol Device:C
- removed Con4: (no value), Connector_PinHeader_2.54mm:PinHeader_1x02_P2.54mm_Vertical, symbol MyLIB:Con_power
- removed D13, D14: SS54L, Diode_SMD:D_0603_1608Metric, symbol Diode:PMEG60T30ELR
- removed DRV1, DRV2, DRV3, DRV4, DRV5, DRV6: MC33886PVW, Package_SO:HSOP-20-1EP_11.0x15.9mm_P1.27mm_SlugUp, symbol MyLIB:Driver
- removed I4, I5, I6, I7, I8, I9: INA226, Package_SO:TSSOP-10_3x3mm_P0.5mm, symbol MyLIB:INA226
- removed J1, J2, J3, J4, J5, J6: Conn_01x05_Pin, Connector_PinHeader_2.54mm:PinHeader_1x05_P2.54mm_Vertical, symbol Connector:Conn_01x05_Pin
- removed R25, R32, R33, R34, R35, R36, R37, R44, R45, R46: 1, Resistor_SMD:R_0603_1608Metric, symbol Device:R
- removed R26, R27, R29, R38, R39, R41, R50, R51, R52, R56, R57, R58, R62, R63, R64, R68, R69, R70: 10k, Resistor_SMD:R_0805_2012Metric, symbol Device:R
- removed R28, R30, R31, R40, R42, R43: 10m, Resistor_SMD:R_0805_2012Metric, symbol Device:R
- removed R47, R48, R49, R53, R54, R55, R59, R60, R61, R65, R66, R67: 1k, Resistor_SMD:R_0805_2012Metric, symbol Device:R
- removed U10, U11, U12, U13, U14, U15, U16, U5, U6, U7, U8, U9: PC817, Package_DIP:DIP-4_W7.62mm_SMDSocket_SmallPads, symbol Isolator:PC817
- added ADC1: (no value), Package_SO:TSSOP-38_4.4x9.7mm_P0.5mm, symbol MyLIB:ADS7953
- added C22, C24, C55: 47nF, Capacitor_SMD:C_1210_3225Metric, symbol Device:C
- added C28, C30, C44, C46, C48: 10uF, Capacitor_SMD:C_0603_1608Metric, symbol Device:C_Polarized
- added C31, C33, C35, C49, C50, C51, C52, C53, C54, C61: 0.1uF, Capacitor_SMD:C_0603_1608Metric, symbol Device:C
- added C43, C45, C47: 1uF, Capacitor_SMD:C_0603_1608Metric, symbol Device:C
- added C56, C60: 10uF, Capacitor_SMD:C_0603_1608Metric, symbol Device:C
- added C57, C58, C59: 100nF, Capacitor_SMD:C_0603_1608Metric, symbol Device:C
- added C62: 1nF, Capacitor_SMD:C_0603_1608Metric, symbol Device:C
- added D19, D20: SS54L, Diode_SMD:D_0603_1608Metric, symbol Diode:PMEG60T30ELR
- added J1, J2: Conn_01x18_Pin, Connector_PinHeader_2.54mm:PinHeader_2x09_P2.54mm_Vertical, symbol Connector:Conn_01x18_Pin
- added J3: Conn_01x06_Pin, Connector_PinHeader_2.54mm:PinHeader_1x06_P2.54mm_Vertical, symbol Connector:Conn_01x06_Pin
- added Kontur2: (no value), Library_footprints:JetBot_AI_Kit_3x18650_Hole_Pattern, symbol MyLIB:Con_power
- added U10, U11, U6, U7, U8, U9: DRV8873SPWPRQ1, Library_footprints:C2150678_HTSSOP-24_L7_8-W4_4-P0_65-LS6_4-TL-EP, symbol lcsc_imported:DRV8873SPWPRQ1
- added U12: REF5025AD, Package_SO:SOIC-8_3.9x4.9mm_P1.27mm, symbol Reference_Voltage:REF5025AD
- added U13, U14, U15, U17, U18, U19, U20: ISO7762FDBQ, Package_SO:SSOP-16_3.9x4.9mm_P0.635mm, symbol Isolator:ISO7762FDBQ
- added U16: TLV9061xDBV, Package_TO_SOT_SMD:SOT-23-5, symbol Amplifier_Operational:TLV9061xDBV
- C19, C20, C21, C25, C27, C29, C37, C38, C39: value 100nF -> 1uF
- C23, C40, C41, C42: value 100nF -> 47nF; footprint Capacitor_SMD:C_0603_1608Metric -> Capacitor_SMD:C_1210_3225Metric
- C32, C34, C36: value 100nF -> 0.1uF
- JP4, JP5, JP6, JP7, JP8, JP9: footprint Jumper:SolderJumper-3_P1.3mm_Bridged123_Pad1.0x1.5mm -> Connector_PinHeader_2.54mm:PinHeader_1x03_P2.54mm_Vertical
- R17, R18, R19, R20, R21, R22: value 1k -> 10k
- R24: value 1 -> 10; footprint Resistor_SMD:R_0603_1608Metric -> Resistor_SMD:R_0805_2012Metric
- renumbered D20 to D13, D8 to D14, D19 to D7, D7 to D8
Connections:
- net FS2 is gone; now on net nFault_ISO: R17.2
- net FS3 is gone; now on net nFault_ISO: R18.2
- net FS4 is gone; now on net nFault_ISO: R22.2
- net FS5 is gone; now on net nFault_ISO: R20.2
- net FS6 is gone; now on net nFault_ISO: R21.2
- net INA4 is gone; now on net GND: C36.1
- net INA5 is gone; now on net GND: C34.1
- net INA6 is gone; now on net GND: C32.1
- net +14.4v: now also C25.2, C26.1, C27.2, C29.2, C32.2, C34.2, C36.2, D22.1 (K), D24.1 (K), D26.1 (K), D28.1 (K), D30.1 (K), C28.1, C30.1, C31.2, C33.2, C35.2, C43.2, C44.1, C45.2, C46.1, C47.2, C48.1, C49.2, C50.2, C51.2, C52.2, C53.2, C54.2, D20.1 (K), U10.13 (VM), U10.20 (VM), U11.13 (VM), U11.20 (VM), U6.13 (VM), U6.20 (VM), U7.13 (VM), U7.20 (VM), U8.13 (VM), U8.20 (VM), U9.13 (VM), U9.20 (VM); no longer D11.1 (K), D15.1 (K), D17.1 (K), D9.1 (K), R23.2, R24.2
- net +3,3v: now also R17.1, R18.1, R19.1, R20.1, R21.1, R22.1, U13.16 (Vcc2), U14.16 (Vcc2), U15.16 (Vcc2), U17.16 (Vcc2), U18.16 (Vcc2), U19.16 (Vcc2), U20.16 (Vcc2)
- net +5v: no longer R17.1, R18.1, R19.1, R20.1, R21.1, R22.1
- net ENC_A_M1: now also U13.11 (INE)
- net ENC_A_M1_mk: now also J1.5 (Pin_5), U13.6 (OUTE)
- net ENC_A_M2: now also U14.11 (INE)
- net ENC_A_M2_mk: now also J1.11 (Pin_11), U14.6 (OUTE)
- net ENC_A_M3: now also U15.11 (INE)
- net ENC_A_M3_mk: now also J1.17 (Pin_17), U15.6 (OUTE)
- net ENC_A_M4: now also U17.11 (INE)
- net ENC_A_M4_mk: now also J2.5 (Pin_5), U17.6 (OUTE)
- net ENC_A_M5: now also U19.11 (INE)
- net ENC_A_M5_mk: now also J2.11 (Pin_11), U19.6 (OUTE)
- net ENC_A_M6: now also U18.11 (INE)
- net ENC_A_M6_mk: now also J2.17 (Pin_17), U18.6 (OUTE)
- net ENC_B_M1: now also U13.10 (INF)
- net ENC_B_M1_mk: now also J1.6 (Pin_6), U13.7 (OUTF)
- net ENC_B_M2: now also U14.10 (INF)
- net ENC_B_M2_mk: now also J1.12 (Pin_12), U14.7 (OUTF)
- net ENC_B_M3: now also U15.10 (INF)
- net ENC_B_M3_mk: now also J1.18 (Pin_18), U15.7 (OUTF)
- net ENC_B_M4: now also U17.10 (INF)
- net ENC_B_M4_mk: now also J2.6 (Pin_6), U17.7 (OUTF)
- net ENC_B_M5: now also U19.10 (INF)
- net ENC_B_M5_mk: now also J2.12 (Pin_12), U19.7 (OUTF)
- net ENC_B_M6: now also U18.10 (INF)
- net ENC_B_M6_mk: now also J2.18 (Pin_18), U18.7 (OUTF)
- net GND: now also C19.1, C20.1, C21.1, C37.1, C38.1, C39.1, D11.2 (A), D15.2 (A), D17.2 (A), D9.2 (A), C28.2, C30.2, C31.1, C33.1, C35.1, C44.2, C46.2, C48.2, C49.1, C50.1, C51.1, C52.1, C53.1, C54.1, D19.2 (A), U10.16 (SRC), U10.17 (SRC), U10.24 (GND), U10.25 (EP), U11.16 (SRC), U11.17 (SRC), U11.24 (GND), U11.25 (EP), U13.9 (GND2), U14.9 (GND2), U15.9 (GND2), U17.9 (GND2), U18.9 (GND2), U19.9 (GND2), U20.9 (GND2), U6.16 (SRC), U6.17 (SRC), U6.24 (GND), U6.25 (EP), U7.16 (SRC), U7.17 (SRC), U7.24 (GND), U7.25 (EP), U8.16 (SRC), U8.17 (SRC), U8.24 (GND), U8.25 (EP), U9.16 (SRC), U9.17 (SRC), U9.24 (GND), U9.25 (EP); no longer C19.2, C20.2, C21.2, C23.2, C25.2, C27.2, C29.2, C32.2, C34.2, C36.2, D22.2 (A), D24.2 (A), D26.2 (A), D28.2 (A), D30.2 (A)
- net at C42.1: now also U11.23 (CPL)
- net at C42.2: now also U11.22 (CPH)
- net at C38.2: now also U10.1 (DVDD)
- net at C40.1: now also U9.23 (CPL)
- net at R24.1: now also U16.1, U16.4 (-); no longer C38.1
- net at C40.2: now also U9.22 (CPH)
- net at C29.1: now also U8.21 (VCP)
- net at C39.2: now also U11.1 (DVDD)
- net at R23.1: now also ADC1.4 (REFP), C60.1, U12.6 (Vout); no longer C37.1
- net at C41.1: now also U10.23 (CPL)
- net at C37.2: now also U9.1 (DVDD)
- net at C41.2: now also U10.22 (CPH)
- net CONN_M1_1 renamed CONN_2_M1
- net CONN_2_M1: now also M_Con1.1, U6.14 (OUT2), U6.15 (OUT2); no longer M_Con1.2
- net CONN_M1_2 renamed CONN_1_M1
- net CONN_1_M1: now also M_Con1.2, U6.18 (OUT1), U6.19 (OUT1); no longer M_Con1.1
- net CONN_M2_1 renamed CONN_1_M2
- net CONN_1_M2: now also D9.1 (K), U7.18 (OUT1), U7.19 (OUT1); no longer D22.1 (K)
- removed net CONN_M2_2: D21.1 (K), D9.2 (A), M_Con2.1
- net CONN_M3_1 renamed CONN_1_M3
- net CONN_1_M3: now also D11.1 (K), U8.18 (OUT1), U8.19 (OUT1); no longer D24.1 (K)
- removed net CONN_M3_2: D11.2 (A), D23.1 (K), M_Con3.1
- net CONN_M4_1 renamed CONN_1_M4
- net CONN_1_M4: now also D19.1 (K), D20.2 (A), U9.18 (OUT1), U9.19 (OUT1); no longer D26.1 (K)
- net CONN_M4_2 renamed CONN_2_M4
- net CONN_2_M4: now also D26.2 (A), U9.14 (OUT2), U9.15 (OUT2)
- removed net CONN_M5_1: D16.2 (A), D28.1 (K), M_Con5.2
- net CONN_M5_2 renamed CONN_2_M5
- net CONN_2_M5: now also D28.2 (A), U10.14 (OUT2), U10.15 (OUT2); no longer D15.2 (A)
- removed net CONN_M6_1: D18.2 (A), D30.1 (K), M_Con6.2
- net CONN_M6_2 renamed CONN_2_M6
- net CONN_2_M6: now also D30.2 (A), U11.14 (OUT2), U11.15 (OUT2); no longer D17.2 (A)
- net FS1 renamed nFault_ISO
- net nFault_ISO: now also U10.2 (nFAULT), U11.2 (nFAULT), U20.10 (INF), U6.2 (nFAULT), U7.2 (nFAULT), U8.2 (nFAULT), U9.2 (nFAULT)
- net INA1: no longer names the net of C27.1
- net INA1: now also U7.21 (VCP); no longer C26.1
- net INA2: no longer names the net of C23.1
- net INA2: now also U7.23 (CPL)
- net INA3: no longer names the net of C25.1
- net INA3: now also U6.21 (VCP)
- new net: C23.2, U7.22 (CPH)
- new net: J3.1 (Pin_1), U20.2 (INA)
- new net: J3.2 (Pin_2), U20.3 (INB)
- new net: J3.3 (Pin_3), U20.4 (INC)
- new net: J3.4 (Pin_4), U20.5 (IND)
- new net: J3.6 (Pin_6), U20.7 (OUTF)
- new net: C43.1, U9.21 (VCP)
- new net: C19.2, U6.1 (DVDD)
- new net: C22.2, U6.22 (CPH)
- new net: C22.1, U6.23 (CPL)
- new net: C20.2, U7.1 (DVDD)
- new net: ADC1.8 (AINP), C62.2, R24.2
- new net: C24.1, U8.23 (CPL)
- new net: C24.2, U8.22 (CPH)
- new net: ADC1.7 (MXO), U16.3 (+)
- new net: C21.2, U8.1 (DVDD)
- new net: C45.1, U10.21 (VCP)
- new net: C55.1, R23.2
- new net: C47.1, U11.21 (VCP)
- new net +3,3v*: ADC1.29 (+VA), ADC1.36 (+VBD), ADC1.5 (+VA), C56.1, C57.1, C58.1, C59.1, C61.2, U12.2 (Vin), U13.1 (Vcc1), U14.1 (Vcc1), U15.1 (Vcc1), U16.5 (V+), U17.1 (Vcc1), U18.1 (Vcc1), U19.1 (Vcc1), U20.1 (Vcc1)
- new net CONN_1_M5: D21.1 (K), D22.2 (A), M_Con5.2, U10.18 (OUT1), U10.19 (OUT1)
- new net CONN_1_M6: D23.1 (K), D24.2 (A), M_Con6.2, U11.18 (OUT1), U11.19 (OUT1)
- new net CONN_2_M2: D15.1 (K), D16.2 (A), M_Con2.1, U7.14 (OUT2), U7.15 (OUT2)
- new net CONN_2_M3: D17.1 (K), D18.2 (A), M_Con3.1, U8.14 (OUT2), U8.15 (OUT2)
- new net CS_ISO: ADC1.31 (CS#), U20.13 (OUTC)
- new net DISABLE_ISO_1: U13.12 (OUTD), U6.9 (DISABLE)
- new net DISABLE_ISO_2: U14.12 (OUTD), U7.9 (DISABLE)
- new net DISABLE_ISO_3: U15.12 (OUTD), U8.9 (DISABLE)
- new net DISABLE_ISO_4: U17.12 (OUTD), U9.9 (DISABLE)
- new net DISABLE_ISO_5: U10.9 (DISABLE), U19.12 (OUTD)
- new net DISABLE_ISO_6: U11.9 (DISABLE), U18.12 (OUTD)
- new net DISABLE_mk_1: J1.4 (Pin_4), U13.5 (IND)
- new net DISABLE_mk_2: J1.10 (Pin_10), U14.5 (IND)
- new net DISABLE_mk_3: J1.16 (Pin_16), U15.5 (IND)
- new net DISABLE_mk_4: J2.4 (Pin_4), U17.5 (IND)
- new net DISABLE_mk_5: J2.10 (Pin_10), U19.5 (IND)
- new net DISABLE_mk_6: J2.16 (Pin_16), U18.5 (IND)
- new net EN/IN1_ISO_1: U13.14 (OUTB), U6.7 (EN/IN1)
- new net EN/IN1_ISO_2: U14.14 (OUTB), U7.7 (EN/IN1)
- new net EN/IN1_ISO_3: U15.14 (OUTB), U8.7 (EN/IN1)
- new net EN/IN1_ISO_4: U17.14 (OUTB), U9.7 (EN/IN1)
- new net EN/IN1_ISO_5: U10.7 (EN/IN1), U19.14 (OUTB)
- new net EN/IN1_ISO_6: U11.7 (EN/IN1), U18.14 (OUTB)
- new net EN/IN1_mk_1: J1.2 (Pin_2), U13.3 (INB)
- new net EN/IN1_mk_2: J1.8 (Pin_8), U14.3 (INB)
- new net EN/IN1_mk_3: J1.14 (Pin_14), U15.3 (INB)
- new net EN/IN1_mk_4: J2.2 (Pin_2), U17.3 (INB)
- new net EN/IN1_mk_5: J2.8 (Pin_8), U19.3 (INB)
- new net EN/IN1_mk_6: J2.14 (Pin_14), U18.3 (INB)
- new net GND*: ADC1.10 (AGND), ADC1.19 (AGND), ADC1.20 (AGND), ADC1.3 (REFM), ADC1.30 (AGND), ADC1.35 (BDGND), ADC1.6 (AGND), ADC1.9 (AINM), C55.2, C56.2, C57.2, C58.2, C59.2, C60.2, C61.1, C62.1, U12.4 (GND), U13.8 (GND1), U14.8 (GND1), U15.8 (GND1), U16.2 (V-), U17.8 (GND1), U18.8 (GND1), U19.8 (GND1), U20.8 (GND1)
- new net IPROPI1_1: ADC1.11 (CH15), U6.10 (IPROPI1)
- new net IPROPI1_2: ADC1.13 (CH13), U7.10 (IPROPI1)
- new net IPROPI1_3: ADC1.15 (CH11), U8.10 (IPROPI1)
- new net IPROPI1_4: ADC1.28 (CH0), U9.10 (IPROPI1)
- new net IPROPI1_5: ADC1.26 (CH2), U10.10 (IPROPI1)
- new net IPROPI1_6: ADC1.24 (CH4), U11.10 (IPROPI1)
- new net IPROPI2_1: ADC1.12 (CH14), U6.12 (IPROPI2)
- new net IPROPI2_2: ADC1.14 (CH12), U7.12 (IPROPI2)
- new net IPROPI2_3: ADC1.16 (CH10), U8.12 (IPROPI2)
- new net IPROPI2_4: ADC1.27 (CH1), U9.12 (IPROPI2)
- new net IPROPI2_5: ADC1.25 (CH3), U10.12 (IPROPI2)
- new net IPROPI2_6: ADC1.23 (CH5), U11.12 (IPROPI2)
- new net PH/IN2_ISO_1: U13.13 (OUTC), U6.8 (PH/IN2)
- new net PH/IN2_ISO_2: U14.13 (OUTC), U7.8 (PH/IN2)
- new net PH/IN2_ISO_3: U15.13 (OUTC), U8.8 (PH/IN2)
- new net PH/IN2_ISO_4: U17.13 (OUTC), U9.8 (PH/IN2)
- new net PH/IN2_ISO_5: U10.8 (PH/IN2), U19.13 (OUTC)
- new net PH/IN2_ISO_6: U11.8 (PH/IN2), U18.13 (OUTC)
- new net PH/IN2_mk_1: J1.3 (Pin_3), U13.4 (INC)
- new net PH/IN2_mk_2: J1.9 (Pin_9), U14.4 (INC)
- new net PH/IN2_mk_3: J1.15 (Pin_15), U15.4 (INC)
- new net PH/IN2_mk_4: J2.3 (Pin_3), U17.4 (INC)
- new net PH/IN2_mk_5: J2.9 (Pin_9), U19.4 (INC)
- new net PH/IN2_mk_6: J2.15 (Pin_15), U18.4 (INC)
- new net SCLK_ISO: ADC1.32 (SCLK), U10.5 (SCLK), U11.5 (SCLK), U20.14 (OUTB), U6.5 (SCLK), U7.5 (SCLK), U8.5 (SCLK), U9.5 (SCLK)
- new net SDI_ISO: ADC1.33 (SDI), U10.4 (SDI), U11.4 (SDI), U20.15 (OUTA), U6.4 (SDI), U7.4 (SDI), U8.4 (SDI), U9.4 (SDI)
- new net SDO_ISO: ADC1.34 (SDO), U10.3 (SDO), U11.3 (SDO), U20.11 (INE), U6.3 (SDO), U7.3 (SDO), U8.3 (SDO), U9.3 (SDO)
- new net nSCS_ISO_1: U13.15 (OUTA), U6.6 (nSCS)
- new net nSCS_ISO_2: U14.15 (OUTA), U7.6 (nSCS)
- new net nSCS_ISO_3: U15.15 (OUTA), U8.6 (nSCS)
- new net nSCS_ISO_4: U17.15 (OUTA), U9.6 (nSCS)
- new net nSCS_ISO_5: U10.6 (nSCS), U19.15 (OUTA)
- new net nSCS_ISO_6: U11.6 (nSCS), U18.15 (OUTA)
- new net nSCS_mk_1: J1.1 (Pin_1), U13.2 (INA)
- new net nSCS_mk_2: J1.7 (Pin_7), U14.2 (INA)
- new net nSCS_mk_3: J1.13 (Pin_13), U15.2 (INA)
- new net nSCS_mk_4: J2.1 (Pin_1), U17.2 (INA)
- new net nSCS_mk_5: J2.7 (Pin_7), U19.2 (INA)
- new net nSCS_mk_6: J2.13 (Pin_13), U18.2 (INA)
- no-connect marks 18 -> 21
Other:
- note removed: "I2C с INA226 на логическую плату"
- note removed: "Сигналы с драйверов на физическое подключение моторов к силовой плате"
- note removed: "Сигналы, идущие на логическую плату (по группам)"
- moved on the sheet: D13, D14, D7, D8

Commit message: tray
Parts:
- removed J3: Conn_01x06_Pin, Connector_PinHeader_2.54mm:PinHeader_1x06_P2.54mm_Vertical, symbol Connector:Conn_01x06_Pin
- added ISO8: ISO1540, Package_SO:SOIC-8_3.9x4.9mm_P1.27mm, symbol Isolator:ISO1540
- added J3: Conn_01x12_Pin, Connector_PinHeader_2.54mm:PinHeader_2x06_P2.54mm_Vertical, symbol Connector:Conn_01x12_Pin
- renumbered U6 to DRV1, U7 to DRV2, U8 to DRV3, U9 to DRV4, U10 to DRV5, U11 to DRV6, U13 to ISO1, U14 to ISO2, U15 to ISO3, U17 to ISO4, U18 to ISO5, U19 to ISO6, U20 to ISO7, Kontur2 to Kontur1, U16 to OPER1, U12 to REF1
Connections:
- net +3,3v: now also ISO8.1 (VCC1)
- net +3,3v*: now also ISO8.8 (VCC2), J3.10 (Pin_10)
- net +5v: now also J3.9 (Pin_9)
- net CONN_1_M1: now also M_Con1.3; no longer M_Con1.2
- net CONN_1_M2: now also M_Con2.3; no longer M_Con2.2
- net CONN_1_M3: now also M_Con3.3; no longer M_Con3.2
- net CONN_1_M4: now also M_Con4.3; no longer M_Con4.2
- net CONN_1_M5: now also M_Con5.3; no longer M_Con5.2
- net CONN_1_M6: now also M_Con6.3; no longer M_Con6.2
- net CONN_2_M1: now also M_Con1.4; no longer M_Con1.1
- net CONN_2_M2: now also M_Con2.4; no longer M_Con2.1
- net CONN_2_M3: now also M_Con3.4; no longer M_Con3.1
- net CONN_2_M4: now also M_Con4.4; no longer M_Con4.1
- net CONN_2_M5: now also M_Con5.4; no longer M_Con5.1
- net CONN_2_M6: now also M_Con6.4; no longer M_Con6.1
- net DISABLE_mk_2: now also J2.4 (Pin_4); no longer J1.10 (Pin_10)
- net DISABLE_mk_3: now also J1.10 (Pin_10); no longer J1.16 (Pin_16)
- net DISABLE_mk_4: now also J2.10 (Pin_10); no longer J2.4 (Pin_4)
- net DISABLE_mk_5: now also J1.16 (Pin_16); no longer J2.10 (Pin_10)
- net ENC_A_M2: now also M_Con2.1; no longer M_Con2.5
- net ENC_A_M2_mk: now also J2.5 (Pin_5); no longer J1.11 (Pin_11)
- net ENC_A_M3_mk: now also J1.11 (Pin_11); no longer J1.17 (Pin_17)
- net ENC_A_M4: now also M_Con4.1; no longer M_Con4.5
- net ENC_A_M4_mk: now also J2.11 (Pin_11); no longer J2.5 (Pin_5)
- net ENC_A_M5_mk: now also J1.17 (Pin_17); no longer J2.11 (Pin_11)
- net ENC_A_M6: now also M_Con6.1; no longer M_Con6.5
- net ENC_B_M1: now also M_Con1.6; no longer M_Con1.4
- net ENC_B_M2: now also M_Con2.2; no longer M_Con2.4
- net ENC_B_M2_mk: now also J2.6 (Pin_6); no longer J1.12 (Pin_12)
- net ENC_B_M3: now also M_Con3.6; no longer M_Con3.4
- net ENC_B_M3_mk: now also J1.12 (Pin_12); no longer J1.18 (Pin_18)
- net ENC_B_M4: now also M_Con4.2; no longer M_Con4.4
- net ENC_B_M4_mk: now also J2.12 (Pin_12); no longer J2.6 (Pin_6)
- net ENC_B_M5: now also M_Con5.6; no longer M_Con5.4
- net ENC_B_M5_mk: now also J1.18 (Pin_18); no longer J2.12 (Pin_12)
- net ENC_B_M6: now also M_Con6.2; no longer M_Con6.4
- net EN/IN1_mk_2: now also J2.2 (Pin_2); no longer J1.8 (Pin_8)
- net EN/IN1_mk_3: now also J1.8 (Pin_8); no longer J1.14 (Pin_14)
- net EN/IN1_mk_4: now also J2.8 (Pin_8); no longer J2.2 (Pin_2)
- net EN/IN1_mk_5: now also J1.14 (Pin_14); no longer J2.8 (Pin_8)
- net GND: now also M_Con1.2, M_Con2.5, M_Con3.2, M_Con4.5, M_Con5.2, M_Con6.5, ISO8.4 (GND1), J3.11 (Pin_11); no longer M_Con1.6, M_Con2.6, M_Con3.6, M_Con4.6, M_Con5.6, M_Con6.6
- net GND*: now also ISO8.5 (GND2), J3.12 (Pin_12)
- net IPROPI1_2: now also ADC1.28 (CH0); no longer ADC1.13 (CH13)
- net IPROPI1_3: now also ADC1.13 (CH13); no longer ADC1.15 (CH11)
- net IPROPI1_4: now also ADC1.26 (CH2); no longer ADC1.28 (CH0)
- net IPROPI1_5: now also ADC1.16 (CH10); no longer ADC1.26 (CH2)
- net IPROPI2_2: now also ADC1.27 (CH1); no longer ADC1.14 (CH12)
- net IPROPI2_3: now also ADC1.14 (CH12); no longer ADC1.16 (CH10)
- net IPROPI2_4: now also ADC1.25 (CH3); no longer ADC1.27 (CH1)
- net IPROPI2_5: now also ADC1.15 (CH11); no longer ADC1.25 (CH3)
- net PH/IN2_mk_2: now also J2.3 (Pin_3); no longer J1.9 (Pin_9)
- net PH/IN2_mk_3: now also J1.9 (Pin_9); no longer J1.15 (Pin_15)
- net PH/IN2_mk_4: now also J2.9 (Pin_9); no longer J2.3 (Pin_3)
- net PH/IN2_mk_5: now also J1.15 (Pin_15); no longer J2.9 (Pin_9)
- net nSCS_mk_2: now also J2.1 (Pin_1); no longer J1.7 (Pin_7)
- net nSCS_mk_3: now also J1.7 (Pin_7); no longer J1.13 (Pin_13)
- net nSCS_mk_4: now also J2.7 (Pin_7); no longer J2.1 (Pin_1)
- net nSCS_mk_5: now also J1.13 (Pin_13); no longer J2.7 (Pin_7)
- net at JP8.2 (C): now also M_Con5.1; no longer M_Con5.3
- net at ISO7.2 (INA): now also J3.1 (Pin_1)
- net at ISO7.3 (INB): now also J3.2 (Pin_2)
- net at ISO7.4 (INC): now also J3.3 (Pin_3)
- net at ISO7.5 (IND): now also J3.4 (Pin_4)
- net at ISO7.7 (OUTF): now also J3.6 (Pin_6)
- net at JP5.2 (C): now also M_Con2.6; no longer M_Con2.3
- net at JP6.2 (C): now also M_Con3.1; no longer M_Con3.3
- net at JP7.2 (C): now also M_Con4.6; no longer M_Con4.3
- net at JP4.2 (C): now also M_Con1.1; no longer M_Con1.3
- net at JP9.2 (C): now also M_Con6.6; no longer M_Con6.3
- new net: ISO8.7 (SDA2), J3.5 (Pin_5)
- new net: ISO8.6 (SCL2), J3.7 (Pin_7)
- new net +5v*: J3.8 (Pin_8)
- new net SCL_INA: ISO8.3 (SCL1)
- new net SDA_INA: ISO8.2 (SDA1)
- no-connect marks 21 -> 20
Other:
- moved on the sheet: JP4, JP5, JP6, JP8

Commit message: trass
Parts:
- removed J3: Conn_01x12_Pin, Connector_PinHeader_2.54mm:PinHeader_2x06_P2.54mm_Vertical, symbol Connector:Conn_01x12_Pin
- added J3: Conn_01x10_Pin, Connector_PinHeader_2.54mm:PinHeader_2x05_P2.54mm_Vertical, symbol Connector:Conn_01x10_Pin
- renumbered C19 to C18, C20 to C19, C21 to C20, C22 to C21, C23 to C22, C24 to C23, C25 to C24, C26 to C25, C27 to C26, C28 to C27, C29 to C28, C30 to C29, C31 to C30, C32 to C31, C33 to C32, C34 to C33, C35 to C34, C36 to C35, C37 to C36, C38 to C37, C39 to C38, C40 to C39, C41 to C40, C42 to C41, C43 to C42, C44 to C43, C45 to C44, C46 to C45, C47 to C46, C48 to C47, C49 to C48, C50 to C49, C51 to C50, C52 to C51, C53 to C52, C54 to C53, C55 to C54, C56 to C55, C57 to C56, C58 to C57, C59 to C58, C60 to C59, C61 to C60, C62 to C61, R17 to R18, R18 to R19, R19 to R20, R20 to R21, R21 to R22, R22 to R23, R23 to R24, R24 to R25
Connections:
- net +3,3v* is gone; now on net +3,3v: ADC1.29 (+VA), ADC1.36 (+VBD), ADC1.5 (+VA), C55.1, C56.1, C57.1, C58.1, C60.2, ISO1.1 (Vcc1), ISO2.1 (Vcc1), ISO3.1 (Vcc1), ISO4.1 (Vcc1), ISO5.1 (Vcc1), ISO6.1 (Vcc1), ISO7.1 (Vcc1), ISO8.8 (VCC2), OPER1.5 (V+), REF1.2 (Vin)
- net GND* is gone; now on net GND: ADC1.10 (AGND), ADC1.19 (AGND), ADC1.20 (AGND), ADC1.3 (REFM), ADC1.30 (AGND), ADC1.35 (BDGND), ADC1.6 (AGND), ADC1.9 (AINM), C54.2, C55.2, C56.2, C57.2, C58.2, C59.2, C60.1, C61.1, ISO1.8 (GND1), ISO2.8 (GND1), ISO3.8 (GND1), ISO4.8 (GND1), ISO5.8 (GND1), ISO6.8 (GND1), ISO7.8 (GND1), ISO8.5 (GND2), OPER1.2 (V-), REF1.4 (GND)
- net +3,3v: now also J3.7 (Pin_7)
- net +5v: now also J3.5 (Pin_5)
- net GND: now also J3.9 (Pin_9)
- net at ISO7.2 (INA): now also J3.2 (Pin_2)
- net at ISO7.3 (INB): now also J3.4 (Pin_4)
- net at ISO7.4 (INC): now also J3.6 (Pin_6)
- net at ISO7.5 (IND): now also J3.8 (Pin_8)
- net at ISO7.7 (OUTF): now also J3.10 (Pin_10)
- net at ISO8.7 (SDA2): now also J3.1 (Pin_1)
- net at ISO8.6 (SCL2): now also J3.3 (Pin_3)

Commit message: I2C
Connections:
- net CS_ISO: now also ISO7.11 (INE); no longer ISO7.13 (OUTC)
- net DISABLE_mk_1: now also J1.3 (Pin_3); no longer J1.4 (Pin_4)
- net DISABLE_mk_4: now also J2.9 (Pin_9); no longer J2.10 (Pin_10)
- net DISABLE_mk_5: now also J1.15 (Pin_15); no longer J1.16 (Pin_16)
- net DISABLE_mk_6: now also J2.15 (Pin_15); no longer J2.16 (Pin_16)
- net ENC_A_M1_mk: now also J1.6 (Pin_6); no longer J1.5 (Pin_5)
- net ENC_A_M2_mk: now also J2.1 (Pin_1); no longer J2.5 (Pin_5)
- net ENC_A_M3_mk: now also J1.7 (Pin_7); no longer J1.11 (Pin_11)
- net ENC_A_M4_mk: now also J2.12 (Pin_12); no longer J2.11 (Pin_11)
- net ENC_A_M5_mk: now also J1.18 (Pin_18); no longer J1.17 (Pin_17)
- net ENC_A_M6_mk: now also J2.18 (Pin_18); no longer J2.17 (Pin_17)
- net ENC_B_M1_mk: now also J1.5 (Pin_5); no longer J1.6 (Pin_6)
- net ENC_B_M2_mk: now also J2.2 (Pin_2); no longer J2.6 (Pin_6)
- net ENC_B_M3_mk: now also J1.8 (Pin_8); no longer J1.12 (Pin_12)
- net ENC_B_M4_mk: now also J2.11 (Pin_11); no longer J2.12 (Pin_12)
- net ENC_B_M5_mk: now also J1.17 (Pin_17); no longer J1.18 (Pin_18)
- net ENC_B_M6_mk: now also J2.17 (Pin_17); no longer J2.18 (Pin_18)
- net EN/IN1_mk_1: now also J1.1 (Pin_1); no longer J1.2 (Pin_2)
- net EN/IN1_mk_2: now also J2.6 (Pin_6); no longer J2.2 (Pin_2)
- net EN/IN1_mk_3: now also J1.12 (Pin_12); no longer J1.8 (Pin_8)
- net EN/IN1_mk_4: now also J2.7 (Pin_7); no longer J2.8 (Pin_8)
- net EN/IN1_mk_5: now also J1.13 (Pin_13); no longer J1.14 (Pin_14)
- net EN/IN1_mk_6: now also J2.13 (Pin_13); no longer J2.14 (Pin_14)
- net PH/IN2_mk_1: now also J1.4 (Pin_4); no longer J1.3 (Pin_3)
- net PH/IN2_mk_4: now also J2.10 (Pin_10); no longer J2.9 (Pin_9)
- net PH/IN2_mk_5: now also J1.16 (Pin_16); no longer J1.15 (Pin_15)
- net PH/IN2_mk_6: now also J2.16 (Pin_16); no longer J2.15 (Pin_15)
- net SDI_ISO: now also ISO7.13 (OUTC); no longer ISO7.15 (OUTA)
- net SDO_ISO: now also ISO7.12 (OUTD); no longer ISO7.11 (INE)
- net nSCS_mk_1: now also J1.2 (Pin_2); no longer J1.1 (Pin_1)
- net nSCS_mk_2: now also J2.5 (Pin_5); no longer J2.1 (Pin_1)
- net nSCS_mk_3: now also J1.11 (Pin_11); no longer J1.7 (Pin_7)
- net nSCS_mk_4: now also J2.8 (Pin_8); no longer J2.7 (Pin_7)
- net nSCS_mk_5: now also J1.14 (Pin_14); no longer J1.13 (Pin_13)
- net nSCS_mk_6: now also J2.14 (Pin_14); no longer J2.13 (Pin_13)

Commit message: 3v3MK
Connections:
- net CONN_1_M1: now also M_Con1.4; no longer M_Con1.3
- net CONN_1_M6: now also M_Con6.4; no longer M_Con6.3
- net CONN_2_M1: now also M_Con1.3; no longer M_Con1.4
- net CONN_2_M6: now also M_Con6.3; no longer M_Con6.4
Changed lines of the file:
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@@
 	(wire
 		(pts
+			(xy 538.48 31.75) (xy 546.1 31.75)
+		)
+		(stroke
+			(width 0)
+			(type default)
+		)
+	)
+	(wire
+		(pts
 			(xy 473.71 186.69) (xy 473.71 187.96)
 		)
@@
 	(wire
 		(pts
+			(xy 538.48 34.29) (xy 546.1 34.29)
+		)
+		(stroke
+			(width 0)
+			(type default)
+		)
+	)
+	(wire
+		(pts
 			(xy 347.98 54.61) (xy 349.25 54.61)
 		)
@@
 	(wire
 		(pts
-			(xy 535.94 156.21) (xy 546.1 156.21)
-		)
-		(stroke
-			(width 0)
-			(type default)
-		)
-	)
-	(wire
-		(pts
 			(xy 356.87 106.68) (xy 359.41 106.68)
 		)
@@
 	(wire
 		(pts
-			(xy 535.94 158.75) (xy 546.1 158.75)
-		)
-		(stroke
-			(width 0)
-			(type default)
-		)
-	)
-	(wire
-		(pts
 			(xy 515.62 129.54) (xy 515.62 125.73)
 		)
@@
 	(wire
 		(pts
-			(xy 538.48 31.75) (xy 546.1 31.75)
-		)
-		(stroke
-			(width 0)
-			(type default)
-		)
-	)
-	(wire
-		(pts
 			(xy 383.54 64.77) (xy 386.08 64.77)
 		)
@@
 	(wire
 		(pts
+			(xy 535.94 156.21) (xy 546.1 156.21)
+		)
+		(stroke
+			(width 0)
+			(type default)
+		)
+	)
+	(wire
+		(pts
 			(xy 260.35 189.23) (xy 256.54 189.23)
 		)
@@
 	(wire
 		(pts
+			(xy 535.94 158.75) (xy 546.1 158.75)
+		)
+		(stroke
+			(width 0)
+			(type default)
+		)
+	)
+	(wire
+		(pts
 			(xy 424.18 213.36) (xy 425.45 213.36)
 		)
@@
 	(wire
 		(pts
-			(xy 538.48 34.29) (xy 546.1 34.29)
-		)
-		(stroke
-			(width 0)
-			(type default)
-		)
-	)
-	(wire
-		(pts
 			(xy 113.03 293.37) (xy 110.49 293.37)
 		)
@@
 	(global_label "CONN_1_M6"
 		(shape input)
-		(at 535.94 156.21 180)
+		(at 535.94 158.75 180)
 		(effects
 			(font
@@
 		)
 		(property "Intersheetrefs" "${INTERSHEET_REFS}"
-			(at 535.94 156.21 0)
+			(at 535.94 158.75 0)
 			(hide yes)
 			(show_name no)
@@
 	(global_label "CONN_2_M6"
 		(shape input)
-		(at 535.94 158.75 180)
+		(at 535.94 156.21 180)
 		(effects
 			(font
@@
 		)
 		(property "Intersheetrefs" "${INTERSHEET_REFS}"
-			(at 535.94 158.75 0)
+			(at 535.94 156.21 0)
 			(hide yes)
 			(show_name no)
@@
 	(global_label "CONN_2_M1"
 		(shape input)
-		(at 538.48 34.29 180)
+		(at 538.48 31.75 180)
 		(effects
 			(font
@@
 		)
 		(property "Intersheetrefs" "${INTERSHEET_REFS}"
-			(at 538.48 34.29 0)
+			(at 538.48 31.75 0)
 			(hide yes)
 			(show_name no)
@@
 	(global_label "CONN_1_M1"
 		(shape input)
-		(at 538.48 31.75 180)
+		(at 538.48 34.29 180)
 		(effects
 			(font
@@
 		)
 		(property "Intersheetrefs" "${INTERSHEET_REFS}"
-			(at 538.48 31.75 0)
+			(at 538.48 34.29 0)
 			(hide yes)
 			(show_name no)
